File: RF-SWITCH.kicad_sch (KiCad schematic)
At the start: 4 parts, among them K1 G6S-2, K2 G6S-2

Commit message: more
Parts:
- added J1: BNC, Xenir:BNC, symbol Xenir:BNC
Connections:
- net Antenna: no longer names the net of K2.4, K2.9
- net Antenna: now also J1.S (OUT)
- new net GND: J1.GND
Changed lines of the file:
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@@
     (stroke (width 0) (type default) (color 0 0 0 0))
   )
-  (wire (pts (xy 180.34 105.41) (xy 182.88 105.41))
+  (wire (pts (xy 180.34 105.41) (xy 196.85 105.41))
     (stroke (width 0) (type default) (color 0 0 0 0))
   )
@@
     (effects (font (size 1.27 1.27)) (justify left))
   )
-  (hierarchical_label "Antenna" (shape input) (at 182.88 105.41 0)
-    (effects (font (size 1.27 1.27)) (justify left))
-  )
   (hierarchical_label "From-Enc" (shape input) (at 99.06 97.79 180)
     (effects (font (size 1.27 1.27)) (justify right))
@@
   (hierarchical_label "PA-IN" (shape input) (at 99.06 107.95 180)
     (effects (font (size 1.27 1.27)) (justify right))
+  )
+  (symbol (lib_id "Xenir:BNC") (at 201.93 105.41 0) (mirror y) (unit 1)
+    (in_bom yes) (on_board yes) (fields_autoplaced)
+    (property "Reference" "J1" (id 0) (at 205.74 104.1399 0)
+      (effects (font (size 1.27 1.27)) (justify right))
+    )
+    (property "Value" "BNC" (id 1) (at 205.74 106.6799 0)
+      (effects (font (size 1.27 1.27)) (justify right))
+    )
+    (property "Footprint" "Xenir:BNC" (id 2) (at 201.93 101.6 0)
+      (effects (font (size 1.27 1.27)) hide)
+    )
+    (property "Datasheet" "" (id 3) (at 201.93 101.6 0)
+      (effects (font (size 1.27 1.27)) hide)
+    )
+    (pin "GND")
+    (pin "S")
   )
   (symbol (lib_id "Diode:1N4148W") (at 168.91 130.81 0) (unit 1)
@@
     (pin "2")
   )
+  (symbol (lib_id "power:GND") (at 201.93 110.49 0) (unit 1)
+    (in_bom yes) (on_board yes) (fields_autoplaced)
+    (property "Reference" "#PWR0104" (id 0) (at 201.93 116.84 0)
+      (effects (font (size 1.27 1.27)) hide)
+    )
+    (property "Value" "GND" (id 1) (at 201.93 115.57 0))
+    (property "Footprint" "" (id 2) (at 201.93 110.49 0)
+      (effects (font (size 1.27 1.27)) hide)
+    )
+    (property "Datasheet" "" (id 3) (at 201.93 110.49 0)
+      (effects (font (size 1.27 1.27)) hide)
+    )
+    (pin "1")
+  )
 )
