File: RF-SWITCH.kicad_sch (KiCad schematic)
At the start: 5 parts, among them J1 BNC, K1 G6S-2, K2 G6S-2

Commit message: gg
Parts:
- removed J1: BNC, Xenir:BNC, symbol Xenir:BNC
Connections:
- net Antenna: now reaches K2.4, K2.9
Changed lines of the file:
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@@
     (effects (font (size 1.27 1.27)) (justify right))
   )
-  (symbol (lib_id "Xenir:BNC") (at 201.93 105.41 0) (mirror y) (unit 1)
-    (in_bom yes) (on_board yes) (fields_autoplaced)
-    (property "Reference" "J1" (id 0) (at 205.74 104.1399 0)
-      (effects (font (size 1.27 1.27)) (justify right))
-    )
-    (property "Value" "BNC" (id 1) (at 205.74 106.6799 0)
-      (effects (font (size 1.27 1.27)) (justify right))
-    )
-    (property "Footprint" "Xenir:BNC" (id 2) (at 201.93 101.6 0)
-      (effects (font (size 1.27 1.27)) hide)
-    )
-    (property "Datasheet" "" (id 3) (at 201.93 101.6 0)
-      (effects (font (size 1.27 1.27)) hide)
-    )
-    (pin "GND")
-    (pin "S")
+  (hierarchical_label "Antenna" (shape bidirectional) (at 196.85 105.41 0)
+    (effects (font (size 1.27 1.27)) (justify left))
   )
   (symbol (lib_id "Diode:1N4148W") (at 168.91 130.81 0) (unit 1)
@@
     (pin "2")
   )
-  (symbol (lib_id "power:GND") (at 201.93 110.49 0) (unit 1)
-    (in_bom yes) (on_board yes) (fields_autoplaced)
-    (property "Reference" "#PWR0104" (id 0) (at 201.93 116.84 0)
-      (effects (font (size 1.27 1.27)) hide)
-    )
-    (property "Value" "GND" (id 1) (at 201.93 115.57 0))
-    (property "Footprint" "" (id 2) (at 201.93 110.49 0)
-      (effects (font (size 1.27 1.27)) hide)
-    )
-    (property "Datasheet" "" (id 3) (at 201.93 110.49 0)
-      (effects (font (size 1.27 1.27)) hide)
-    )
-    (pin "1")
-  )
 )

Commit message: added relay fet
Parts:
- added Q1: AO3400A, Package_TO_SOT_SMD:SOT-23, symbol Transistor_FET:AO3400A
- added R31: 1k, Resistor_SMD:R_0805_2012Metric, symbol xenir:Resistor
Connections:
- net T/R: now also R31.1
- net +12V: now reaches D2.1 (K), K2.1
- net +12V: now also D1.1 (K), K1.1
- net RELAY-ON: now reaches D2.2 (A), K2.12
- net RELAY-ON: now also D1.2 (A), K1.12, Q1.3 (D)
- new net: Q1.1 (G), R31.2
- new net GND: Q1.2 (S)
Changed lines of the file:
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@@
 (kicad_sch (version 20211123) (generator eeschema)
   (paper "A4")
+  (junction (at 99.06 120.65) (diameter 0) (color 0 0 0 0)
+  )
   (junction (at 180.34 105.41) (diameter 0) (color 0 0 0 0)
   )
   (junction (at 151.13 99.06) (diameter 0) (color 0 0 0 0)
   )
+  (junction (at 161.29 120.65) (diameter 0) (color 0 0 0 0)
+  )
+  (junction (at 176.53 120.65) (diameter 0) (color 0 0 0 0)
+  )
+  (junction (at 114.3 120.65) (diameter 0) (color 0 0 0 0)
+  )
   (junction (at 153.67 110.49) (diameter 0) (color 0 0 0 0)
   )
+  (wire (pts (xy 176.53 120.65) (xy 182.88 120.65))
+    (stroke (width 0) (type default) (color 0 0 0 0))
+  )
   (wire (pts (xy 161.29 113.03) (xy 153.67 113.03))
     (stroke (width 0) (type default) (color 0 0 0 0))
@@
     (stroke (width 0) (type default) (color 0 0 0 0))
   )
+  (wire (pts (xy 146.05 72.39) (xy 148.59 72.39))
+    (stroke (width 0) (type default) (color 0 0 0 0))
+  )
   (wire (pts (xy 146.05 99.06) (xy 151.13 99.06))
     (stroke (width 0) (type default) (color 0 0 0 0))
@@
     (stroke (width 0) (type default) (color 0 0 0 0))
   )
+  (wire (pts (xy 153.67 120.65) (xy 161.29 120.65))
+    (stroke (width 0) (type default) (color 0 0 0 0))
+  )
+  (wire (pts (xy 91.44 120.65) (xy 99.06 120.65))
+    (stroke (width 0) (type default) (color 0 0 0 0))
+  )
   (wire (pts (xy 180.34 110.49) (xy 180.34 105.41))
     (stroke (width 0) (type default) (color 0 0 0 0))
@@
     (stroke (width 0) (type default) (color 0 0 0 0))
   )
+  (wire (pts (xy 114.3 120.65) (xy 120.65 120.65))
+    (stroke (width 0) (type default) (color 0 0 0 0))
+  )
   (wire (pts (xy 161.29 120.65) (xy 161.29 130.81))
     (stroke (width 0) (type default) (color 0 0 0 0))
@@
     (stroke (width 0) (type default) (color 0 0 0 0))
   )
+  (wire (pts (xy 156.21 63.5) (xy 156.21 67.31))
+    (stroke (width 0) (type default) (color 0 0 0 0))
+  )
   (wire (pts (xy 176.53 110.49) (xy 180.34 110.49))
     (stroke (width 0) (type default) (color 0 0 0 0))
@@
     (stroke (width 0) (type default) (color 0 0 0 0))
   )
+  (wire (pts (xy 133.35 72.39) (xy 135.89 72.39))
+    (stroke (width 0) (type default) (color 0 0 0 0))
+  )
   (wire (pts (xy 151.13 97.79) (xy 161.29 97.79))
     (stroke (width 0) (type default) (color 0 0 0 0))
@@
     (stroke (width 0) (type default) (color 0 0 0 0))
   )
+  (global_label "RELAY-ON" (shape input) (at 120.65 120.65 0) (fields_autoplaced)
+    (effects (font (size 1.27 1.27)) (justify left))
+    (property "Intersheet References" "${INTERSHEET_REFS}" (id 0) (at 132.9207 120.5706 0)
+      (effects (font (size 1.27 1.27)) (justify left) hide)
+    )
+  )
+  (global_label "RELAY-ON" (shape input) (at 156.21 63.5 90) (fields_autoplaced)
+    (effects (font (size 1.27 1.27)) (justify left))
+    (property "Intersheet References" "${INTERSHEET_REFS}" (id 0) (at 156.1306 51.2293 90)
+      (effects (font (size 1.27 1.27)) (justify left) hide)
+    )
+  )
+  (global_label "RELAY-ON" (shape input) (at 182.88 120.65 0) (fields_autoplaced)
+    (effects (font (size 1.27 1.27)) (justify left))
+    (property "Intersheet References" "${INTERSHEET_REFS}" (id 0) (at 195.1507 120.5706 0)
+      (effects (font (size 1.27 1.27)) (justify left) hide)
+    )
+  )
   (hierarchical_label "BPF-OUT" (shape input) (at 114.3 110.49 0)
     (effects (font (size 1.27 1.27)) (justify left))
@@
     (effects (font (size 1.27 1.27)) (justify left))
   )
-  (hierarchical_label "T{slash}R" (shape input) (at 134.62 82.55 0)
-    (effects (font (size 1.27 1.27)) (justify left))
+  (hierarchical_label "T{slash}R" (shape input) (at 133.35 72.39 180)
+    (effects (font (size 1.27 1.27)) (justify right))
   )
   (hierarchical_label "PA-IN" (shape output) (at 99.06 107.95 180)
@@
   (hierarchical_label "Antenna" (shape bidirectional) (at 196.85 105.41 0)
     (effects (font (size 1.27 1.27)) (justify left))
+  )
+  (symbol (lib_id "power:+12V") (at 91.44 120.65 0) (unit 1)
+    (in_bom yes) (on_board yes)
+    (property "Reference" "#PWR0157" (id 0) (at 91.44 124.46 0)
+      (effects (font (size 1.27 1.27)) hide)
+    )
+    (property "Value" "+12V" (id 1) (at 87.63 119.38 0))
+    (property "Footprint" "" (id 2) (at 91.44 120.65 0)
+      (effects (font (size 1.27 1.27)) hide)
+    )
+    (property "Datasheet" "" (id 3) (at 91.44 120.65 0)
+      (effects (font (size 1.27 1.27)) hide)
+    )
+    (pin "1")
+  )
+  (symbol (lib_id "power:GND") (at 156.21 77.47 0) (unit 1)
+    (in_bom yes) (on_board yes) (fields_autoplaced)
+    (property "Reference" "#PWR0158" (id 0) (at 156.21 83.82 0)
+      (effects (font (size 1.27 1.27)) hide)
+    )
+    (property "Value" "GND" (id 1) (at 156.21 82.55 0))
+    (property "Footprint" "" (id 2) (at 156.21 77.47 0)
+      (effects (font (size 1.27 1.27)) hide)
+    )
+    (property "Datasheet" "" (id 3) (at 156.21 77.47 0)
+      (effects (font (size 1.27 1.27)) hide)
+    )
+    (pin "1")
   )
   (symbol (lib_id "Diode:1N4148W") (at 168.91 130.81 0) (unit 1)
@@
     (pin "9")
   )
+  (symbol (lib_id "xenir:Resistor") (at 140.97 72.39 0) (unit 1)
+    (in_bom yes) (on_board yes) (fields_autoplaced)
+    (property "Reference" "R31" (id 0) (at 140.97 67.31 0)
+      (effects (font (size 0.7112 0.7112)))
+    )
+    (property "Value" "1k" (id 1) (at 140.97 69.85 0)
+      (effects (font (size 0.7112 0.7112)))
+    )
+    (property "Footprint" "Resistor_SMD:R_0805_2012Metric" (id 2) (at 140.97 74.93 0)
+      (effects (font (size 1.27 1.27)) hide)
+    )
+    (property "Datasheet" "" (id 3) (at 140.97 74.93 0)
+      (effects (font (size 1.27 1.27)) hide)
+    )
+    (pin "1")
+    (pin "2")
+  )
+  (symbol (lib_id "power:+12V") (at 153.67 120.65 0) (unit 1)
+    (in_bom yes) (on_board yes)
+    (property "Reference" "#PWR0159" (id 0) (at 153.67 124.46 0)
+      (effects (font (size 1.27 1.27)) hide)
+    )
+    (property "Value" "+12V" (id 1) (at 149.86 119.38 0))
+    (property "Footprint" "" (id 2) (at 153.67 120.65 0)
+      (effects (font (size 1.27 1.27)) hide)
+    )
+    (property "Datasheet" "" (id 3) (at 153.67 120.65 0)
+      (effects (font (size 1.27 1.27)) hide)
+    )
+    (pin "1")
+  )
   (symbol (lib_id "Diode:1N4148W") (at 106.68 130.81 0) (unit 1)
     (in_bom yes) (on_board yes)
@@
     (pin "2")
   )
+  (symbol (lib_id "Transistor_FET:AO3400A") (at 153.67 72.39 0) (unit 1)
+    (in_bom yes) (on_board yes) (fields_autoplaced)
+    (property "Reference" "Q1" (id 0) (at 160.02 71.1199 0)
+      (effects (font (size 1.27 1.27)) (justify left))
+    )
+    (property "Value" "AO3400A" (id 1) (at 160.02 73.6599 0)
+      (effects (font (size 1.27 1.27)) (justify left))
+    )
+    (property "Footprint" "Package_TO_SOT_SMD:SOT-23" (id 2) (at 158.75 74.295 0)
+      (effects (font (size 1.27 1.27) italic) (justify left) hide)
+    )
+    (property "Datasheet" "http://www.aosmd.com/pdfs/datasheet/AO3400A.pdf" (id 3) (at 153.67 72.39 0)
+      (effects (font (size 1.27 1.27)) (justify left) hide)
+    )
+    (pin "1")
+    (pin "2")
+    (pin "3")
+  )
 )
