File: taylor-detector.kicad_sch (KiCad schematic)
At the start: 0 parts

Commit message: lots of updates
Parts:
- added C10, C9: .1uF, Capacitor_SMD:C_1206_3216Metric, symbol Xenir:Capacitor
- added C11, C12, C13, C14: 470nF, Capacitor_SMD:C_1206_3216Metric, symbol Xenir:Capacitor
- added C15, C16: 1nF, Capacitor_SMD:C_1206_3216Metric, symbol Xenir:Capacitor
- added R1, R2, R3, R4: 100, Resistor_SMD:R_0805_2012Metric, symbol Xenir:Resistor
- added R5, R6: 10k, Resistor_SMD:R_0805_2012Metric, symbol Xenir:Resistor
- added T3: T50_SPLITTER, Xenir:T50 Trifilar, symbol Xenir:T50_SPLITTER
- added U1: FST3253, Xenir:SO16, symbol Xenir:FST3253
- added U2: LM4562, Xenir:SO08, symbol Amplifier_Operational:LM358
Connections:
- net 0-Degree: now also U1.2 (S1)
- net 90-Degree: now also U1.14 (S0)
- net Detector-In: now also T3.C1B
- new net: C15.1, R1.2, R5.1, U2.2 (-)
- new net: R4.2, U2.5 (+)
- new net: T3.C2B, U1.7 (1A)
- new net: T3.C3A, U1.9 (2A)
- new net: R3.2, U2.3 (+)
- new net: C16.1, R2.2, R6.1, U2.6 (-)
- new net +12V: C10.2, U2.8 (V+)
- new net +2V5: T3.C2A, T3.C3B
- new net +5V: C9.2, U1.16 (VCC)
- new net Detector-0: C11.2, C12.2, C13.2, C14.2, R1.1, R2.1, R3.1, R4.1, U1.10 (2B1), U1.11 (2B2), U1.12 (2B3), U1.13 (2B4), U1.3 (1B4), U1.4 (1B3), U1.5 (1B2), U1.6 (1B1)
- new net Detector-I: C15.2, R5.2, U2.1
- new net Detector-Q: C16.2, R6.2, U2.7
- new net GND: C10.1, C11.1, C12.1, C13.1, C14.1, C9.1, T3.C1A, U1.1 (OE1), U1.15 (OE2), U1.8 (GND), U2.4 (V-)
