File: taylor-detector.kicad_sch (KiCad schematic)
At the start: 17 parts, among them T3 T50_SPLITTER, U1 FST3253, U2 LM4562

Commit message: fixed decoder
Connections:
- net Detector-0: no longer C12.2, C13.2, C14.2, R2.1, R3.1, R4.1, U1.11 (2B2), U1.12 (2B3), U1.13 (2B4), U1.4 (1B3), U1.5 (1B2), U1.6 (1B1)
- new net Detector-180: C13.2, R3.1, U1.13 (2B4), U1.6 (1B1)
- new net Detector-270: C14.2, R4.1, U1.12 (2B3), U1.5 (1B2)
- new net Detector-90: C12.2, R2.1, U1.11 (2B2), U1.4 (1B3)
Changed lines of the file:
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@@
   (junction (at 140.97 106.68) (diameter 0) (color 0 0 0 0)
-  )
-  (junction (at 104.14 106.68) (diameter 0) (color 0 0 0 0)
-  )
-  (junction (at 104.14 104.14) (diameter 0) (color 0 0 0 0)
   )
   (junction (at 143.51 101.6) (diameter 0) (color 0 0 0 0)
@@
   )
   (junction (at 220.98 106.68) (diameter 0) (color 0 0 0 0)
-  )
-  (junction (at 104.14 109.22) (diameter 0) (color 0 0 0 0)
   )
   (junction (at 104.14 96.52) (diameter 0) (color 0 0 0 0)
@@
     (stroke (width 0) (type default) (color 0 0 0 0))
   )
-  (wire (pts (xy 104.14 120.65) (xy 104.14 109.22))
+  (wire (pts (xy 104.14 101.6) (xy 104.14 120.65))
     (stroke (width 0) (type default) (color 0 0 0 0))
   )
   (wire (pts (xy 101.6 123.19) (xy 101.6 106.68))
-    (stroke (width 0) (type default) (color 0 0 0 0))
-  )
-  (wire (pts (xy 104.14 104.14) (xy 104.14 101.6))
     (stroke (width 0) (type default) (color 0 0 0 0))
   )
@@
     (stroke (width 0) (type default) (color 0 0 0 0))
   )
-  (wire (pts (xy 104.14 106.68) (xy 104.14 104.14))
-    (stroke (width 0) (type default) (color 0 0 0 0))
-  )
   (wire (pts (xy 220.98 69.85) (xy 220.98 74.93))
     (stroke (width 0) (type default) (color 0 0 0 0))
@@
     (stroke (width 0) (type default) (color 0 0 0 0))
   )
-  (wire (pts (xy 104.14 109.22) (xy 104.14 106.68))
-    (stroke (width 0) (type default) (color 0 0 0 0))
-  )

Commit message: updated opamp voltage - thanks andre!
Connections:
- net +12V is gone; now on net +5V: C10.2, U2.8 (V+)
Changed lines of the file:
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@@
     (pin "2")
-  )
-  (symbol (lib_id "power:+12V") (at 234.95 36.83 0) (unit 1)
-    (in_bom yes) (on_board yes) (fields_autoplaced)
-    (property "Reference" "#PWR0111" (id 0) (at 234.95 40.64 0)
-      (effects (font (size 1.27 1.27)) hide)
-    )
-    (property "Value" "+12V" (id 1) (at 234.95 31.75 0))
-    (property "Footprint" "" (id 2) (at 234.95 36.83 0)
-      (effects (font (size 1.27 1.27)) hide)
-    )
-    (property "Datasheet" "" (id 3) (at 234.95 36.83 0)
-      (effects (font (size 1.27 1.27)) hide)
-    )
-    (pin "1")
   )
   (symbol (lib_id "Xenir:Resistor") (at 205.74 81.28 0) (unit 1)
@@
       (effects (font (size 1.27 1.27)) hide)
     )
+    (pin "1")
+  )
+  (symbol (lib_id "power:+5V") (at 234.95 36.83 0) (unit 1)
+    (in_bom yes) (on_board yes) (fields_autoplaced)
+    (property "Reference" "#PWR0111" (id 0) (at 234.95 40.64 0)
+      (effects (font (size 1.27 1.27)) hide)
+    )
+    (property "Value" "+5V" (id 1) (at 234.95 31.75 0))
+    (property "Footprint" "" (id 2) (at 234.95 36.83 0)
+      (effects (font (size 1.27 1.27)) hide)
+    )
+    (property "Datasheet" "" (id 3) (at 234.95 36.83 0)
+      (effects (font (size 1.27 1.27)) hide)
+    )

Commit message: gg
Connections:
- net Detector-I: now also C16.2, R6.2, U2.7; no longer C15.2, R5.2, U2.1
- net Detector-Q: now also C15.2, R5.2, U2.1; no longer C16.2, R6.2, U2.7
Changed lines of the file:
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@@
 (kicad_sch (version 20211123) (generator eeschema)
   (paper "A4")
+  (junction (at 142.24 104.14) (diameter 0) (color 0 0 0 0)
+  )
+  (junction (at 140.97 106.68) (diameter 0) (color 0 0 0 0)
+  )
+  (junction (at 143.51 101.6) (diameter 0) (color 0 0 0 0)
+  )
+  (junction (at 71.12 85.09) (diameter 0) (color 0 0 0 0)
+  )
+  (junction (at 234.95 39.37) (diameter 0) (color 0 0 0 0)
+  )
+  (junction (at 242.57 74.93) (diameter 0) (color 0 0 0 0)
+  )
+  (junction (at 242.57 83.82) (diameter 0) (color 0 0 0 0)
+  )
+  (junction (at 220.98 100.33) (diameter 0) (color 0 0 0 0)
+  )
+  (junction (at 121.92 66.04) (diameter 0) (color 0 0 0 0)
+  )
+  (junction (at 220.98 74.93) (diameter 0) (color 0 0 0 0)
+  )
+  (junction (at 139.7 109.22) (diameter 0) (color 0 0 0 0)
+  )
+  (junction (at 220.98 81.28) (diameter 0) (color 0 0 0 0)
+  )
   (junction (at 243.84 109.22) (diameter 0) (color 0 0 0 0)
   )
-  (junction (at 142.24 104.14) (diameter 0) (color 0 0 0 0)
-  )
-  (junction (at 140.97 106.68) (diameter 0) (color 0 0 0 0)
-  )
-  (junction (at 143.51 101.6) (diameter 0) (color 0 0 0 0)
-  )
-  (junction (at 71.12 85.09) (diameter 0) (color 0 0 0 0)
-  )
-  (junction (at 234.95 39.37) (diameter 0) (color 0 0 0 0)
-  )
-  (junction (at 242.57 74.93) (diameter 0) (color 0 0 0 0)
-  )
-  (junction (at 242.57 83.82) (diameter 0) (color 0 0 0 0)
-  )
-  (junction (at 220.98 100.33) (diameter 0) (color 0 0 0 0)
-  )
-  (junction (at 121.92 66.04) (diameter 0) (color 0 0 0 0)
-  )
-  (junction (at 220.98 74.93) (diameter 0) (color 0 0 0 0)
-  )
-  (junction (at 139.7 109.22) (diameter 0) (color 0 0 0 0)
-  )
-  (junction (at 220.98 81.28) (diameter 0) (color 0 0 0 0)
-  )
   (junction (at 243.84 100.33) (diameter 0) (color 0 0 0 0)
   )
@@
     (stroke (width 0) (type default) (color 0 0 0 0))
   )
+  (wire (pts (xy 243.84 109.22) (xy 250.19 109.22))
+    (stroke (width 0) (type default) (color 0 0 0 0))
+  )
   (wire (pts (xy 143.51 124.46) (xy 100.33 124.46))
     (stroke (width 0) (type default) (color 0 0 0 0))
@@
     (stroke (width 0) (type default) (color 0 0 0 0))
   )
-  (wire (pts (xy 252.73 83.82) (xy 242.57 83.82))
-    (stroke (width 0) (type default) (color 0 0 0 0))
-  )
   (wire (pts (xy 71.12 82.55) (xy 71.12 85.09))
     (stroke (width 0) (type default) (color 0 0 0 0))
@@
     (stroke (width 0) (type default) (color 0 0 0 0))
   )
-  (wire (pts (xy 252.73 109.22) (xy 243.84 109.22))
-    (stroke (width 0) (type default) (color 0 0 0 0))
-  )
   (wire (pts (xy 227.33 69.85) (xy 220.98 69.85))
     (stroke (width 0) (type default) (color 0 0 0 0))
@@
     (stroke (width 0) (type default) (color 0 0 0 0))
   )
+  (wire (pts (xy 242.57 83.82) (xy 250.19 83.82))
+    (stroke (width 0) (type default) (color 0 0 0 0))
+  )
   (wire (pts (xy 100.33 124.46) (xy 100.33 109.22))
     (stroke (width 0) (type default) (color 0 0 0 0))
@@
     )
   )
-  (hierarchical_label "Detector-Q" (shape output) (at 252.73 109.22 0)
+  (hierarchical_label "Detector-Q" (shape output) (at 250.19 83.82 0)
     (effects (font (size 1.27 1.27)) (justify left))
   )
@@
     (effects (font (size 1.27 1.27)) (justify left))
   )
-  (hierarchical_label "Detector-I" (shape output) (at 252.73 83.82 0)
-    (effects (font (size 1.27 1.27)) (justify left))
-  )
+  (hierarchical_label "Detector-I" (shape output) (at 250.19 109.22 0)
+    (effects (font (size 1.27 1.27)) (justify left))
+  )

Commit message: added more decoupling caps
Parts:
- added C56: .1uF, Capacitor_SMD:C_1206_3216Metric, symbol Xenir:Capacitor
Connections:
- net +2V5: now also C56.2
- net GND: now also C56.1
Changed lines of the file:
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@@
   (junction (at 142.24 104.14) (diameter 0) (color 0 0 0 0)
   )
+  (junction (at 73.66 85.09) (diameter 0) (color 0 0 0 0)
+  )
   (junction (at 140.97 106.68) (diameter 0) (color 0 0 0 0)
   )
@@
     (stroke (width 0) (type default) (color 0 0 0 0))
   )
+  (wire (pts (xy 73.66 85.09) (xy 76.2 85.09))
+    (stroke (width 0) (type default) (color 0 0 0 0))
+  )
   (wire (pts (xy 236.22 100.33) (xy 243.84 100.33))
     (stroke (width 0) (type default) (color 0 0 0 0))
@@
     (stroke (width 0) (type default) (color 0 0 0 0))
   )
-  (wire (pts (xy 71.12 85.09) (xy 76.2 85.09))
+  (wire (pts (xy 71.12 85.09) (xy 73.66 85.09))
     (stroke (width 0) (type default) (color 0 0 0 0))
   )
@@
     (pin "1")
   )
+  (symbol (lib_id "Xenir:Capacitor") (at 73.66 88.9 90) (unit 1)
+    (in_bom yes) (on_board yes)
+    (property "Reference" "C56" (id 0) (at 71.12 86.36 90)
+      (effects (font (size 0.7112 0.7112)) (justify right))
+    )
+    (property "Value" ".1uF" (id 1) (at 74.93 86.36 90)
+      (effects (font (size 0.7112 0.7112)) (justify right))
+    )
+    (property "Footprint" "Capacitor_SMD:C_1206_3216Metric" (id 2) (at 77.47 88.9 0)
+      (effects (font (size 1.27 1.27)) hide)
+    )
+    (property "Datasheet" "" (id 3) (at 77.47 88.9 0)
+      (effects (font (size 1.27 1.27)) hide)
+    )
+    (pin "1")
+    (pin "2")
+  )
   (symbol (lib_id "Xenir:Capacitor") (at 196.85 85.09 90) (unit 1)
     (in_bom yes) (on_board yes)
@@
     (pin "2")
   )
+  (symbol (lib_id "power:GND") (at 73.66 92.71 0) (unit 1)
+    (in_bom yes) (on_board yes)
+    (property "Reference" "#PWR0216" (id 0) (at 73.66 99.06 0)
+      (effects (font (size 1.27 1.27)) hide)
+    )
+    (property "Value" "GND" (id 1) (at 76.2 92.71 0))
+    (property "Footprint" "" (id 2) (at 73.66 92.71 0)
+      (effects (font (size 1.27 1.27)) hide)
+    )
+    (property "Datasheet" "" (id 3) (at 73.66 92.71 0)
+      (effects (font (size 1.27 1.27)) hide)
+    )
+    (pin "1")
+  )
   (symbol (lib_id "Xenir:Capacitor") (at 224.79 49.53 90) (unit 1)
