File: SDR-Transceiver.kicad_sch (KiCad schematic)
At the start: 0 parts

Commit message: lots of updates
Other:
- added sheet Audio-Switch (audio-switch.kicad_sch)
- sheet Tayloe-Detector ports: added Detector-I, Detector-Q; removed none
- sheet Tayloe-Encoder ports: added Encoder-I, Encoder-Q; removed none

Commit message: gg
Other:
- added sheet DSP (DSP.kicad_sch)
Changed lines of the file:
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@@
+    )
+  )
+  (sheet (at 40.64 81.28) (size 22.86 49.53) (fields_autoplaced)
+    (stroke (width 0.1524) (type solid) (color 0 0 0 0))
+    (fill (color 0 0 0 0.0000))
+    (property "Sheet name" "DSP" (id 0) (at 40.64 80.5684 0)
+      (effects (font (size 1.27 1.27)) (justify left bottom))
+    )
+    (property "Sheet file" "DSP.kicad_sch" (id 1) (at 40.64 131.3946 0)
+      (effects (font (size 1.27 1.27)) (justify left top) hide)
+    )
+    (pin "DSP-OUTL" output (at 63.5 118.11 0)
+      (effects (font (size 1.27 1.27)) (justify right))
+    )
+    (pin "DSP-OUTR" output (at 63.5 121.92 0)
+      (effects (font (size 1.27 1.27)) (justify right))
+    )
+    (pin "DSP-INR" input (at 63.5 92.71 0)
+      (effects (font (size 1.27 1.27)) (justify right))
+    )
+    (pin "DSP-INL" input (at 63.5 88.9 0)
+      (effects (font (size 1.27 1.27)) (justify right))
     )
   )
@@
     (path "/5722f6fa-2bcc-4202-8947-4321e1b76cf2" (page "8"))
     (path "/38ec5edb-504e-48c9-aada-546359fe144d" (page "9"))
+    (path "/85cf5236-19af-47bd-b6dc-799e0e38ef1d" (page "10"))
   )
   (symbol_instances
@@
       (reference "#PWR0137") (unit 1) (value "+2V5") (footprint "")
     )
+    (path "/85cf5236-19af-47bd-b6dc-799e0e38ef1d/53286237-6086-46a9-9434-25d6f0672810"
+      (reference "#PWR0138") (unit 1) (value "GND") (footprint "")
+    )
+    (path "/85cf5236-19af-47bd-b6dc-799e0e38ef1d/1f97ee07-4b41-4a0b-a2a9-d374b2038851"
+      (reference "#PWR0139") (unit 1) (value "GND") (footprint "")
+    )
     (path "/3c85d954-82ab-4b0c-952d-ee98ece6c954/dd12f21a-378a-48c3-99c8-be75492147f4"
       (reference "C1") (unit 1) (value "270pF") (footprint "Capacitor_SMD:C_1206_3216Metric")
@@
       (reference "C23") (unit 1) (value ".1uF") (footprint "Capacitor_SMD:C_1206_3216Metric")
     )
+    (path "/85cf5236-19af-47bd-b6dc-799e0e38ef1d/fc04a4e4-1dba-4730-a534-63e52692b1d5"
+      (reference "C24") (unit 1) (value "22uF") (footprint "Capacitor_SMD:C_1206_3216Metric")
+    )
+    (path "/85cf5236-19af-47bd-b6dc-799e0e38ef1d/14ef25cd-943e-4963-b96c-01a2a554ca76"
+      (reference "C25") (unit 1) (value "1uF") (footprint "Capacitor_SMD:C_1206_3216Metric")
+    )
+    (path "/85cf5236-19af-47bd-b6dc-799e0e38ef1d/6a34666e-bc5a-495c-8fdd-3d7ede3a07ba"
+      (reference "C26") (unit 1) (value "22uF") (footprint "Capacitor_SMD:C_1206_3216Metric")
+    )
+    (path "/85cf5236-19af-47bd-b6dc-799e0e38ef1d/57ec3002-cebc-4d33-997d-28a28aea6d28"
+      (reference "C27") (unit 1) (value "1uF") (footprint "Capacitor_SMD:C_1206_3216Metric")
+    )
+    (path "/85cf5236-19af-47bd-b6dc-799e0e38ef1d/ba66c4ae-62cc-413e-af5c-8776b1e6b95b"
+      (reference "C28") (unit 1) (value "1uF") (footprint "Capacitor_SMD:C_1206_3216Metric")
+    )
+    (path "/85cf5236-19af-47bd-b6dc-799e0e38ef1d/7abe07da-f11a-4f67-8752-13f40d07bb5a"
+      (reference "C29") (unit 1) (value "1uF") (footprint "Capacitor_SMD:C_1206_3216Metric")
+    )
     (path "/ccad2f77-41ee-4855-83bb-0372e01592b3/dd78a2a3-3b94-4c56-a19a-5c168aa90dff"
       (reference "D1") (unit 1) (value "1N4148W") (footprint "Diode_SMD:D_SOD-123")
@@
       (reference "R20") (unit 1) (value "50") (footprint "Resistor_SMD:R_0805_2012Metric")
     )
+    (path "/85cf5236-19af-47bd-b6dc-799e0e38ef1d/d72aa15a-233f-4946-8730-8d68e7c9346c"
+      (reference "R21") (unit 1) (value "330") (footprint "Resistor_SMD:R_0805_2012Metric")
+    )
+    (path "/85cf5236-19af-47bd-b6dc-799e0e38ef1d/24826017-976d-4a17-b619-71be51ca0009"
+      (reference "R22") (unit 1) (value "330") (footprint "Resistor_SMD:R_0805_2012Metric")
+    )
     (path "/4b1ef805-7fd0-4a4a-b5da-5feeaa035c65/dbc98a07-c075-4ec8-822f-59596956d619"
       (reference "T1") (unit 1) (value "T37-6 5:25") (footprint "Xenir:T37 Transformer")
@@
       (reference "U5") (unit 3) (value "LM4562") (footprint "Xenir:SO08")
     )
+    (path "/85cf5236-19af-47bd-b6dc-799e0e38ef1d/bfc5e1cf-d28e-44f7-b8ad-5f46427e5b43"
+      (reference "U6") (unit 1) (value "ESP32-A1S") (footprint "Xenir:ESP32-A1S")
+    )
     (path "/4b1ef805-7fd0-4a4a-b5da-5feeaa035c65/a3e1d27e-f1e5-419b-8a71-6427134bb505"

Commit message: more updates
Other:
- sheet DSP ports: added SCL, SDA; removed none
- sheet Local-Oscillator ports: added SCL, SDA; removed none

Commit message: gg
Other:
- sheet Audio-Switch ports: added T/R; removed none
- sheet DSP ports: added T/R; removed none
Changed lines of the file:
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@@
+    (stroke (width 0) (type default) (color 0 0 0 0))
+  )
+  (wire (pts (xy 63.5 85.09) (xy 92.71 85.09))
     (stroke (width 0) (type default) (color 0 0 0 0))
   )
@@
     )
   )
+  (global_label "T{slash}R" (shape input) (at 67.31 85.09 90) (fields_autoplaced)
+    (effects (font (size 1.27 1.27)) (justify left))
+    (property "Intersheet References" "${INTERSHEET_REFS}" (id 0) (at 67.2306 79.1088 90)
+      (effects (font (size 1.27 1.27)) (justify left) hide)
+    )
+  )
+  (global_label "T{slash}R" (shape input) (at 191.77 88.9 180) (fields_autoplaced)
+    (effects (font (size 1.27 1.27)) (justify right))
+    (property "Intersheet References" "${INTERSHEET_REFS}" (id 0) (at 185.7888 88.9794 0)
+      (effects (font (size 1.27 1.27)) (justify right) hide)
+    )
+  )
   (global_label "LO-90" (shape input) (at 138.43 95.25 180) (fields_autoplaced)
     (effects (font (size 1.27 1.27)) (justify right))
@@
     )
   )
+  (global_label "T{slash}R" (shape input) (at 229.87 91.44 180) (fields_autoplaced)
+    (effects (font (size 1.27 1.27)) (justify right))
+    (property "Intersheet References" "${INTERSHEET_REFS}" (id 0) (at 223.8888 91.5194 0)
+      (effects (font (size 1.27 1.27)) (justify right) hide)
+    )
+  )
   (global_label "LO-0" (shape input) (at 138.43 110.49 180) (fields_autoplaced)
     (effects (font (size 1.27 1.27)) (justify right))
@@
       (effects (font (size 1.27 1.27)) (justify left))
     )
+    (pin "T{slash}R" input (at 92.71 85.09 180)
+      (effects (font (size 1.27 1.27)) (justify left))
+    )
   )
   (sheet (at 229.87 104.14) (size 20.32 8.89) (fields_autoplaced)
@@
       (effects (font (size 1.27 1.27)) (justify left))
     )
-  )
+    (pin "T{slash}R" output (at 63.5 85.09 0)
+      (effects (font (size 1.27 1.27)) (justify right))
+    )
+  )

Commit message: added mic amp
Other:
- added sheet AUDIO-AMP (audio-amp.kicad_sch)
- added sheet MIC (mic.kicad_sch)
Changed lines of the file:
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@@
   (junction (at 209.55 86.36) (diameter 0) (color 0 0 0 0)
   )
+  (junction (at 121.92 85.09) (diameter 0) (color 0 0 0 0)
+  )
   (wire (pts (xy 256.54 110.49) (xy 250.19 110.49))
     (stroke (width 0) (type default) (color 0 0 0 0))
   )
+  (wire (pts (xy 138.43 148.59) (xy 121.92 148.59))
+    (stroke (width 0) (type default) (color 0 0 0 0))
+  )
+  (wire (pts (xy 121.92 85.09) (xy 121.92 87.63))
+    (stroke (width 0) (type default) (color 0 0 0 0))
+  )
   (wire (pts (xy 34.29 60.96) (xy 34.29 106.68))
     (stroke (width 0) (type default) (color 0 0 0 0))
@@
     (stroke (width 0) (type default) (color 0 0 0 0))
   )
+  (wire (pts (xy 138.43 59.69) (xy 121.92 59.69))
+    (stroke (width 0) (type default) (color 0 0 0 0))
+  )
   (wire (pts (xy 125.73 78.74) (xy 125.73 92.71))
     (stroke (width 0) (type default) (color 0 0 0 0))
@@
     (stroke (width 0) (type default) (color 0 0 0 0))
   )
+  (wire (pts (xy 121.92 87.63) (xy 115.57 87.63))
+    (stroke (width 0) (type default) (color 0 0 0 0))
+  )
   (wire (pts (xy 128.27 114.3) (xy 128.27 123.19))
     (stroke (width 0) (type default) (color 0 0 0 0))
@@
     (stroke (width 0) (type default) (color 0 0 0 0))
   )
+  (wire (pts (xy 121.92 59.69) (xy 121.92 85.09))
+    (stroke (width 0) (type default) (color 0 0 0 0))
+  )
   (wire (pts (xy 63.5 92.71) (xy 92.71 92.71))
     (stroke (width 0) (type default) (color 0 0 0 0))
@@
     (stroke (width 0) (type default) (color 0 0 0 0))
   )
+  (wire (pts (xy 121.92 148.59) (xy 121.92 124.46))
+    (stroke (width 0) (type default) (color 0 0 0 0))
+  )
   (wire (pts (xy 115.57 114.3) (xy 128.27 114.3))
     (stroke (width 0) (type default) (color 0 0 0 0))
   )
   (wire (pts (xy 128.27 82.55) (xy 128.27 95.25))
+    (stroke (width 0) (type default) (color 0 0 0 0))
+  )
+  (wire (pts (xy 115.57 85.09) (xy 121.92 85.09))
+    (stroke (width 0) (type default) (color 0 0 0 0))
+  )
+  (wire (pts (xy 121.92 124.46) (xy 115.57 124.46))
     (stroke (width 0) (type default) (color 0 0 0 0))
   )
@@
     )
   )
+  (sheet (at 138.43 140.97) (size 20.32 15.24) (fields_autoplaced)
+    (stroke (width 0.1524) (type solid) (color 0 0 0 0))
+    (fill (color 0 0 0 0.0000))
+    (property "Sheet name" "AUDIO-AMP" (id 0) (at 138.43 140.2584 0)
+      (effects (font (size 1.27 1.27)) (justify left bottom))
+    )
+    (property "Sheet file" "audio-amp.kicad_sch" (id 1) (at 138.43 156.7946 0)
+      (effects (font (size 1.27 1.27)) (justify left top) hide)
+    )
+    (pin "AUDIO-AMP-IN" input (at 138.43 148.59 180)
+      (effects (font (size 1.27 1.27)) (justify left))
+    )
+  )
   (sheet (at 92.71 81.28) (size 22.86 49.53) (fields_autoplaced)
     (stroke (width 0.1524) (type solid) (color 0 0 0 0))
@@
     )
     (pin "SDA" input (at 41.91 60.96 180)
+      (effects (font (size 1.27 1.27)) (justify left))
+    )
+  )
+  (sheet (at 138.43 52.07) (size 20.32 15.24) (fields_autoplaced)
+    (stroke (width 0.1524) (type solid) (color 0 0 0 0))
+    (fill (color 0 0 0 0.0000))
+    (property "Sheet name" "MIC" (id 0) (at 138.43 51.3584 0)
+      (effects (font (size 1.27 1.27)) (justify left bottom))
+    )
+    (property "Sheet file" "mic.kicad_sch" (id 1) (at 138.43 67.8946 0)
+      (effects (font (size 1.27 1.27)) (justify left top) hide)
+    )
+    (pin "MIC-OUT" output (at 138.43 59.69 180)
       (effects (font (size 1.27 1.27)) (justify left))
     )
@@
     (path "/38ec5edb-504e-48c9-aada-546359fe144d" (page "9"))
     (path "/85cf5236-19af-47bd-b6dc-799e0e38ef1d" (page "10"))
+    (path "/5f063c95-df15-40e2-976b-527eb6081e78" (page "11"))
+    (path "/2f85a458-660d-4f57-88f2-6e8a918eb0ad" (page "12"))
   )
   (symbol_instances

Commit message: added switch
Changed lines of the file:
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@@
       (effects (font (size 1.27 1.27)) (justify right))
     )
-    (pin "OUTL" output (at 92.71 118.11 180)
-      (effects (font (size 1.27 1.27)) (justify left))
-    )
-    (pin "OUTR" output (at 92.71 121.92 180)
-      (effects (font (size 1.27 1.27)) (justify left))
-    )
-    (pin "INL" input (at 92.71 88.9 180)
-      (effects (font (size 1.27 1.27)) (justify left))
-    )
-    (pin "INR" input (at 92.71 92.71 180)
+    (pin "OUTL" input (at 92.71 118.11 180)
+      (effects (font (size 1.27 1.27)) (justify left))
+    )
+    (pin "OUTR" input (at 92.71 121.92 180)
+      (effects (font (size 1.27 1.27)) (justify left))
+    )
+    (pin "INL" output (at 92.71 88.9 180)
+      (effects (font (size 1.27 1.27)) (justify left))
+    )
+    (pin "INR" output (at 92.71 92.71 180)
       (effects (font (size 1.27 1.27)) (justify left))
     )
@@
       (reference "#PWR0139") (unit 1) (value "GND") (footprint "")
     )
+    (path "/38ec5edb-504e-48c9-aada-546359fe144d/da759f4a-bb37-45f9-8648-7a8f0d9161e0"
+      (reference "#PWR0140") (unit 1) (value "+5V") (footprint "")
+    )
+    (path "/38ec5edb-504e-48c9-aada-546359fe144d/3f27d171-45ab-427d-959c-a990870f131c"
+      (reference "#PWR0141") (unit 1) (value "GND") (footprint "")
+    )
+    (path "/38ec5edb-504e-48c9-aada-546359fe144d/af19facd-c48d-4885-913c-109787c3abbd"
+      (reference "#PWR0142") (unit 1) (value "+5V") (footprint "")
+    )
+    (path "/38ec5edb-504e-48c9-aada-546359fe144d/3b8a8636-1821-40a6-b9aa-a8a7f6220414"
+      (reference "#PWR0143") (unit 1) (value "GND") (footprint "")
+    )
+    (path "/38ec5edb-504e-48c9-aada-546359fe144d/83630885-b5c9-42dd-9fb3-3af13411a0b4"
+      (reference "#PWR0144") (unit 1) (value "+5V") (footprint "")
+    )
+    (path "/38ec5edb-504e-48c9-aada-546359fe144d/b304b9ff-e8e7-472e-8da3-c9d79fd305d2"
+      (reference "#PWR0145") (unit 1) (value "GND") (footprint "")
+    )
+    (path "/38ec5edb-504e-48c9-aada-546359fe144d/6e3c7440-55f5-4be0-8b3d-af70e6864ecb"
+      (reference "#PWR0146") (unit 1) (value "GND") (footprint "")
+    )
+    (path "/38ec5edb-504e-48c9-aada-546359fe144d/60bf082b-eccd-4f58-9a30-1b22e73e6f55"
+      (reference "#PWR0147") (unit 1) (value "+5V") (footprint "")
+    )
+    (path "/38ec5edb-504e-48c9-aada-546359fe144d/bfed3ace-3a53-4c2e-9b12-09e454682124"
+      (reference "#PWR0148") (unit 1) (value "+5V") (footprint "")
+    )
+    (path "/38ec5edb-504e-48c9-aada-546359fe144d/484badff-90d0-451f-a8ea-431339845deb"
+      (reference "#PWR0149") (unit 1) (value "GND") (footprint "")
+    )
     (path "/3c85d954-82ab-4b0c-952d-ee98ece6c954/dd12f21a-378a-48c3-99c8-be75492147f4"
       (reference "C1") (unit 1) (value "270pF") (footprint "Capacitor_SMD:C_1206_3216Metric")
@@
       (reference "C29") (unit 1) (value "1uF") (footprint "Capacitor_SMD:C_1206_3216Metric")
     )
+    (path "/38ec5edb-504e-48c9-aada-546359fe144d/989ddabe-5b85-42a3-966f-52ccd0070438"
+      (reference "C30") (unit 1) (value ".1uF") (footprint "Capacitor_SMD:C_0805_2012Metric")
+    )
+    (path "/38ec5edb-504e-48c9-aada-546359fe144d/e85ac339-278f-4383-9b56-2176d2088091"
+      (reference "C31") (unit 1) (value ".1uF") (footprint "Capacitor_SMD:C_0805_2012Metric")
+    )
+    (path "/38ec5edb-504e-48c9-aada-546359fe144d/0c60bc95-f173-49a3-bd44-1a0dbb0a9ed7"
+      (reference "C32") (unit 1) (value ".1uF") (footprint "Capacitor_SMD:C_0805_2012Metric")
+    )
+    (path "/38ec5edb-504e-48c9-aada-546359fe144d/66106ecd-227c-4beb-8846-4845cfa384fe"
+      (reference "C33") (unit 1) (value ".1uF") (footprint "Capacitor_SMD:C_0805_2012Metric")
+    )
+    (path "/38ec5edb-504e-48c9-aada-546359fe144d/6ff452d3-3904-4c39-a51d-66948c9e4903"
+      (reference "C34") (unit 1) (value ".1uF") (footprint "Capacitor_SMD:C_0805_2012Metric")
+    )
+    (path "/38ec5edb-504e-48c9-aada-546359fe144d/114216fc-421a-4c70-b02e-a6e479b3acf6"
+      (reference "C35") (unit 1) (value ".1uF") (footprint "Capacitor_SMD:C_0805_2012Metric")
+    )
+    (path "/38ec5edb-504e-48c9-aada-546359fe144d/d9fd056d-89f3-4b72-8996-24c1e5107117"
+      (reference "C36") (unit 1) (value ".1uF") (footprint "Capacitor_SMD:C_0805_2012Metric")
+    )
+    (path "/38ec5edb-504e-48c9-aada-546359fe144d/2bb25b0b-5c2a-4fa7-8532-8e764a8b7dd8"
+      (reference "C37") (unit 1) (value ".1uF") (footprint "Capacitor_SMD:C_0805_2012Metric")
+    )
     (path "/ccad2f77-41ee-4855-83bb-0372e01592b3/dd78a2a3-3b94-4c56-a19a-5c168aa90dff"
       (reference "D1") (unit 1) (value "1N4148W") (footprint "Diode_SMD:D_SOD-123")
@@
       (reference "R22") (unit 1) (value "330") (footprint "Resistor_SMD:R_0805_2012Metric")
     )
+    (path "/38ec5edb-504e-48c9-aada-546359fe144d/123a37c6-adb1-4a6c-b308-8c44db238c5d"
+      (reference "R23") (unit 1) (value "10k") (footprint "Resistor_SMD:R_0805_2012Metric")
+    )
+    (path "/38ec5edb-504e-48c9-aada-546359fe144d/150d5c70-080f-4e58-8143-02f77bdd6360"
+      (reference "R24") (unit 1) (value "10k") (footprint "Resistor_SMD:R_0805_2012Metric")
+    )
+    (path "/38ec5edb-504e-48c9-aada-546359fe144d/3a13e60a-10e5-4eb1-b5d7-34735052e6e8"
+      (reference "R25") (unit 1) (value "10k") (footprint "Resistor_SMD:R_0805_2012Metric")
+    )
+    (path "/38ec5edb-504e-48c9-aada-546359fe144d/69d3b0d0-871c-4b71-8aff-1526a131545d"
+      (reference "R26") (unit 1) (value "10k") (footprint "Resistor_SMD:R_0805_2012Metric")
+    )
+    (path "/38ec5edb-504e-48c9-aada-546359fe144d/b01c7c89-d823-4bde-85f1-84745239d269"
+      (reference "R27") (unit 1) (value "10k") (footprint "Resistor_SMD:R_0805_2012Metric")
+    )
+    (path "/38ec5edb-504e-48c9-aada-546359fe144d/5f3ce1b6-f498-4f65-8b9f-02381cd0c75b"
+      (reference "R28") (unit 1) (value "10k") (footprint "Resistor_SMD:R_0805_2012Metric")
+    )
+    (path "/38ec5edb-504e-48c9-aada-546359fe144d/7114254b-7844-4f95-8cb6-728c7892b39d"
+      (reference "R29") (unit 1) (value "10k") (footprint "Resistor_SMD:R_0805_2012Metric")
+    )
+    (path "/38ec5edb-504e-48c9-aada-546359fe144d/3bcbbb2b-6426-4545-823e-f370ca7587b8"
+      (reference "R30") (unit 1) (value "10k") (footprint "Resistor_SMD:R_0805_2012Metric")
+    )
     (path "/4b1ef805-7fd0-4a4a-b5da-5feeaa035c65/dbc98a07-c075-4ec8-822f-59596956d619"
       (reference "T1") (unit 1) (value "T37-6 5:25") (footprint "Xenir:T37 Transformer")
@@
       (reference "U6") (unit 1) (value "ESP32-A1S") (footprint "Xenir:ESP32-A1S")
     )
+    (path "/38ec5edb-504e-48c9-aada-546359fe144d/36f74fc8-7aa3-4ba8-81d0-37fd62bf6dc9"
+      (reference "U7") (unit 1) (value "FST3257") (footprint "Xenir:SO16")
+    )
     (path "/4b1ef805-7fd0-4a4a-b5da-5feeaa035c65/a3e1d27e-f1e5-419b-8a71-6427134bb505"
