File: SDR-Transceiver.kicad_sch (KiCad schematic)
At the start: 0 parts

Commit message: added legend
Other:
- sheet AUDIO-AMP renamed Audio Amp
- sheet Audio-Switch renamed Audio Switch
- sheet Local-Oscillator renamed Local Oscillator
- sheet RF-SWITCH renamed RF Switch
- sheet Tayloe-Detector renamed Tayloe Detector
- sheet Tayloe-Encoder renamed Tayloe Encoder
- note added: "Receive Path"
- note added: "Transmit Path"
- note added: "Transmit/Receive"

Commit message: gg
Parts:
- added J1: BNC, Xenir:BNC, symbol Xenir:BNC
Connections:
- new net GND: J1.GND
- new net RF Switch/Antenna: J1.S (OUT)
Other:
- sheet RF Switch ports: added Antenna; removed none
Changed lines of the file:
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@@
   (junction (at 121.92 85.09) (diameter 0) (color 0 0 0 0)
   )
-  (wire (pts (xy 256.54 110.49) (xy 250.19 110.49))
-    (stroke (width 0.508) (type default) (color 255 0 0 1))
+  (wire (pts (xy 254 96.52) (xy 254 107.95))
+    (stroke (width 0.5) (type default) (color 255 0 0 1))
   )
   (wire (pts (xy 138.43 148.59) (xy 121.92 148.59))
@@
     (stroke (width 0) (type default) (color 0 0 0 0))
   )
-  (wire (pts (xy 250.19 96.52) (xy 256.54 96.52))
-    (stroke (width 0.508) (type default) (color 255 0 0 1))
-  )
   (wire (pts (xy 176.53 87.63) (xy 176.53 100.33))
     (stroke (width 0.508) (type default) (color 0 255 0 1))
@@
     (stroke (width 0) (type default) (color 0 0 0 0))
   )
+  (wire (pts (xy 250.19 96.52) (xy 254 96.52))
+    (stroke (width 0.5) (type default) (color 255 0 0 1))
+  )
   (wire (pts (xy 158.75 87.63) (xy 176.53 87.63))
     (stroke (width 0.508) (type default) (color 0 255 0 1))
@@
     (stroke (width 0.508) (type default) (color 0 0 255 1))
   )
+  (wire (pts (xy 220.98 115.57) (xy 224.79 115.57))
+    (stroke (width 0.5) (type solid) (color 0 0 255 1))
+  )
   (wire (pts (xy 176.53 118.11) (xy 176.53 104.14))
     (stroke (width 0.508) (type default) (color 255 0 0 1))
@@
     (stroke (width 0.508) (type default) (color 255 0 0 1))
   )
-  (wire (pts (xy 220.98 110.49) (xy 229.87 110.49))
+  (wire (pts (xy 220.98 107.95) (xy 229.87 107.95))
     (stroke (width 0.508) (type default) (color 255 0 0 1))
   )
   (wire (pts (xy 138.43 59.69) (xy 121.92 59.69))
     (stroke (width 0.508) (type default) (color 255 0 0 1))
+  )
+  (wire (pts (xy 254 107.95) (xy 250.19 107.95))
+    (stroke (width 0.5) (type default) (color 255 0 0 1))
   )
   (wire (pts (xy 125.73 78.74) (xy 125.73 92.71))
@@
     (stroke (width 0.508) (type default) (color 0 0 255 1))
   )
+  (wire (pts (xy 224.79 128.27) (xy 229.87 128.27))
+    (stroke (width 0.5) (type solid) (color 0 0 255 1))
+  )
   (wire (pts (xy 209.55 86.36) (xy 209.55 88.9))
     (stroke (width 0) (type default) (color 0 0 0 0))
@@
     (stroke (width 0.508) (type default) (color 0 0 255 1))
   )
-  (wire (pts (xy 256.54 96.52) (xy 256.54 110.49))
-    (stroke (width 0.508) (type default) (color 255 0 0 1))
-  )
   (wire (pts (xy 138.43 78.74) (xy 125.73 78.74))
     (stroke (width 0.508) (type default) (color 0 255 0 1))
@@
   (wire (pts (xy 121.92 124.46) (xy 115.57 124.46))
     (stroke (width 0.508) (type default) (color 0 255 0 1))
+  )
+  (wire (pts (xy 224.79 115.57) (xy 224.79 128.27))
+    (stroke (width 0.5) (type solid) (color 0 0 255 1))
   )
   (wire (pts (xy 220.98 96.52) (xy 229.87 96.52))
@@
     )
   )
-  (global_label "T{slash}R" (shape input) (at 229.87 91.44 180) (fields_autoplaced)
+  (global_label "T{slash}R" (shape input) (at 229.87 92.71 180) (fields_autoplaced)
     (effects (font (size 1.27 1.27)) (justify right))
-    (property "Intersheet References" "${INTERSHEET_REFS}" (id 0) (at 223.8888 91.5194 0)
+    (property "Intersheet References" "${INTERSHEET_REFS}" (id 0) (at 223.8888 92.7894 0)
       (effects (font (size 1.27 1.27)) (justify right) hide)
     )
@@
     )
   )
+  (symbol (lib_id "power:GND") (at 234.95 133.35 0) (unit 1)
+    (in_bom yes) (on_board yes) (fields_autoplaced)
+    (property "Reference" "#PWR0104" (id 0) (at 234.95 139.7 0)
+      (effects (font (size 1.27 1.27)) hide)
+    )
+    (property "Value" "GND" (id 1) (at 234.95 138.43 0))
+    (property "Footprint" "" (id 2) (at 234.95 133.35 0)
+      (effects (font (size 1.27 1.27)) hide)
+    )
+    (property "Datasheet" "" (id 3) (at 234.95 133.35 0)
+      (effects (font (size 1.27 1.27)) hide)
+    )
+    (pin "1")
+  )
+  (symbol (lib_id "Xenir:BNC") (at 234.95 128.27 0) (mirror y) (unit 1)
+    (in_bom yes) (on_board yes) (fields_autoplaced)
+    (property "Reference" "J1" (id 0) (at 238.76 126.9999 0)
+      (effects (font (size 1.27 1.27)) (justify right))
+    )
+    (property "Value" "BNC" (id 1) (at 238.76 129.5399 0)
+      (effects (font (size 1.27 1.27)) (justify right))
+    )
+    (property "Footprint" "Xenir:BNC" (id 2) (at 234.95 124.46 0)
+      (effects (font (size 1.27 1.27)) hide)
+    )
+    (property "Datasheet" "" (id 3) (at 234.95 124.46 0)
+      (effects (font (size 1.27 1.27)) hide)
+    )
+    (pin "GND")
+    (pin "S")
+  )
   (sheet (at 138.43 140.97) (size 20.32 15.24) (fields_autoplaced)
     (stroke (width 0.1524) (type solid) (color 0 0 0 0))
@@
     )
   )
-  (sheet (at 229.87 104.14) (size 20.32 8.89)
+  (sheet (at 229.87 104.14) (size 20.32 7.62)
     (stroke (width 0.1524) (type solid) (color 0 0 0 0))
     (fill (color 0 0 0 0.0000))
@@
       (effects (font (size 1.27 1.27)) (justify left top) hide)
     )
-    (pin "IN-LPF" input (at 250.19 110.49 0)
-      (effects (font (size 1.27 1.27)) (justify right))
-    )
-    (pin "OUT-LPF" output (at 229.87 110.49 180)
-      (effects (font (size 1.27 1.27)) (justify left))
-    )
-  )
-  (sheet (at 195.58 66.04) (size 20.32 13.97) (fields_autoplaced)
-    (stroke (width 0.1524) (type solid) (color 0 0 0 0))
-    (fill (color 0 0 0 0.0000))
-    (property "Sheet name" "BPF" (id 0) (at 194.5509 80.01 90)
+    (pin "IN-LPF" input (at 250.19 107.95 0)
+      (effects (font (size 1.27 1.27)) (justify right))
+    )
+    (pin "OUT-LPF" output (at 229.87 107.95 180)
+      (effects (font (size 1.27 1.27)) (justify left))
+    )
+  )
+  (sheet (at 195.58 66.04) (size 20.32 13.97)
+    (stroke (width 0.1524) (type solid) (color 0 0 0 0))
+    (fill (color 0 0 0 0.0000))
+    (property "Sheet name" "BPF" (id 0) (at 195.58 66.04 0)
       (effects (font (size 1.905 1.905)) (justify left bottom))
     )
@@
       (effects (font (size 1.27 1.27)) (justify left))
     )
-    (pin "From-LPF" input (at 220.98 110.49 0)
+    (pin "From-LPF" input (at 220.98 107.95 0)
       (effects (font (size 1.27 1.27)) (justify right))
     )
@@
       (effects (font (size 1.27 1.27)) (justify right))
     )
+    (pin "Antenna" bidirectional (at 220.98 115.57 0)
+      (effects (font (size 1.27 1.27)) (justify right))
+    )
   )
   (sheet (at 229.87 90.17) (size 20.32 8.89) (fields_autoplaced)
@@
       (effects (font (size 1.27 1.27)) (justify right))
     )
-    (pin "T{slash}R" input (at 229.87 91.44 180)
+    (pin "T{slash}R" input (at 229.87 92.71 180)
       (effects (font (size 1.27 1.27)) (justify left))
     )
@@
       (reference "#PWR0103") (unit 1) (value "GND") (footprint "")
     )
-    (path "/ccad2f77-41ee-4855-83bb-0372e01592b3/ddbec5bb-7c8b-4048-b8e3-d23936937af1"
+    (path "/0eab1020-38b9-4653-8be0-bdfc79f8dc1e"
       (reference "#PWR0104") (unit 1) (value "GND") (footprint "")
     )
@@
       (reference "D2") (unit 1) (value "1N4148W") (footprint "Diode_SMD:D_SOD-123")
     )
-    (path "/ccad2f77-41ee-4855-83bb-0372e01592b3/1dadd5ca-5944-4652-9415-19e79d3e293b"
+    (path "/593abb02-8f1b-4ca5-9026-3e326ffd66bf"
       (reference "J1") (unit 1) (value "BNC") (footprint "Xenir:BNC")
     )

Commit message: gg
Other:
- note added: "High on Transmit Low on Receive"
Changed lines of the file:
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@@
     (effects (font (size 1.905 1.905)) (justify left bottom))
+  )
+  (text "High on Transmit\nLow on Receive" (at 69.85 81.28 0)
+    (effects (font (size 0.762 0.762)) (justify left bottom))
   )
   (text "Receive Path" (at 238.76 30.48 0)
