File: SDR-Transceiver.kicad_sch (KiCad schematic)
At the start: 1 part, among them J1 BNC

Commit message: added ptt
Other:
- sheet DSP ports: added PTT-IN; removed none
- sheet MIC ports: added PTT; removed none
Changed lines of the file:
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@@
     (stroke (width 0.508) (type default) (color 0 149 0 1))
+  )
+  (wire (pts (xy 97.79 55.88) (xy 97.79 72.39))
+    (stroke (width 0) (type default) (color 0 0 0 0))
   )
   (wire (pts (xy 34.29 60.96) (xy 34.29 106.68))
@@
     (stroke (width 0.508) (type default) (color 0 0 255 1))
   )
+  (wire (pts (xy 138.43 55.88) (xy 97.79 55.88))
+    (stroke (width 0) (type default) (color 0 0 0 0))
+  )
   (wire (pts (xy 220.98 115.57) (xy 224.79 115.57))
     (stroke (width 0.5) (type solid) (color 0 0 255 1))
@@
     (stroke (width 0.508) (type default) (color 154 0 0 1))
   )
+  (wire (pts (xy 97.79 72.39) (xy 49.53 72.39))
+    (stroke (width 0) (type default) (color 0 0 0 0))
+  )
   (wire (pts (xy 121.92 87.63) (xy 115.57 87.63))
     (stroke (width 0.508) (type default) (color 154 0 0 1))
@@
   (wire (pts (xy 115.57 114.3) (xy 128.27 114.3))
     (stroke (width 0.508) (type default) (color 154 0 0 1))
+  )
+  (wire (pts (xy 49.53 72.39) (xy 49.53 81.28))
+    (stroke (width 0) (type default) (color 0 0 0 0))
   )
   (wire (pts (xy 128.27 82.55) (xy 128.27 95.25))
@@
       (effects (font (size 1.27 1.27)) (justify left))
     )
+    (pin "PTT" output (at 138.43 55.88 180)
+      (effects (font (size 1.27 1.27)) (justify left))
+    )
   )
   (sheet (at 40.64 143.51) (size 22.86 13.97) (fields_autoplaced)
@@
       (effects (font (size 1.27 1.27)) (justify right))
     )
+    (pin "PTT-IN" input (at 49.53 81.28 90)
+      (effects (font (size 1.27 1.27)) (justify right))
+    )

Commit message: added mounting holes
Parts:
- added H1, H2, H3, H4: MountingHole_Pad, MountingHole:MountingHole_3.2mm_M3, symbol Mechanical:MountingHole_Pad
Connections:
- no-connect marks 0 -> 4
Changed lines of the file:
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@@
   (junction (at 121.92 85.09) (diameter 0) (color 0 0 0 0)
   )
+  (no_connect (at 95.25 35.56))
+  (no_connect (at 87.63 27.94))
+  (no_connect (at 87.63 35.56))
+  (no_connect (at 95.25 27.94))
   (wire (pts (xy 254 96.52) (xy 254 107.95))
     (stroke (width 0.5) (type default) (color 255 0 0 1))
@@
     (pin "1")
   )
+  (symbol (lib_id "Mechanical:MountingHole_Pad") (at 95.25 25.4 0) (unit 1)
+    (in_bom yes) (on_board yes) (fields_autoplaced)
+    (property "Reference" "H3" (id 0) (at 97.79 24.1299 0)
+      (effects (font (size 1.27 1.27)) (justify left))
+    )
+    (property "Value" "MountingHole_Pad" (id 1) (at 97.79 25.3999 0)
+      (effects (font (size 1.27 1.27)) (justify left) hide)
+    )
+    (property "Footprint" "MountingHole:MountingHole_3.2mm_M3" (id 2) (at 95.25 25.4 0)
+      (effects (font (size 1.27 1.27)) hide)
+    )
+    (property "Datasheet" "~" (id 3) (at 95.25 25.4 0)
+      (effects (font (size 1.27 1.27)) hide)
+    )
+    (pin "1")
+  )
+  (symbol (lib_id "Mechanical:MountingHole_Pad") (at 95.25 33.02 0) (unit 1)
+    (in_bom yes) (on_board yes) (fields_autoplaced)
+    (property "Reference" "H4" (id 0) (at 97.79 31.7499 0)
+      (effects (font (size 1.27 1.27)) (justify left))
+    )
+    (property "Value" "MountingHole_Pad" (id 1) (at 97.79 33.0199 0)
+      (effects (font (size 1.27 1.27)) (justify left) hide)
+    )
+    (property "Footprint" "MountingHole:MountingHole_3.2mm_M3" (id 2) (at 95.25 33.02 0)
+      (effects (font (size 1.27 1.27)) hide)
+    )
+    (property "Datasheet" "~" (id 3) (at 95.25 33.02 0)
+      (effects (font (size 1.27 1.27)) hide)
+    )
+    (pin "1")
+  )
   (symbol (lib_id "Xenir:BNC") (at 234.95 128.27 0) (mirror y) (unit 1)
     (in_bom yes) (on_board yes) (fields_autoplaced)
@@
     (pin "GND")
     (pin "S")
+  )
+  (symbol (lib_id "Mechanical:MountingHole_Pad") (at 87.63 25.4 0) (unit 1)
+    (in_bom yes) (on_board yes)
+    (property "Reference" "H2" (id 0) (at 82.3994 24.2156 0)
+      (effects (font (size 1.27 1.27)) (justify left))
+    )
+    (property "Value" "MountingHole_Pad" (id 1) (at 90.17 25.3999 0)
+      (effects (font (size 1.27 1.27)) (justify left) hide)
+    )
+    (property "Footprint" "MountingHole:MountingHole_3.2mm_M3" (id 2) (at 87.63 25.4 0)
+      (effects (font (size 1.27 1.27)) hide)
+    )
+    (property "Datasheet" "~" (id 3) (at 87.63 25.4 0)
+      (effects (font (size 1.27 1.27)) hide)
+    )
+    (pin "1")
+  )
+  (symbol (lib_id "Mechanical:MountingHole_Pad") (at 87.63 33.02 0) (unit 1)
+    (in_bom yes) (on_board yes)
+    (property "Reference" "H1" (id 0) (at 82.55 31.75 0)
+      (effects (font (size 1.27 1.27)) (justify left))
+    )
+    (property "Value" "MountingHole_Pad" (id 1) (at 90.17 33.0199 0)
+      (effects (font (size 1.27 1.27)) (justify left) hide)
+    )
+    (property "Footprint" "MountingHole:MountingHole_3.2mm_M3" (id 2) (at 87.63 33.02 0)
+      (effects (font (size 1.27 1.27)) hide)
+    )
+    (property "Datasheet" "~" (id 3) (at 87.63 33.02 0)
+      (effects (font (size 1.27 1.27)) hide)
+    )
+    (pin "1")
   )
   (sheet (at 138.43 140.97) (size 20.32 15.24) (fields_autoplaced)
@@
       (reference "D2") (unit 1) (value "1N4148W") (footprint "Diode_SMD:D_SOD-123")
     )
+    (path "/f13dc858-3a27-4037-8443-3b1580373d9d"
+      (reference "H1") (unit 1) (value "MountingHole_Pad") (footprint "MountingHole:MountingHole_3.2mm_M3")
+    )
+    (path "/a1cbfdf6-e208-44a4-8f34-45f4e8001110"
+      (reference "H2") (unit 1) (value "MountingHole_Pad") (footprint "MountingHole:MountingHole_3.2mm_M3")
+    )
+    (path "/3b352b54-e3e2-4616-8f54-c7d036748caa"
+      (reference "H3") (unit 1) (value "MountingHole_Pad") (footprint "MountingHole:MountingHole_3.2mm_M3")
+    )
+    (path "/4c7815e8-dc25-4d27-8696-4a87ca056862"
+      (reference "H4") (unit 1) (value "MountingHole_Pad") (footprint "MountingHole:MountingHole_3.2mm_M3")
+    )
     (path "/593abb02-8f1b-4ca5-9026-3e326ffd66bf"

Commit message: gg
Parts:
- H1, H2, H3, H4: footprint MountingHole:MountingHole_3.2mm_M3 -> MountingHole:MountingHole_3.2mm_M3_Pad_Via
Connections:
- net GND: now also H1.1, H2.1, H3.1, H4.1
- no-connect marks 4 -> 0
Other:
- moved on the sheet: H2, H3
Changed lines of the file:
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@@
   (junction (at 121.92 85.09) (diameter 0) (color 0 0 0 0)
   )
-  (no_connect (at 95.25 35.56))
-  (no_connect (at 87.63 27.94))
-  (no_connect (at 87.63 35.56))
-  (no_connect (at 95.25 27.94))
   (wire (pts (xy 254 96.52) (xy 254 107.95))
     (stroke (width 0.5) (type default) (color 255 0 0 1))
@@
     (pin "1")
   )
-  (symbol (lib_id "Mechanical:MountingHole_Pad") (at 95.25 25.4 0) (unit 1)
+  (symbol (lib_id "Mechanical:MountingHole_Pad") (at 95.25 20.32 0) (unit 1)
     (in_bom yes) (on_board yes) (fields_autoplaced)
-    (property "Reference" "H3" (id 0) (at 97.79 24.1299 0)
-      (effects (font (size 1.27 1.27)) (justify left))
-    )
-    (property "Value" "MountingHole_Pad" (id 1) (at 97.79 25.3999 0)
+    (property "Reference" "H3" (id 0) (at 97.79 19.0499 0)
+      (effects (font (size 1.27 1.27)) (justify left))
+    )
+    (property "Value" "MountingHole_Pad" (id 1) (at 97.79 20.3199 0)
       (effects (font (size 1.27 1.27)) (justify left) hide)
     )
-    (property "Footprint" "MountingHole:MountingHole_3.2mm_M3" (id 2) (at 95.25 25.4 0)
-      (effects (font (size 1.27 1.27)) hide)
-    )
-    (property "Datasheet" "~" (id 3) (at 95.25 25.4 0)
+    (property "Footprint" "MountingHole:MountingHole_3.2mm_M3_Pad_Via" (id 2) (at 95.25 20.32 0)
+      (effects (font (size 1.27 1.27)) hide)
+    )
+    (property "Datasheet" "~" (id 3) (at 95.25 20.32 0)
+      (effects (font (size 1.27 1.27)) hide)
+    )
+    (pin "1")
+  )
+  (symbol (lib_id "power:GND") (at 87.63 35.56 0) (unit 1)
+    (in_bom yes) (on_board yes) (fields_autoplaced)
+    (property "Reference" "#PWR0213" (id 0) (at 87.63 41.91 0)
+      (effects (font (size 1.27 1.27)) hide)
+    )
+    (property "Value" "GND" (id 1) (at 87.63 40.64 0))
+    (property "Footprint" "" (id 2) (at 87.63 35.56 0)
+      (effects (font (size 1.27 1.27)) hide)
+    )
+    (property "Datasheet" "" (id 3) (at 87.63 35.56 0)
       (effects (font (size 1.27 1.27)) hide)
     )
@@
       (effects (font (size 1.27 1.27)) (justify left) hide)
     )
-    (property "Footprint" "MountingHole:MountingHole_3.2mm_M3" (id 2) (at 95.25 33.02 0)
+    (property "Footprint" "MountingHole:MountingHole_3.2mm_M3_Pad_Via" (id 2) (at 95.25 33.02 0)
       (effects (font (size 1.27 1.27)) hide)
     )
@@
     (pin "S")
   )
-  (symbol (lib_id "Mechanical:MountingHole_Pad") (at 87.63 25.4 0) (unit 1)
+  (symbol (lib_id "power:GND") (at 95.25 22.86 0) (unit 1)
+    (in_bom yes) (on_board yes) (fields_autoplaced)
+    (property "Reference" "#PWR0206" (id 0) (at 95.25 29.21 0)
+      (effects (font (size 1.27 1.27)) hide)
+    )
+    (property "Value" "GND" (id 1) (at 95.25 27.94 0))
+    (property "Footprint" "" (id 2) (at 95.25 22.86 0)
+      (effects (font (size 1.27 1.27)) hide)
+    )
+    (property "Datasheet" "" (id 3) (at 95.25 22.86 0)
+      (effects (font (size 1.27 1.27)) hide)
+    )
+    (pin "1")
+  )
+  (symbol (lib_id "power:GND") (at 95.25 35.56 0) (unit 1)
+    (in_bom yes) (on_board yes) (fields_autoplaced)
+    (property "Reference" "#PWR0214" (id 0) (at 95.25 41.91 0)
+      (effects (font (size 1.27 1.27)) hide)
+    )
+    (property "Value" "GND" (id 1) (at 95.25 40.64 0))
+    (property "Footprint" "" (id 2) (at 95.25 35.56 0)
+      (effects (font (size 1.27 1.27)) hide)
+    )
+    (property "Datasheet" "" (id 3) (at 95.25 35.56 0)
+      (effects (font (size 1.27 1.27)) hide)
+    )
+    (pin "1")
+  )
+  (symbol (lib_id "Mechanical:MountingHole_Pad") (at 87.63 20.32 0) (unit 1)
     (in_bom yes) (on_board yes)
-    (property "Reference" "H2" (id 0) (at 82.3994 24.2156 0)
-      (effects (font (size 1.27 1.27)) (justify left))
-    )
-    (property "Value" "MountingHole_Pad" (id 1) (at 90.17 25.3999 0)
+    (property "Reference" "H2" (id 0) (at 82.3994 19.1356 0)
+      (effects (font (size 1.27 1.27)) (justify left))
+    )
+    (property "Value" "MountingHole_Pad" (id 1) (at 90.17 20.3199 0)
       (effects (font (size 1.27 1.27)) (justify left) hide)
     )
-    (property "Footprint" "MountingHole:MountingHole_3.2mm_M3" (id 2) (at 87.63 25.4 0)
-      (effects (font (size 1.27 1.27)) hide)
-    )
-    (property "Datasheet" "~" (id 3) (at 87.63 25.4 0)
+    (property "Footprint" "MountingHole:MountingHole_3.2mm_M3_Pad_Via" (id 2) (at 87.63 20.32 0)
+      (effects (font (size 1.27 1.27)) hide)
+    )
+    (property "Datasheet" "~" (id 3) (at 87.63 20.32 0)
+      (effects (font (size 1.27 1.27)) hide)
+    )
+    (pin "1")
+  )
+  (symbol (lib_id "power:GND") (at 87.63 22.86 0) (unit 1)
+    (in_bom yes) (on_board yes) (fields_autoplaced)
+    (property "Reference" "#PWR0212" (id 0) (at 87.63 29.21 0)
+      (effects (font (size 1.27 1.27)) hide)
+    )
+    (property "Value" "GND" (id 1) (at 87.63 27.94 0))
+    (property "Footprint" "" (id 2) (at 87.63 22.86 0)
+      (effects (font (size 1.27 1.27)) hide)
+    )
+    (property "Datasheet" "" (id 3) (at 87.63 22.86 0)
       (effects (font (size 1.27 1.27)) hide)
     )
@@
       (effects (font (size 1.27 1.27)) (justify left) hide)
     )
-    (property "Footprint" "MountingHole:MountingHole_3.2mm_M3" (id 2) (at 87.63 33.02 0)
+    (property "Footprint" "MountingHole:MountingHole_3.2mm_M3_Pad_Via" (id 2) (at 87.63 33.02 0)
       (effects (font (size 1.27 1.27)) hide)
     )
@@
       (reference "#PWR0205") (unit 1) (value "GND") (footprint "")
     )
+    (path "/8a803909-3cdf-4586-85b3-ed32064db6cd"
+      (reference "#PWR0206") (unit 1) (value "GND") (footprint "")
+    )
     (path "/5f063c95-df15-40e2-976b-527eb6081e78/669502ed-d4c3-4e15-8b90-1c3d1dd6d544"
       (reference "#PWR0207") (unit 1) (value "+5V") (footprint "")
@@
       (reference "#PWR0211") (unit 1) (value "+5V") (footprint "")
     )
+    (path "/e7a8938e-5326-4cab-a9df-89daad7db503"
+      (reference "#PWR0212") (unit 1) (value "GND") (footprint "")
+    )
+    (path "/3f4f24b8-bec8-4051-8a4b-cf484e0d306e"
+      (reference "#PWR0213") (unit 1) (value "GND") (footprint "")
+    )
+    (path "/993bcb89-41cf-4029-9d09-496dbb0d0f28"
+      (reference "#PWR0214") (unit 1) (value "GND") (footprint "")
+    )
     (path "/fcc9c1e3-d78e-4432-bbd5-5698bfd2ca1f/34067e6c-49d8-490e-84ad-4e212d112ce1"
       (reference "C1") (unit 1) (value ".1uF") (footprint "Capacitor_SMD:C_0805_2012Metric")
@@
     )
     (path "/f13dc858-3a27-4037-8443-3b1580373d9d"
-      (reference "H1") (unit 1) (value "MountingHole_Pad") (footprint "MountingHole:MountingHole_3.2mm_M3")
+      (reference "H1") (unit 1) (value "MountingHole_Pad") (footprint "MountingHole:MountingHole_3.2mm_M3_Pad_Via")
     )
     (path "/a1cbfdf6-e208-44a4-8f34-45f4e8001110"
-      (reference "H2") (unit 1) (value "MountingHole_Pad") (footprint "MountingHole:MountingHole_3.2mm_M3")
+      (reference "H2") (unit 1) (value "MountingHole_Pad") (footprint "MountingHole:MountingHole_3.2mm_M3_Pad_Via")
     )
     (path "/3b352b54-e3e2-4616-8f54-c7d036748caa"
-      (reference "H3") (unit 1) (value "MountingHole_Pad") (footprint "MountingHole:MountingHole_3.2mm_M3")
+      (reference "H3") (unit 1) (value "MountingHole_Pad") (footprint "MountingHole:MountingHole_3.2mm_M3_Pad_Via")
     )
     (path "/4c7815e8-dc25-4d27-8696-4a87ca056862"
-      (reference "H4") (unit 1) (value "MountingHole_Pad") (footprint "MountingHole:MountingHole_3.2mm_M3")
+      (reference "H4") (unit 1) (value "MountingHole_Pad") (footprint "MountingHole:MountingHole_3.2mm_M3_Pad_Via")
     )
     (path "/593abb02-8f1b-4ca5-9026-3e326ffd66bf"
