File: SDR-Transceiver.kicad_pcb (KiCad board)
At the start: 2 copper layers, 103 parts, among them J1 BNC, J2 Conn_01x03_Female, J3 Conn_01x03_Female, K1 G6S-2, K2 G6S-2, T1 T37-6 5:25, T2 T37-6 25:5, T3 T50_SPLITTER, T4 T50_SPLITTER, U1 FST3253, U2 LM4562, U3 FST3253, U4 LM4562, U5 LM4562, U6 ESP32-A1S, U7 FST3257

Commit message: gg
Parts:
- added J4: Conn_01x03_Female, Connector_PinSocket_2.54mm:PinSocket_1x03_P2.54mm_Vertical, F.Cu at (164.5, 54.0)
- added J5: Conn_01x03_Female, Connector_PinSocket_2.54mm:PinSocket_1x03_P2.54mm_Vertical, F.Cu at (159.9, 54.0)
Changed lines of the file:
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@@
+  )
+  (footprint "Connector_PinSocket_2.54mm:PinSocket_1x03_P2.54mm_Vertical" (layer "F.Cu")
+    (at 164.465 53.975)
+    (descr "Through hole straight socket strip, 1x03, 2.54mm pitch, single row (from Kicad 4.0.7), script generated")
+    (tags "Through hole socket strip THT 1x03 2.54mm single row")
+    (property "Sheetfile" "LPF.kicad_sch")
+    (property "Sheetname" "LPF")
+    (attr through_hole)
+    (fp_text reference "J4" (at 0 -2.77) (layer "F.SilkS")
+      (effects (font (size 1 1) (thickness 0.15)))
+    )
+    (fp_text value "Conn_01x03_Female" (at 0 7.85) (layer "F.Fab")
+      (effects (font (size 1 1) (thickness 0.15)))
+    )
+    (fp_text user "${REFERENCE}" (at 0 2.54 90) (layer "F.Fab")
+      (effects (font (size 1 1) (thickness 0.15)))
+    )
+    (fp_line (start -1.33 1.27) (end -1.33 6.41) (layer "F.SilkS") (width 0.12))
+    (fp_line (start -1.33 1.27) (end 1.33 1.27) (layer "F.SilkS") (width 0.12))
+    (fp_line (start -1.33 6.41) (end 1.33 6.41) (layer "F.SilkS") (width 0.12))
+    (fp_line (start 1.33 1.27) (end 1.33 6.41) (layer "F.SilkS") (width 0.12))
+    (fp_line (start 0 -1.33) (end 1.33 -1.33) (layer "F.SilkS") (width 0.12))
+    (fp_line (start 1.33 -1.33) (end 1.33 0) (layer "F.SilkS") (width 0.12))
+    (fp_line (start 1.75 6.85) (end -1.8 6.85) (layer "F.CrtYd") (width 0.05))
+    (fp_line (start 1.75 -1.8) (end 1.75 6.85) (layer "F.CrtYd") (width 0.05))
+    (fp_line (start -1.8 6.85) (end -1.8 -1.8) (layer "F.CrtYd") (width 0.05))
+    (fp_line (start -1.8 -1.8) (end 1.75 -1.8) (layer "F.CrtYd") (width 0.05))
+    (fp_line (start 1.27 -0.635) (end 1.27 6.35) (layer "F.Fab") (width 0.1))
+    (fp_line (start -1.27 6.35) (end -1.27 -1.27) (layer "F.Fab") (width 0.1))
+    (fp_line (start 0.635 -1.27) (end 1.27 -0.635) (layer "F.Fab") (width 0.1))
+    (fp_line (start 1.27 6.35) (end -1.27 6.35) (layer "F.Fab") (width 0.1))
+    (fp_line (start -1.27 -1.27) (end 0.635 -1.27) (layer "F.Fab") (width 0.1))
+    (pad "1" thru_hole rect (at 0 0) (size 1.7 1.7) (drill 1) (layers *.Cu *.Mask)
+      (net 1 "GND") (pinfunction "Pin_1") (pintype "passive"))
+    (pad "2" thru_hole oval (at 0 2.54) (size 1.7 1.7) (drill 1) (layers *.Cu *.Mask)
+      (net 2 "/LPF/IN-LPF") (pinfunction "Pin_2") (pintype "passive"))
+    (pad "3" thru_hole oval (at 0 5.08) (size 1.7 1.7) (drill 1) (layers *.Cu *.Mask)
+      (net 1 "GND") (pinfunction "Pin_3") (pintype "passive"))
+    (model "${KICAD6_3DMODEL_DIR}/Connector_PinSocket_2.54mm.3dshapes/PinSocket_1x03_P2.54mm_Vertical.wrl"
+      (offset (xyz 0 0 0))
+      (scale (xyz 1 1 1))
+      (rotate (xyz 0 0 0))
+    )
   )
   (footprint "Connector_PinSocket_2.54mm:PinSocket_1x03_P2.54mm_Vertical" (layer "F.Cu")
@@
     (pad "GND" smd rect locked (at 0.381 12.827) (size 3.8 3.8) (layers "F.Cu" "F.Paste" "F.Mask"))
   )
+  (footprint "Connector_PinSocket_2.54mm:PinSocket_1x03_P2.54mm_Vertical" (layer "F.Cu")
+    (at 159.865 53.975)
+    (descr "Through hole straight socket strip, 1x03, 2.54mm pitch, single row (from Kicad 4.0.7), script generated")
+    (tags "Through hole socket strip THT 1x03 2.54mm single row")
+    (property "Sheetfile" "LPF.kicad_sch")
+    (property "Sheetname" "LPF")
+    (attr through_hole)
+    (fp_text reference "J5" (at 0 -2.77) (layer "F.SilkS")
+      (effects (font (size 1 1) (thickness 0.15)))
+    )
+    (fp_text value "Conn_01x03_Female" (at 0 7.85) (layer "F.Fab")
+      (effects (font (size 1 1) (thickness 0.15)))
+    )
+    (fp_text user "${REFERENCE}" (at 0 2.54 90) (layer "F.Fab")
+      (effects (font (size 1 1) (thickness 0.15)))
+    )
+    (fp_line (start -1.33 6.41) (end 1.33 6.41) (layer "F.SilkS") (width 0.12))
+    (fp_line (start 1.33 -1.33) (end 1.33 0) (layer "F.SilkS") (width 0.12))
+    (fp_line (start -1.33 1.27) (end 1.33 1.27) (layer "F.SilkS") (width 0.12))
+    (fp_line (start 1.33 1.27) (end 1.33 6.41) (layer "F.SilkS") (width 0.12))
+    (fp_line (start 0 -1.33) (end 1.33 -1.33) (layer "F.SilkS") (width 0.12))
+    (fp_line (start -1.33 1.27) (end -1.33 6.41) (layer "F.SilkS") (width 0.12))
+    (fp_line (start 1.75 -1.8) (end 1.75 6.85) (layer "F.CrtYd") (width 0.05))
+    (fp_line (start 1.75 6.85) (end -1.8 6.85) (layer "F.CrtYd") (width 0.05))
+    (fp_line (start -1.8 -1.8) (end 1.75 -1.8) (layer "F.CrtYd") (width 0.05))
+    (fp_line (start -1.8 6.85) (end -1.8 -1.8) (layer "F.CrtYd") (width 0.05))
+    (fp_line (start 1.27 -0.635) (end 1.27 6.35) (layer "F.Fab") (width 0.1))
+    (fp_line (start -1.27 6.35) (end -1.27 -1.27) (layer "F.Fab") (width 0.1))
+    (fp_line (start 0.635 -1.27) (end 1.27 -0.635) (layer "F.Fab") (width 0.1))
+    (fp_line (start -1.27 -1.27) (end 0.635 -1.27) (layer "F.Fab") (width 0.1))
+    (fp_line (start 1.27 6.35) (end -1.27 6.35) (layer "F.Fab") (width 0.1))
+    (pad "1" thru_hole rect (at 0 0) (size 1.7 1.7) (drill 1) (layers *.Cu *.Mask)
+      (net 1 "GND") (pinfunction "Pin_1") (pintype "passive"))
+    (pad "2" thru_hole oval (at 0 2.54) (size 1.7 1.7) (drill 1) (layers *.Cu *.Mask)
+      (net 5 "/LPF/OUT-LPF") (pinfunction "Pin_2") (pintype "passive"))
+    (pad "3" thru_hole oval (at 0 5.08) (size 1.7 1.7) (drill 1) (layers *.Cu *.Mask)
+      (net 1 "GND") (pinfunction "Pin_3") (pintype "passive"))
+    (model "${KICAD6_3DMODEL_DIR}/Connector_PinSocket_2.54mm.3dshapes/PinSocket_1x03_P2.54mm_Vertical.wrl"
+      (offset (xyz 0 0 0))
+      (scale (xyz 1 1 1))
+      (rotate (xyz 0 0 0))
+    )
+  )
   (footprint "Relay_THT:Relay_DPDT_Omron_G6S-2" (layer "F.Cu")

Commit message: fixed decoder
Connections:
- C12 pad 2: Detector-0 -> Detector-90
- C13 pad 2: Detector-0 -> Detector-180
- C14 pad 2: Detector-0 -> Detector-270
- R2 pad 1: Detector-0 -> Detector-90
- R3 pad 1: Detector-0 -> Detector-180
- R4 pad 1: Detector-0 -> Detector-270
- U1 pad 11: Detector-0 -> Detector-90
- U1 pad 12: Detector-0 -> Detector-270
- U1 pad 13: Detector-0 -> Detector-180
- U1 pad 4: Detector-0 -> Detector-90
- U1 pad 5: Detector-0 -> Detector-270
- U1 pad 6: Detector-0 -> Detector-180
Changed lines of the file:
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@@
   (net 116 "/RF Switch/To-Det")
   (net 117 "/RF Switch/From-Enc")
+  (net 118 "Detector-90")
+  (net 119 "Detector-180")
+  (net 120 "Detector-270")
   (footprint "Capacitor_SMD:C_1206_3216Metric" (layer "F.Cu")
     (at 112.44 103.33)
@@
       (net 38 "Detector-0") (pinfunction "1B4") (pintype "output") (solder_mask_margin 0.1016))
     (pad "4" smd rect locked (at 0.115 8.55) (size 0.6 1.2) (layers "F.Cu" "F.Paste" "F.Mask")
-      (net 38 "Detector-0") (pinfunction "1B3") (pintype "output") (solder_mask_margin 0.1016))
+      (net 118 "Detector-90") (pinfunction "1B3") (pintype "output") (solder_mask_margin 0.1016))
     (pad "5" smd rect locked (at 1.385 8.55) (size 0.6 1.2) (layers "F.Cu" "F.Paste" "F.Mask")
-      (net 38 "Detector-0") (pinfunction "1B2") (pintype "input") (solder_mask_margin 0.1016))
+      (net 120 "Detector-270") (pinfunction "1B2") (pintype "input") (solder_mask_margin 0.1016))
     (pad "6" smd rect locked (at 2.655 8.55) (size 0.6 1.2) (layers "F.Cu" "F.Paste" "F.Mask")
-      (net 38 "Detector-0") (pinfunction "1B1") (pintype "input") (solder_mask_margin 0.1016))
+      (net 119 "Detector-180") (pinfunction "1B1") (pintype "input") (solder_mask_margin 0.1016))
     (pad "7" smd rect locked (at 3.925 8.55) (size 0.6 1.2) (layers "F.Cu" "F.Paste" "F.Mask")
       (net 29 "Net-(T3-PadC2B)") (pinfunction "1A") (pintype "bidirectional") (solder_mask_margin 0.1016))
@@
       (net 38 "Detector-0") (pinfunction "2B1") (pintype "output") (solder_mask_margin 0.1016))
     (pad "11" smd rect locked (at 2.655 2.95) (size 0.6 1.2) (layers "F.Cu" "F.Paste" "F.Mask")
-      (net 38 "Detector-0") (pinfunction "2B2") (pintype "output") (solder_mask_margin 0.1016))
+      (net 118 "Detector-90") (pinfunction "2B2") (pintype "output") (solder_mask_margin 0.1016))
     (pad "12" smd rect locked (at 1.385 2.95) (size 0.6 1.2) (layers "F.Cu" "F.Paste" "F.Mask")
-      (net 38 "Detector-0") (pinfunction "2B3") (pintype "input") (solder_mask_margin 0.1016))
+      (net 120 "Detector-270") (pinfunction "2B3") (pintype "input") (solder_mask_margin 0.1016))
     (pad "13" smd rect locked (at 0.115 2.95) (size 0.6 1.2) (layers "F.Cu" "F.Paste" "F.Mask")
-      (net 38 "Detector-0") (pinfunction "2B4") (pintype "input") (solder_mask_margin 0.1016))
+      (net 119 "Detector-180") (pinfunction "2B4") (pintype "input") (solder_mask_margin 0.1016))
     (pad "14" smd rect locked (at -1.155 2.95) (size 0.6 1.2) (layers "F.Cu" "F.Paste" "F.Mask")
       (net 33 "LO-90") (pinfunction "S0") (pintype "bidirectional") (solder_mask_margin 0.1016))
@@
     (fp_line (start -1 -0.625) (end 1 -0.625) (layer "F.Fab") (width 0.1))
     (pad "1" smd roundrect (at -0.9125 0) (size 1.025 1.4) (layers "F.Cu" "F.Paste" "F.Mask") (roundrect_rratio 0.243902)
-      (net 38 "Detector-0") (pinfunction "1") (pintype "passive"))
+      (net 118 "Detector-90") (pinfunction "1") (pintype "passive"))
     (pad "2" smd roundrect (at 0.9125 0) (size 1.025 1.4) (layers "F.Cu" "F.Paste" "F.Mask") (roundrect_rratio 0.243902)
       (net 30 "Net-(C16-Pad1)") (pinfunction "2") (pintype "passive"))
@@
       (net 1 "GND") (pintype "passive"))
     (pad "2" smd roundrect (at 1.475 0) (size 1.15 1.8) (layers "F.Cu" "F.Paste" "F.Mask") (roundrect_rratio 0.217391)
-      (net 38 "Detector-0") (pintype "passive"))
+      (net 120 "Detector-270") (pintype "passive"))
     (model "${KICAD6_3DMODEL_DIR}/Capacitor_SMD.3dshapes/C_1206_3216Metric.wrl"
       (offset (xyz 0 0 0))
@@
       (net 1 "GND") (pintype "passive"))
     (pad "2" smd roundrect (at 1.475 0) (size 1.15 1.8) (layers "F.Cu" "F.Paste" "F.Mask") (roundrect_rratio 0.217391)
-      (net 38 "Detector-0") (pintype "passive"))
+      (net 118 "Detector-90") (pintype "passive"))
     (model "${KICAD6_3DMODEL_DIR}/Capacitor_SMD.3dshapes/C_1206_3216Metric.wrl"
       (offset (xyz 0 0 0))
@@
     (fp_line (start -1 0.625) (end -1 -0.625) (layer "F.Fab") (width 0.1))
     (pad "1" smd roundrect (at -0.9125 0) (size 1.025 1.4) (layers "F.Cu" "F.Paste" "F.Mask") (roundrect_rratio 0.243902)
-      (net 38 "Detector-0") (pinfunction "1") (pintype "passive"))
+      (net 120 "Detector-270") (pinfunction "1") (pintype "passive"))
     (pad "2" smd roundrect (at 0.9125 0) (size 1.025 1.4) (layers "F.Cu" "F.Paste" "F.Mask") (roundrect_rratio 0.243902)
       (net 26 "Net-(R4-Pad2)") (pinfunction "2") (pintype "passive"))
@@
       (net 1 "GND") (pintype "passive"))
     (pad "2" smd roundrect (at 1.475 0) (size 1.15 1.8) (layers "F.Cu" "F.Paste" "F.Mask") (roundrect_rratio 0.217391)
-      (net 38 "Detector-0") (pintype "passive"))
+      (net 119 "Detector-180") (pintype "passive"))
     (model "${KICAD6_3DMODEL_DIR}/Capacitor_SMD.3dshapes/C_1206_3216Metric.wrl"
       (offset (xyz 0 0 0))
@@
     (fp_line (start -1 -0.625) (end 1 -0.625) (layer "F.Fab") (width 0.1))
     (pad "1" smd roundrect (at -0.9125 0) (size 1.025 1.4) (layers "F.Cu" "F.Paste" "F.Mask") (roundrect_rratio 0.243902)
-      (net 38 "Detector-0") (pinfunction "1") (pintype "passive"))
+      (net 119 "Detector-180") (pinfunction "1") (pintype "passive"))
     (pad "2" smd roundrect (at 0.9125 0) (size 1.025 1.4) (layers "F.Cu" "F.Paste" "F.Mask") (roundrect_rratio 0.243902)
       (net 25 "Net-(R3-Pad2)") (pinfunction "2") (pintype "passive"))

Commit message: gg
Parts:
- moved J1 2.85 mm to (209.0, 121.4)
Connections:
- net Net-(J1-PadS) renamed /RF Switch/Antenna

Commit message: added relay fet
Parts:
- added Q1: AO3400A, Package_TO_SOT_SMD:SOT-23, F.Cu at (91.4, 114.9)
- added R31: 1k, Resistor_SMD:R_0805_2012Metric, F.Cu at (86.1, 114.2)
Connections:
- D1 pad 1: Net-(D1-Pad1) -> +12V
- D1 pad 2: Net-(D1-Pad2) -> RELAY-ON
- D2 pad 1: Net-(D2-Pad1) -> +12V
- D2 pad 2: Net-(D2-Pad2) -> RELAY-ON
- K1 pad 1: Net-(D1-Pad1) -> +12V
- K1 pad 12: Net-(D1-Pad2) -> RELAY-ON
- K2 pad 1: Net-(D2-Pad1) -> +12V
- K2 pad 12: Net-(D2-Pad2) -> RELAY-ON

Commit message: added pa
Parts:
- added J6: PCB_SMA_EDGE, Xenir_V6:pcb-sma-edge, F.Cu at (213.4, 148.1)
- added J7: PCB_SMA_EDGE, Xenir_V6:pcb-sma-edge, F.Cu at (220.2, 148.1)
- added J8: Audio_Jack, Xenir:Audio_Jack, F.Cu at (245.6, 153.7)
- added J8: Conn_01x01_Female, Connector_PinSocket_2.54mm:PinSocket_1x01_P2.54mm_Vertical, F.Cu at (226.3, 142.2)
- added Q2: AO3400A, Package_TO_SOT_SMD:SOT-23, F.Cu at (225.9, 149.6)
- added R32: 1k, Resistor_SMD:R_0805_2012Metric, F.Cu at (225.7, 153.3)

Commit message: updated PA
Parts:
- removed C4: 270Pf, Capacitor_SMD:C_1206_3216Metric
- removed C5, C8: 90pF, Capacitor_SMD:C_1206_3216Metric
- removed C6: N/C, Capacitor_SMD:C_1206_3216Metric
- removed C7: 12pF, Capacitor_SMD:C_1206_3216Metric
- removed L2, L3: T37-6, Xenir:T37_Inductor
- removed T1: T37-6 5:25, Xenir:T37 Transformer
- removed T2: T37-6 25:5, Xenir:T37 Transformer
- removed VC1, VC2: 1-40pF, Xenir:trimcap
- added Q3: 2N2222, Package_TO_SOT_SMD:SOT-23, F.Cu at (243.7, 33.5)
- added R33: 2.2k, Resistor_SMD:R_0805_2012Metric, F.Cu at (239.3, 26.8)
- added R34: 475, Resistor_SMD:R_0805_2012Metric, F.Cu at (239.3, 30.5)
- added R35: 56, Resistor_SMD:R_0805_2012Metric, F.Cu at (243.2, 40.1)
- added R36: 50, Resistor_SMD:R_0805_2012Metric, F.Cu at (243.2, 37.6)
- C1: value 270pF -> .1uF; footprint Capacitor_SMD:C_1206_3216Metric -> Capacitor_SMD:C_0805_2012Metric
- C2: value 470pF -> 10nF; footprint Capacitor_SMD:C_1206_3216Metric -> Capacitor_SMD:C_0805_2012Metric
- C3: value 470pF -> .1uF; footprint Capacitor_SMD:C_1206_3216Metric -> Capacitor_SMD:C_0805_2012Metric
- J6: value PCB_SMA_EDGE -> TO-PA
- J7: value PCB_SMA_EDGE -> FROM-PA
- L1: value T37-6 -> BN43-2402 6T; footprint Xenir:T37_Inductor -> Xenir:BN-43-2402
- moved J6 126.9 mm to (255.9, 28.5)
- moved R32 101.1 mm to (244.8, 53.9)
- moved J7 101.1 mm to (239.3, 48.8)
- moved J8 101.1 mm to (264.7, 54.4)
- moved Q2 101.1 mm to (245.0, 50.2)
- moved J8 99.5 mm to (254.3, 46.7)
- moved C1 90.7 mm to (236.5, 30.5), turned to 90 degrees
- moved C2 88.3 mm to (246.6, 39.0), turned to 90 degrees
- moved C3 85.7 mm to (248.3, 33.8)
- moved L1 80.2 mm to (244.6, 31.9), turned to 180 degrees
Connections:
- C1 pad 1: GND -> /PA/PA-IN
- C1 pad 2: /LPF/IN-LPF -> Net-(C1-Pad2)
- C3 pad 1: GND -> Net-(C3-Pad1)
- J6 pad 1: /PA/PA-IN -> Net-(C3-Pad2)
- J8 pad TIP: Net-(Q2-Pad3) -> Net-(J8-PadTIP)
- J8 pad TSH: Net-(Q2-Pad3) -> Net-(J8-PadTIP)
- L1 pad 1: /LPF/IN-LPF -> Net-(C3-Pad1)
- L1 pad 2: Net-(C2-Pad2) -> +12V
- Q2 pad 3: Net-(Q2-Pad3) -> Net-(J8-PadTIP)

Commit message: added cap
Parts:
- added C4: .1uF, Capacitor_SMD:C_0805_2012Metric, F.Cu at (248.9, 26.7)
Changed lines of the file:
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@@
+    )
+  )
+  (footprint "Capacitor_SMD:C_0805_2012Metric" (layer "F.Cu")
+    (at 248.92 26.67 90)
+    (descr "Capacitor SMD 0805 (2012 Metric), square (rectangular) end terminal, IPC_7351 nominal, (Body size source: IPC-SM-782 page 76, https://www.pcb-3d.com/wordpress/wp-content/uploads/ipc-sm-782a_amendment_1_and_2.pdf, https://docs.google.com/spreadsheets/d/1BsfQQcO9C6DZCsRaXUlFlo91Tg2WpOkGARC1WS5S8t0/edit?usp=sharing), generated with kicad-footprint-generator")
+    (tags "capacitor")
+    (property "Sheetfile" "PA.kicad_sch")
+    (property "Sheetname" "PA")
+    (attr smd)
+    (fp_text reference "C4" (at 0 -1.68 90) (layer "F.SilkS")
+      (effects (font (size 1 1) (thickness 0.15)))
+    )
+    (fp_text value ".1uF" (at 0 1.68 90) (layer "F.Fab")
+      (effects (font (size 1 1) (thickness 0.15)))
+    )
+    (fp_text user "${REFERENCE}" (at 0 0 90) (layer "F.Fab")
+      (effects (font (size 0.5 0.5) (thickness 0.08)))
+    )
+    (fp_line (start -0.261252 0.735) (end 0.261252 0.735) (layer "F.SilkS") (width 0.12))
+    (fp_line (start -0.261252 -0.735) (end 0.261252 -0.735) (layer "F.SilkS") (width 0.12))
+    (fp_line (start -1.7 0.98) (end -1.7 -0.98) (layer "F.CrtYd") (width 0.05))
+    (fp_line (start 1.7 0.98) (end -1.7 0.98) (layer "F.CrtYd") (width 0.05))
+    (fp_line (start -1.7 -0.98) (end 1.7 -0.98) (layer "F.CrtYd") (width 0.05))
+    (fp_line (start 1.7 -0.98) (end 1.7 0.98) (layer "F.CrtYd") (width 0.05))
+    (fp_line (start 1 0.625) (end -1 0.625) (layer "F.Fab") (width 0.1))
+    (fp_line (start 1 -0.625) (end 1 0.625) (layer "F.Fab") (width 0.1))
+    (fp_line (start -1 0.625) (end -1 -0.625) (layer "F.Fab") (width 0.1))
+    (fp_line (start -1 -0.625) (end 1 -0.625) (layer "F.Fab") (width 0.1))
+    (pad "1" smd roundrect (at -0.95 0 90) (size 1 1.45) (layers "F.Cu" "F.Paste" "F.Mask") (roundrect_rratio 0.25)
+      (net 1 "GND") (pintype "passive"))
+    (pad "2" smd roundrect (at 0.95 0 90) (size 1 1.45) (layers "F.Cu" "F.Paste" "F.Mask") (roundrect_rratio 0.25)
+      (net 15 "+12V") (pintype "passive"))
+    (model "${KICAD6_3DMODEL_DIR}/Capacitor_SMD.3dshapes/C_0805_2012Metric.wrl"
+      (offset (xyz 0 0 0))
+      (scale (xyz 1 1 1))
+      (rotate (xyz 0 0 0))
     )
   )

Commit message: gg
Parts:
- added R37: 50, Resistor_SMD:R_0805_2012Metric, F.Cu at (237.2, 33.5)
- added TP1: TestPoint, TestPoint:TestPoint_THTPad_1.0x1.0mm_Drill0.5mm, F.Cu at (250.4, 32.5)
- moved C2 2.50 mm to (245.6, 36.8)
- moved C3 2.18 mm to (246.6, 32.5)
- moved R35 2.05 mm to (242.4, 38.2)
- moved R36 2.05 mm to (242.4, 35.7)
- moved Q3 1.44 mm to (242.6, 32.5)
- moved J6 1.27 mm to (255.9, 27.2)
- moved C4 0.95 mm to (248.2, 26.1)
Routing:
- net Net-(C3-Pad2): track 0.00 -> 8.58 mm
- net Net-(Q3-Pad2): track 0.00 -> 4.85 mm
- net Net-(C1-Pad2): track 0.00 -> 4.69 mm
- net +12V: track 0.00 -> 3.74 mm
- net /PA/PA-IN: track 0.00 -> 2.16 mm
- net Net-(C2-Pad2): track 0.00 -> 2.03 mm
- net Net-(C3-Pad1): track 0.00 -> 2.03 mm
