File: SDR-Transceiver.kicad_pcb (KiCad board)
At the start: 2 copper layers, 110 parts, among them J1 BNC, J2 Conn_01x03_Female, J3 Conn_01x03_Female, J4 Conn_01x03_Female, J5 Conn_01x03_Female, J6 TO-PA, J7 FROM-PA, J8 Audio_Jack, J8 Conn_01x01_Female, K1 G6S-2, K2 G6S-2, Q1 AO3400A, Q2 AO3400A, Q3 2N2222, T3 T50_SPLITTER, T4 T50_SPLITTER, U1 FST3253, U2 LM4562, U3 FST3253, U4 LM4562, U5 LM4562, U6 ESP32-A1S, U7 FST3257

Commit message: added caps in encoder
Parts:
- added C5: 10uF, Capacitor_SMD:CP_Elec_4x4.5, F.Cu at (117.7, 163.1)
- added C6: 10uF, Capacitor_SMD:CP_Elec_4x4.5, F.Cu at (125.5, 168.9)
- added C7: 10uF, Capacitor_SMD:CP_Elec_4x4.5, F.Cu at (125.5, 163.1)
- added C8: 10uF, Capacitor_SMD:CP_Elec_4x4.5, F.Cu at (117.7, 168.9)
- moved R18 30.3 mm to (100.8, 168.7)
- moved C23 30.3 mm to (97.0, 162.6)
- moved R14 30.3 mm to (96.4, 168.7)
- moved R16 30.3 mm to (105.2, 165.3)
- moved R17 30.3 mm to (100.8, 165.7)
- moved U5 30.3 mm to (90.9, 161.6)
- moved R13 30.3 mm to (102.1, 162.4)
- moved R15 30.3 mm to (96.4, 165.7)
- moved R8 27.6 mm to (94.7, 141.2)
- moved C20 27.6 mm to (84.0, 141.4)
- moved C21 27.6 mm to (89.7, 141.4)
- moved C22 27.6 mm to (84.0, 144.7)
- moved R10 27.6 mm to (83.4, 147.9)
- moved R19 27.6 mm to (93.5, 144.5)
- moved R20 27.6 mm to (87.8, 147.9)
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Connections:
- R18 pad 2: Net-(R10-Pad1) -> Net-(R18-Pad2)
- R7 pad 1: Net-(R11-Pad2) -> Net-(R7-Pad1)
- R8 pad 1: Net-(R12-Pad2) -> Net-(R8-Pad1)
- R9 pad 1: Net-(R15-Pad2) -> Net-(R9-Pad1)
- U5 pad 7: Net-(R10-Pad1) -> Net-(R18-Pad2)

Commit message: gg
Parts:
- moved Q1 73.2 mm to (158.3, 85.1)
- moved R31 73.2 mm to (152.9, 84.3)
- moved J1 35.3 mm to (182.5, 98.1)
- moved K2 21.5 mm to (162.9, 90.3)
- moved D1 21.5 mm to (146.1, 86.1)
- moved D2 21.5 mm to (165.6, 86.1)
- moved K1 21.5 mm to (143.8, 90.2)
Routing:
- net RELAY-ON: track 0.00 -> 33.0 mm
- net Net-(K1-Pad10): track 0.00 -> 19.2 mm
- net /RF Switch/Antenna: track 0.00 -> 15.7 mm
- net +12V: track 3.74 -> 12.7 mm
- net /LPF/OUT-LPF: track 0.00 -> 5.08 mm
- net Net-(Q1-Pad1): track 0.00 -> 3.59 mm
Changed lines of the file:
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@@
   )
   (footprint "Package_TO_SOT_SMD:SOT-23" (layer "F.Cu")
-    (at 91.44 114.935)
+    (at 158.2655 85.078)
     (descr "SOT, 3 Pin (https://www.jedec.org/system/files/docs/to-236h.pdf variant AB), generated with kicad-footprint-generator ipc_gullwing_generator.py")
     (tags "SOT TO_SOT_SMD")
@@
   )
   (footprint "Resistor_SMD:R_0805_2012Metric" (layer "F.Cu")
-    (at 86.0825 114.185)
+    (at 152.908 84.328)
     (descr "Resistor SMD 0805 (2012 Metric), square (rectangular) end terminal, IPC_7351 nominal, (Body size source: IPC-SM-782 page 72, https://www.pcb-3d.com/wordpress/wp-content/uploads/ipc-sm-782a_amendment_1_and_2.pdf), generated with kicad-footprint-generator")
     (tags "resistor")
@@
   )
   (footprint "Relay_THT:Relay_DPDT_Omron_G6S-2" (layer "F.Cu")
-    (at 146.304 111.506)
+    (at 143.764 90.17)
     (descr "Relay Omron G6S-2, see http://omronfs.omron.com/en_US/ecb/products/pdf/en-g6s.pdf")
     (tags "Relay Omron G6S-2")
@@
   )
   (footprint "Diode_SMD:D_SOD-123" (layer "F.Cu")
-    (at 168.148 107.442)
+    (at 165.608 86.106)
     (descr "SOD-123")
     (tags "SOD-123")
@@
   )
   (footprint "Relay_THT:Relay_DPDT_Omron_G6S-2" (layer "F.Cu")
-    (at 165.4865 111.6485)
+    (at 162.9465 90.3125)
     (descr "Relay Omron G6S-2, see http://omronfs.omron.com/en_US/ecb/products/pdf/en-g6s.pdf")
     (tags "Relay Omron G6S-2")
@@
   )
   (footprint "Xenir:BNC" (layer "F.Cu")
-    (at 209.005 121.385 -90)
+    (at 182.462 98.144 -90)
     (property "Sheetfile" "SDR-Transceiver.kicad_sch")
     (property "Sheetname" "")
@@
   )
   (footprint "Diode_SMD:D_SOD-123" (layer "F.Cu")
-    (at 148.59 107.442)
+    (at 146.05 86.106)
     (descr "SOD-123")
     (tags "SOD-123")
@@
   (segment (start 255.76251 32.512) (end 255.88227 32.39224) (width 0.5) (layer "F.Cu") (net 4))
   (segment (start 247.518 32.512) (end 255.76251 32.512) (width 0.5) (layer "F.Cu") (net 4))
+  (segment (start 168.0265 100.4725) (end 162.9465 100.4725) (width 1) (layer "F.Cu") (net 5))
+  (segment (start 159.524 85.078) (end 160.528 84.074) (width 0.5) (layer "F.Cu") (net 6))
+  (segment (start 159.203 85.078) (end 159.203 87.939) (width 0.5) (layer "F.Cu") (net 6))
+  (segment (start 150.622 88.392) (end 148.844 90.17) (width 0.5) (layer "F.Cu") (net 6))
+  (segment (start 167.258 85.216) (end 167.258 86.106) (width 0.5) (layer "F.Cu") (net 6))
+  (segment (start 167.258 86.106) (end 167.258 89.544) (width 0.5) (layer "F.Cu") (net 6))
+  (segment (start 159.203 87.939) (end 158.75 88.392) (width 0.5) (layer "F.Cu") (net 6))
+  (segment (start 160.528 84.074) (end 166.116 84.074) (width 0.5) (layer "F.Cu") (net 6))
+  (segment (start 159.203 85.078) (end 159.524 85.078) (width 0.5) (layer "F.Cu") (net 6))
+  (segment (start 166.116 84.074) (end 167.258 85.216) (width 0.5) (layer "F.Cu") (net 6))
+  (segment (start 158.75 88.392) (end 150.622 88.392) (width 0.5) (layer "F.Cu") (net 6))
+  (segment (start 147.7 86.106) (end 147.7 89.026) (width 0.5) (layer "F.Cu") (net 6))
+  (segment (start 147.7 89.026) (end 148.844 90.17) (width 0.5) (layer "F.Cu") (net 6))
+  (segment (start 167.258 89.544) (end 168.0265 90.3125) (width 0.5) (layer "F.Cu") (net 6))
+  (segment (start 153.8205 84.328) (end 157.128 84.328) (width 0.5) (layer "F.Cu") (net 7))
+  (segment (start 157.128 84.328) (end 157.328 84.128) (width 0.5) (layer "F.Cu") (net 7))
   (segment (start 236.3235 31.5805) (end 236.474 31.43) (width 0.5) (layer "F.Cu") (net 11))
   (segment (start 236.3235 33.528) (end 236.3235 31.5805) (width 0.5) (layer "F.Cu") (net 11))
+  (segment (start 148.9865 95.3925) (end 148.844 95.25) (width 1) (layer "F.Cu") (net 13))
+  (segment (start 168.0265 95.3925) (end 162.9465 95.3925) (width 1) (layer "F.Cu") (net 13))
+  (segment (start 162.9465 95.3925) (end 148.9865 95.3925) (width 1) (layer "F.Cu") (net 13))
   (segment (start 244.602 25.146) (end 248.346 25.146) (width 0.5) (layer "F.Cu") (net 15))
+  (segment (start 144.4 86.106) (end 144.4 89.534) (width 0.5) (layer "F.Cu") (net 15))
+  (segment (start 163.958 89.301) (end 162.9465 90.3125) (width 0.5) (layer "F.Cu") (net 15))
+  (segment (start 163.958 86.106) (end 163.958 89.301) (width 0.5) (layer "F.Cu") (net 15))
+  (segment (start 144.4 89.534) (end 143.764 90.17) (width 0.5) (layer "F.Cu") (net 15))
+  (segment (start 168.0265 97.9325) (end 178.4505 97.9325) (width 1) (layer "F.Cu") (net 115))
+  (segment (start 168.0265 97.9325) (end 162.9465 97.9325) (width 1) (layer "F.Cu") (net 115))
+  (segment (start 178.4505 97.9325) (end 178.562 98.044) (width 1) (layer "F.Cu") (net 115))
   (segment (start 239.2305 29.53) (end 239.268 29.5675) (width 0.5) (layer "F.Cu") (net 120))
   (segment (start 239.268 27.686) (end 239.268 29.5675) (width 0.5) (layer "F.Cu") (net 120))

Commit message: gg
Routing:
- net +12V: track 12.7 -> 18.3 mm
- net Net-(C3-Pad1): track 2.03 -> 7.02 mm
Changed lines of the file:
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@@
   (segment (start 168.0265 95.3925) (end 162.9465 95.3925) (width 1) (layer "F.Cu") (net 13))
   (segment (start 162.9465 95.3925) (end 148.9865 95.3925) (width 1) (layer "F.Cu") (net 13))
+  (segment (start 239.268 25.861) (end 239.983 25.146) (width 0.5) (layer "F.Cu") (net 15))
   (segment (start 244.602 25.146) (end 248.346 25.146) (width 0.5) (layer "F.Cu") (net 15))
   (segment (start 144.4 86.106) (end 144.4 89.534) (width 0.5) (layer "F.Cu") (net 15))
+  (segment (start 239.983 25.146) (end 244.602 25.146) (width 0.5) (layer "F.Cu") (net 15))
   (segment (start 163.958 89.301) (end 162.9465 90.3125) (width 0.5) (layer "F.Cu") (net 15))
   (segment (start 163.958 86.106) (end 163.958 89.301) (width 0.5) (layer "F.Cu") (net 15))
@@
   (segment (start 236.474 29.53) (end 239.2305 29.53) (width 0.5) (layer "F.Cu") (net 120))
   (segment (start 243.586 32.512) (end 245.618 32.512) (width 0.5) (layer "F.Cu") (net 121))
+  (segment (start 243.586 31.496) (end 243.586 32.512) (width 0.5) (layer "F.Cu") (net 121))
+  (segment (start 244.602 30.48) (end 243.586 31.496) (width 0.5) (layer "F.Cu") (net 121))
+  (segment (start 244.602 27.94) (end 244.602 30.48) (width 0.5) (layer "F.Cu") (net 121))
   (segment (start 241.507 35.692) (end 241.507 38.232) (width 0.5) (layer "F.Cu") (net 123))
   (segment (start 241.711 35.488) (end 241.507 35.692) (width 0.5) (layer "F.Cu") (net 123))

Commit message: added output resistors to switch
Parts:
- added R38: 47k, Resistor_SMD:R_0805_2012Metric, F.Cu at (62.7, 186.4)
- added R39: 47k, Resistor_SMD:R_0805_2012Metric, F.Cu at (58.3, 186.4)
- added R40: 47k, Resistor_SMD:R_0805_2012Metric, F.Cu at (62.7, 183.5)
- added R41: 47k, Resistor_SMD:R_0805_2012Metric, F.Cu at (58.3, 183.5)
- C30, C31, C32, C33, C34, C35, C36, C37, C39, C40, C41, C42: value .1uF -> 1uF
Connections:
- C15 pad 2: /Audio Switch/INR2 -> /Audio Switch/INR1
- C16 pad 2: /Audio Switch/INL2 -> /Audio Switch/INL1
- C32 pad 1: /Audio Switch/INL1 -> /Audio Switch/INR1
- C33 pad 1: /Audio Switch/INR2 -> /Audio Switch/INL2
- C34 pad 1: /Audio Amp/AUDIO-AMP-IN -> /Audio Switch/OUTR2
- C37 pad 1: /Audio Switch/OUTL1 -> /Audio Amp/AUDIO-AMP-IN
- R13 pad 1: /Audio Switch/OUTL1 -> /Audio Switch/OUTL2
- R14 pad 1: /Audio Switch/OUTR1 -> /Audio Switch/OUTR2
- R5 pad 2: /Audio Switch/INR2 -> /Audio Switch/INR1
- R6 pad 2: /Audio Switch/INL2 -> /Audio Switch/INL1
- U2 pad 1: /Audio Switch/INR2 -> /Audio Switch/INR1
- U2 pad 7: /Audio Switch/INL2 -> /Audio Switch/INL1

Commit message: added power supply
Parts:
- added C43: 100uF, Capacitor_SMD:CP_Elec_6.3x5.4, F.Cu at (259.3, 103.1)
- added C44: 22uF, Capacitor_SMD:CP_Elec_4x5.4, F.Cu at (242.1, 98.0)
- added C45: .1uF, Xenir:Capacitor 0805, F.Cu at (248.2, 93.9)
- added C46: 22uF, Capacitor_SMD:CP_Elec_4x5.4, F.Cu at (230.9, 98.1)
- added C47: .1uF, Xenir:Capacitor 0805, F.Cu at (235.2, 110.2)
- added J9: Barrel_Jack_Switch, Xenir:BarrelJack_Horizontal, F.Cu at (268.0, 100.3)
- added R42: Resistor, Resistor_SMD:R_0805_2012Metric, F.Cu at (236.6, 99.8)
- added R43: Resistor, Resistor_SMD:R_0805_2012Metric, F.Cu at (236.6, 96.8)
- added U8: L7805, Package_TO_SOT_SMD:TO-252-3_TabPin2, F.Cu at (249.4, 104.4)
- added U9: AMS1117CD-3.3, Package_TO_SOT_SMD:SOT-223-3_TabPin2, F.Cu at (239.8, 108.2)

Commit message: updated DSP
Parts:
- added J10: Conn_01x07_Female, Connector_PinSocket_2.54mm:PinSocket_1x07_P2.54mm_Vertical, F.Cu at (22.1, 68.3)
- added J11: Conn_01x04, Connector_PinSocket_2.54mm:PinSocket_1x04_P2.54mm_Vertical, F.Cu at (63.8, 68.3)
- added Q4: 2N3904-SMD, Package_TO_SOT_SMD:SOT-23, F.Cu at (63.9, 80.5)
- added Q5: 2N3904-SMD, Package_TO_SOT_SMD:SOT-23, F.Cu at (37.4, 83.5)
- added Q6: AO3400A, Package_TO_SOT_SMD:SOT-23, F.Cu at (42.3, 83.5)
- added R44: 10k, Resistor_SMD:R_0805_2012Metric, F.Cu at (22.0, 90.3)
- added R45: 10k, Resistor_SMD:R_0805_2012Metric, F.Cu at (37.1, 87.2)
- added R46: 1k, Resistor_SMD:R_0805_2012Metric, F.Cu at (26.4, 91.3)
- added R47: 10k, Resistor_SMD:R_0805_2012Metric, F.Cu at (22.0, 87.3)
- added SW1: SW_DIP_x01, Button_Switch_THT:SW_PUSH_6mm, F.Cu at (26.4, 83.3)
- added SW2: Frequency, Rotary_Encoder:RotaryEncoder_Alps_EC11E-Switch_Vertical_H20mm, F.Cu at (44.9, 71.1)
- added SW3: Menu, Rotary_Encoder:RotaryEncoder_Alps_EC11E-Switch_Vertical_H20mm, F.Cu at (26.4, 71.1)
Connections:
- U6 pad 31: /DSP/SDA -> SDA
- U6 pad 32: /DSP/SCL -> SCL
- U6 pad 33: T/R -> unconnected-(U6-Pad33)
- U6 pad 34: unconnected-(U6-Pad34) -> GPIO21
- U6 pad 35: unconnected-(U6-Pad35) -> EN
- U6 pad 36: unconnected-(U6-Pad36) -> RX0
- U6 pad 37: unconnected-(U6-Pad37) -> TX0
- U6 pad 7: unconnected-(U6-Pad7) -> GPIO14
- U6 pad 8: unconnected-(U6-Pad8) -> GPIO12
- U6 pad 9: unconnected-(U6-Pad9) -> GPIO13

Commit message: Update SDR-Transceiver.kicad_pcb
Connections:
- SW2 pad S2: GPIO13 -> GPIO12
- U6 pad 10: unconnected-(U6-Pad10) -> GPIO15
- U6 pad 12: unconnected-(U6-Pad12) -> GPIO4
- U6 pad 5: unconnected-(U6-Pad5) -> GPIO34

Commit message: added LO
Parts:
- added U10: si5351, Xenir:si5351, F.Cu at (25.7, 47.2)
Connections:
- U6 pad 1: unconnected-(U6-Pad1) -> GND
- U6 pad 19: unconnected-(U6-Pad19) -> GND
- U6 pad 2: unconnected-(U6-Pad2) -> +3V3
- U6 pad 20: unconnected-(U6-Pad20) -> GND
- U6 pad 38: unconnected-(U6-Pad38) -> GND
