File: SDR-Transceiver.kicad_pcb (KiCad board)
At the start: 2 copper layers, 139 parts, among them J1 BNC, J10 Conn_01x07_Female, J11 Conn_01x04, J2 IN-BPF, J3 OUT-LPF, J4 IN-LPF, J5 OUT-LPF, J6 TO-PA, J7 FROM-PA, J8 Amplifier T/R, J8 Conn_01x01_Female, J9 Barrel_Jack_Switch, K1 G6S-2, K2 G6S-2, Q1 AO3400A, Q2 AO3400A, Q3 2N2222, Q4 2N3904-SMD, Q5 2N3904-SMD, Q6 AO3400A, SW1 SW_DIP_x01, SW2 Frequency, SW3 Menu, T3 T50_SPLITTER, T4 T50_COMBINER, U1 FST3253, U10 si5351, U2 LM4562, U3 FST3253, U4 LM4562, U5 LM4562, U6 ESP32-A1S, U7 FST3257, U8 L7805, U9 AMS1117CD-3.3

Commit message: gg
Parts:
- moved C33 98.9 mm to (105.6, 91.9)
- moved C34 98.9 mm to (119.3, 92.7)
- moved C35 98.9 mm to (123.0, 91.9)
- moved C38 98.9 mm to (113.2, 80.3)
- moved R39 98.9 mm to (126.4, 92.6)
- moved C37 98.9 mm to (124.0, 82.8)
- moved C40 98.9 mm to (105.0, 95.9)
- moved C41 98.9 mm to (120.3, 96.7)
- moved R25 98.9 mm to (108.2, 96.8)
- moved R26 98.9 mm to (108.2, 94.5)
- moved R27 98.9 mm to (116.9, 95.2)
- moved R28 98.9 mm to (116.9, 97.5)
- moved R38 98.9 mm to (123.6, 96.7)
- moved R40 98.9 mm to (127.4, 85.7)
- moved U7 98.9 mm to (118.9, 87.4)
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
Commit message: gg
Parts:
- moved R28 2.16 mm to (114.7, 97.5)
- moved C41 2.02 mm to (118.4, 97.5), turned to 0 degrees
- moved R38 1.57 mm to (123.2, 95.1)
Routing:
- net +5V: track 22.3 -> 86.5 mm, vias 2 -> 5
- net Detector-0: track 20.6 -> 35.0 mm, vias 2 -> 3
- net GND: track 1.59 -> 5.74 mm, vias 1 -> 3
- net /Audio Switch/OUTR2: track 0.00 -> 3.77 mm
- net Net-(C41-Pad1): track 8.26 -> 6.97 mm

Commit message: hh
Parts:
- moved C24 13.1 mm to (82.5, 180.3)
Changed lines of the file:
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@@
   )
   (footprint "Capacitor_SMD:CP_Elec_4x4.5" (layer "F.Cu")
-    (at 85.09 167.513)
+    (at 82.528 180.34)
     (descr "SMD capacitor, aluminum electrolytic, Nichicon, 4.0x4.5mm")
     (tags "capacitor electrolytic")

Commit message: gg
Parts:
- D1, D2, Q1, R31: moved to B.Cu
- J3: value OUT-LPF -> OUT-BPF
- moved J2 68.6 mm to (237.6, 60.5), turned to 90 degrees
- moved R5 38.9 mm to (103.7, 67.2)
- moved U2 38.9 mm to (105.0, 55.9)
- moved C10 38.9 mm to (99.6, 61.7)
- moved C11 38.9 mm to (115.5, 67.7)
- moved C12 38.9 mm to (115.5, 52.2)
- moved C13 38.9 mm to (115.5, 62.5)
- moved C14 38.9 mm to (115.5, 57.3)
- moved R1 38.9 mm to (111.4, 63.4)
- moved R2 38.9 mm to (111.4, 55.8)
- moved R3 38.9 mm to (111.4, 60.9)
- moved R4 38.9 mm to (111.4, 58.4)
- moved T3 38.9 mm to (118.2, 48.5)
- moved U1 38.9 mm to (119.9, 60.4)
- moved C15 38.9 mm to (104.0, 70.2)
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Routing:
- net /BPF/BPF-OUT: track 0.00 -> 73.8 mm
- net /LPF/IN-LPF: track 0.00 -> 25.5 mm, vias 0 -> 1
- net RELAY-ON: track 33.0 -> 14.3 mm
- net /BPF/BPF-IN: track 0.00 -> 18.7 mm
- net /RF Switch/Antenna: track 15.7 -> 34.1 mm
- net /LPF/OUT-LPF: track 5.08 -> 16.7 mm
- net /PA/PA-IN: track 2.16 -> 12.2 mm, vias 0 -> 1
- net Net-(C3-Pad2): track 8.58 -> 12.7 mm
- net Net-(Q1-Pad1): track 3.59 -> 3.07 mm

Commit message: gg
Parts:
- SW1: footprint Button_Switch_THT:SW_PUSH_6mm -> Button_Switch_SMD:SW_SPST_B3U-1000P
- U6: footprint Xenir:ESP32-A1S -> xenir_v6:esp32-a1s-header
- moved R47 88.5 mm to (131.9, 158.0), turned to 180 degrees
- moved J9 85.9 mm to (199.9, 152.6)
- moved C43 85.9 mm to (191.3, 155.4)
- moved C44 85.9 mm to (174.0, 150.3)
- moved C47 85.9 mm to (167.1, 162.5)
- moved U9 85.9 mm to (171.7, 160.5)
- moved C45 85.9 mm to (180.1, 146.2)
- moved C46 85.9 mm to (162.8, 150.4)
- moved R43 85.9 mm to (168.5, 149.1)
- moved U8 85.9 mm to (181.4, 156.7)
- moved R42 85.9 mm to (168.5, 152.1)
- moved R46 79.2 mm to (126.8, 161.3)
- moved SW1 78.2 mm to (127.0, 148.4), turned to -90 degrees
- moved C25 77.9 mm to (127.2, 189.5)
- moved Q6 71.8 mm to (131.9, 162.1)
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Connections:
- U6 pad 6: unconnected-(U6-Pad6) -> IO0

Commit message: gg
Parts:
- added C50: 1uF, Capacitor_SMD:C_1206_3216Metric, F.Cu at (33.0, 89.1)
- added C51: 1uF, Capacitor_SMD:C_1206_3216Metric, F.Cu at (47.8, 89.1)
- added SW4: BOOT, Button_Switch_SMD:SW_SPST_B3U-1000P, F.Cu at (29.2, 89.1)
- SW1: value SW_DIP_x01 -> RST
- moved SW1 95.7 mm to (51.8, 89.2)
- moved C25 83.3 mm to (63.7, 135.6)
- moved C24 83.3 mm to (64.5, 125.5)
- moved C26 83.3 mm to (64.5, 120.2)
- moved C27 83.3 mm to (63.7, 132.8)
- moved Q6 83.3 mm to (68.4, 108.2)
- moved R21 83.3 mm to (71.2, 125.5)
- moved R22 83.3 mm to (71.3, 120.2)
- moved U6 83.3 mm to (39.4, 95.6)
- moved C28 83.3 mm to (75.4, 126.7)
- moved R46 83.3 mm to (63.3, 107.4)
- moved R47 83.3 mm to (68.4, 104.1)
- moved C29 83.3 mm to (75.4, 121.4)
- moved J11 83.2 mm to (17.3, 73.7)
- moved Q4 82.7 mm to (43.7, 104.9)
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Routing:
- net EN: track 0.00 -> 30.6 mm, vias 0 -> 1
- net IO0: track 0.00 -> 29.7 mm, vias 0 -> 1
- net Net-(Q5-Pad1): track 0.00 -> 2.96 mm
- net DTR: track 0.00 -> 2.96 mm
- net RTS: track 0.00 -> 2.86 mm
- net Net-(Q4-Pad1): track 0.00 -> 2.65 mm

Commit message: gg
Parts:
- moved J9 157.3 mm to (42.7, 147.1), turned to 0 degrees
- moved C43 156.4 mm to (35.8, 138.4), turned to 180 degrees
- moved U8 150.5 mm to (33.2, 130.0), turned to 180 degrees
- moved U9 143.6 mm to (33.7, 120.8), turned to 90 degrees
- moved C47 142.6 mm to (32.3, 116.1), turned to 180 degrees
- moved C45 135.6 mm to (44.9, 136.4)
- moved C44 129.2 mm to (45.7, 135.0), turned to 0 degrees
- moved R42 126.0 mm to (44.5, 129.9), turned to -90 degrees
- moved R43 122.3 mm to (47.8, 129.9), turned to 90 degrees
- moved C46 120.1 mm to (45.7, 123.8), turned to 0 degrees
- moved SW2 104.5 mm to (-52.2, 81.6)
- moved SW3 104.5 mm to (-51.8, 97.0)
- moved R2 80.8 mm to (90.9, 134.0)
- moved C14 80.8 mm to (95.0, 135.5)
- moved R4 80.8 mm to (90.9, 136.5)
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Connections:
- C15 pad 2: /Audio Switch/INR1 -> /Audio Switch/INL1
- C16 pad 2: /Audio Switch/INL1 -> /Audio Switch/INR1
- C47 pad 1: +3.3V -> +3V3
- R5 pad 2: /Audio Switch/INR1 -> /Audio Switch/INL1
- R6 pad 2: /Audio Switch/INL1 -> /Audio Switch/INR1
- U2 pad 1: /Audio Switch/INR1 -> /Audio Switch/INL1
- U2 pad 7: /Audio Switch/INL1 -> /Audio Switch/INR1
- U9 pad 2: +3.3V -> +3V3
Routing:
- net /Audio Switch/OUTL: track 0.00 -> 59.7 mm, vias 0 -> 2
- net /Audio Switch/INL1: track 6.87 -> 60.6 mm
- net /Audio Switch/OUTR: track 0.00 -> 40.6 mm, vias 0 -> 2
- net /Audio Switch/INR: track 0.00 -> 31.6 mm, vias 0 -> 2
- net +3V3: track 0.00 -> 22.5 mm, vias 0 -> 1
- net /Audio Switch/INL: track 0.00 -> 22.1 mm, vias 0 -> 2
- net +5V: track 86.5 -> 107.6 mm
- net /Audio Switch/INR1: track 6.22 -> 25.7 mm
- net +12V: track 17.9 -> 34.9 mm
- net GPIO21: track 0.00 -> 10.3 mm, vias 0 -> 1
- net +2V5: track 20.1 -> 28.9 mm
- net Net-(C24-Pad1): track 0.00 -> 6.62 mm
- net Net-(C26-Pad1): track 0.00 -> 5.35 mm
- net Net-(C25-Pad1): track 0.00 -> 4.95 mm
- net Net-(C27-Pad1): track 0.00 -> 4.85 mm
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Other:
- board outline added: 150 x 100 mm

Commit message: gg
Parts:
- moved J7 158.9 mm to (157.0, 148.6)
- moved J6 158.7 mm to (157.0, 138.2)
- moved J1 157.4 mm to (153.0, 125.8)
- moved C2 155.6 mm to (146.1, 147.9)
- moved J4 155.6 mm to (134.3, 156.2)
- moved J5 155.6 mm to (134.3, 120.2)
- moved C1 155.6 mm to (136.9, 141.6)
- moved C3 155.6 mm to (147.0, 143.7)
- moved D1 155.6 mm to (116.5, 147.4)
- moved D2 155.6 mm to (116.5, 128.4)
- moved J3 155.6 mm to (115.0, 120.2)
- moved K1 155.6 mm to (119.9, 150.0)
- moved K2 155.6 mm to (120.0, 130.8)
- moved L1 155.6 mm to (145.0, 143.0)
- moved Q1 155.6 mm to (115.1, 138.9)
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Routing:
- net /Audio Switch/OUTR2: track 3.77 -> 30.9 mm
- net /Audio Switch/OUTL2: track 5.97 -> 31.5 mm
- net /LPF/IN-LPF: track 25.5 -> 5.74 mm
- net /RF Switch/Antenna: track 34.1 -> 17.9 mm
- net Net-(C3-Pad2): track 12.7 -> 2.93 mm
- net /Audio Switch/INL1: track 60.6 -> 54.5 mm
- net /Audio Switch/INR1: track 25.7 -> 20.5 mm
- net +12V: track 34.9 -> 39.9 mm
