File: audio-switch.kicad_sch (KiCad schematic)
At the start: 0 parts

Commit message: gg
Changed lines of the file:
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@@
+    (effects (font (size 1.27 1.27)) (justify left))
+  )
+  (hierarchical_label "T{slash}R" (shape input) (at 111.76 78.74 0)
     (effects (font (size 1.27 1.27)) (justify left))
   )

Commit message: added switch
Parts:
- added C30, C31, C32, C33, C34, C35, C36, C37: .1uF, Capacitor_SMD:C_0805_2012Metric, symbol Xenir:Capacitor
- added R23, R24, R25, R26, R27, R28, R29, R30: 10k, Resistor_SMD:R_0805_2012Metric, symbol Xenir:Resistor
- added U7: FST3257, Xenir:SO16, symbol Xenir_v6:FST3257
Connections:
- net INL: now also R23.2, R24.1, U7.4 (1A)
- net INL1: now also C30.1
- net INL2: now also C31.1
- net INR: now also R25.2, R26.1, U7.7 (2A)
- net INR1: now also C32.1
- net INR2: now also C33.1
- net OUTL: now also R29.1, R30.2, U7.12 (4A)
- net OUTL1: now also C37.1
- net OUTL2: now also C36.1
- net OUTR: now also R27.1, R28.2, U7.9 (3A)
- net OUTR1: now also C35.1
- net OUTR2: now also C34.1
- new net: C32.2, U7.5 (2B1)
- new net: C35.2, U7.11 (3B1)
- new net: C37.2, U7.14 (4B1)
- new net: C34.2, U7.10 (3B2)
- new net: C36.2, U7.13 (4B2)
- new net: C30.2, U7.2 (1B1)
- new net: C31.2, U7.3 (1B2)
- new net: C33.2, U7.6 (2B2)
- new net +5V: R23.1, R25.1, R28.1, R30.1, U7.16 (VCC)
- new net GND: R24.2, R26.2, R27.2, R29.2, U7.8 (GND)

Commit message: updated switch
Parts:
- added C38: .1uF, Capacitor_SMD:C_0805_2012Metric, symbol Xenir:Capacitor
Connections:
- net +5V: now also C38.1
- net GND: now also U7.15 (OE), C38.2
- net T/R: now also U7.1 (S)
Changed lines of the file:
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@@
 (kicad_sch (version 20211123) (generator eeschema)
   (paper "A4")
+  (junction (at 147.32 80.01) (diameter 0) (color 0 0 0 0)
+  )
   (junction (at 104.14 123.19) (diameter 0) (color 0 0 0 0)
   )
@@
     (stroke (width 0) (type default) (color 0 0 0 0))
   )
+  (wire (pts (xy 147.32 76.2) (xy 147.32 80.01))
+    (stroke (width 0) (type default) (color 0 0 0 0))
+  )
   (wire (pts (xy 76.2 87.63) (xy 85.09 87.63))
     (stroke (width 0) (type default) (color 0 0 0 0))
@@
   )
   (wire (pts (xy 210.82 97.79) (xy 210.82 101.6))
+    (stroke (width 0) (type default) (color 0 0 0 0))
+  )
+  (wire (pts (xy 147.32 80.01) (xy 147.32 83.82))
     (stroke (width 0) (type default) (color 0 0 0 0))
   )
@@
     (effects (font (size 1.27 1.27)) (justify left))
   )
-  (hierarchical_label "T{slash}R" (shape input) (at 140.97 64.77 0)
-    (effects (font (size 1.27 1.27)) (justify left))
+  (hierarchical_label "T{slash}R" (shape input) (at 129.54 92.71 180)
+    (effects (font (size 1.27 1.27)) (justify right))
   )
   (hierarchical_label "OUTR" (shape input) (at 198.12 123.19 0)
@@
     (pin "1")
   )
+  (symbol (lib_id "Xenir:Capacitor") (at 143.51 80.01 0) (mirror y) (unit 1)
+    (in_bom yes) (on_board yes)
+    (property "Reference" "C38" (id 0) (at 142.24 83.82 0)
+      (effects (font (size 0.7112 0.7112)))
+    )
+    (property "Value" ".1uF" (id 1) (at 144.78 83.82 0)
+      (effects (font (size 0.7112 0.7112)))
+    )
+    (property "Footprint" "Capacitor_SMD:C_0805_2012Metric" (id 2) (at 143.51 83.82 0)
+      (effects (font (size 1.27 1.27)) hide)
+    )
+    (property "Datasheet" "" (id 3) (at 143.51 83.82 0)
+      (effects (font (size 1.27 1.27)) hide)
+    )
+    (pin "1")
+    (pin "2")
+  )
   (symbol (lib_id "Xenir:Capacitor") (at 109.22 113.03 0) (unit 1)
     (in_bom yes) (on_board yes) (fields_autoplaced)
@@
     (pin "2")
   )
-  (symbol (lib_id "power:+5V") (at 147.32 83.82 0) (unit 1)
-    (in_bom yes) (on_board yes)
-    (property "Reference" "#PWR0142" (id 0) (at 147.32 87.63 0)
-      (effects (font (size 1.27 1.27)) hide)
-    )
-    (property "Value" "+5V" (id 1) (at 143.51 82.55 0))
-    (property "Footprint" "" (id 2) (at 147.32 83.82 0)
-      (effects (font (size 1.27 1.27)) hide)
-    )
-    (property "Datasheet" "" (id 3) (at 147.32 83.82 0)
+  (symbol (lib_id "power:+5V") (at 147.32 76.2 0) (unit 1)
+    (in_bom yes) (on_board yes)
+    (property "Reference" "#PWR0142" (id 0) (at 147.32 80.01 0)
+      (effects (font (size 1.27 1.27)) hide)
+    )
+    (property "Value" "+5V" (id 1) (at 143.51 74.93 0))
+    (property "Footprint" "" (id 2) (at 147.32 76.2 0)
+      (effects (font (size 1.27 1.27)) hide)
+    )
+    (property "Datasheet" "" (id 3) (at 147.32 76.2 0)
       (effects (font (size 1.27 1.27)) hide)
     )
@@
     (pin "1")
   )
+  (symbol (lib_id "power:GND") (at 139.7 80.01 0) (mirror y) (unit 1)
+    (in_bom yes) (on_board yes)
+    (property "Reference" "#PWR0150" (id 0) (at 139.7 86.36 0)
+      (effects (font (size 1.27 1.27)) hide)
+    )
+    (property "Value" "GND" (id 1) (at 137.16 78.74 0))
+    (property "Footprint" "" (id 2) (at 139.7 80.01 0)
+      (effects (font (size 1.27 1.27)) hide)
+    )
+    (property "Datasheet" "" (id 3) (at 139.7 80.01 0)
+      (effects (font (size 1.27 1.27)) hide)
+    )
+    (pin "1")
+  )
   (symbol (lib_id "Xenir:Capacitor") (at 88.9 87.63 0) (unit 1)
     (in_bom yes) (on_board yes) (fields_autoplaced)
@@
     (pin "2")
   )
+  (symbol (lib_id "power:GND") (at 165.1 92.71 0) (mirror y) (unit 1)
+    (in_bom yes) (on_board yes)
+    (property "Reference" "#PWR?" (id 0) (at 165.1 99.06 0)
+      (effects (font (size 1.27 1.27)) hide)
+    )
+    (property "Value" "GND" (id 1) (at 167.64 92.71 0))
+    (property "Footprint" "" (id 2) (at 165.1 92.71 0)
+      (effects (font (size 1.27 1.27)) hide)
+    )
+    (property "Datasheet" "" (id 3) (at 165.1 92.71 0)
+      (effects (font (size 1.27 1.27)) hide)
+    )
+    (pin "1")
+  )
 )

Commit message: gg
Parts:
- added C39, C40, C41, C42: .1uF, Capacitor_SMD:C_0805_2012Metric, symbol Xenir:Capacitor
Connections:
- net INL: now also C39.1; no longer R23.2, R24.1, U7.4 (1A)
- net INR: now also C40.1; no longer R25.2, R26.1, U7.7 (2A)
- net OUTL: now also C42.2; no longer R29.1, R30.2, U7.12 (4A)
- net OUTR: now also C41.2; no longer R27.1, R28.2, U7.9 (3A)
- new net: C39.2, R23.2, R24.1, U7.4 (1A)
- new net: C41.1, R27.1, R28.2, U7.9 (3A)
- new net: C42.1, R29.1, R30.2, U7.12 (4A)
- new net: C40.2, R25.2, R26.1, U7.7 (2A)
Changed lines of the file:
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@@
   (junction (at 190.5 123.19) (diameter 0) (color 0 0 0 0)
   )
-  (wire (pts (xy 96.52 123.19) (xy 104.14 123.19))
+  (wire (pts (xy 86.36 123.19) (xy 91.44 123.19))
     (stroke (width 0) (type default) (color 0 0 0 0))
   )
@@
     (stroke (width 0) (type default) (color 0 0 0 0))
   )
+  (wire (pts (xy 215.9 97.79) (xy 210.82 97.79))
+    (stroke (width 0) (type default) (color 0 0 0 0))
+  )
   (wire (pts (xy 118.11 115.57) (xy 129.54 115.57))
     (stroke (width 0) (type default) (color 0 0 0 0))
@@
     (stroke (width 0) (type default) (color 0 0 0 0))
   )
-  (wire (pts (xy 218.44 97.79) (xy 210.82 97.79))
+  (wire (pts (xy 226.06 97.79) (xy 223.52 97.79))
     (stroke (width 0) (type default) (color 0 0 0 0))
   )
@@
     (stroke (width 0) (type default) (color 0 0 0 0))
   )
+  (wire (pts (xy 195.58 123.19) (xy 190.5 123.19))
+    (stroke (width 0) (type default) (color 0 0 0 0))
+  )
   (wire (pts (xy 210.82 97.79) (xy 196.85 97.79))
     (stroke (width 0) (type default) (color 0 0 0 0))
@@
     (stroke (width 0) (type default) (color 0 0 0 0))
   )
-  (wire (pts (xy 76.2 97.79) (xy 83.82 97.79))
+  (wire (pts (xy 66.04 97.79) (xy 71.12 97.79))
     (stroke (width 0) (type default) (color 0 0 0 0))
   )
@@
     (stroke (width 0) (type default) (color 0 0 0 0))
   )
+  (wire (pts (xy 99.06 123.19) (xy 104.14 123.19))
+    (stroke (width 0) (type default) (color 0 0 0 0))
+  )
   (wire (pts (xy 181.61 104.14) (xy 181.61 90.17))
     (stroke (width 0) (type default) (color 0 0 0 0))
@@
     (stroke (width 0) (type default) (color 0 0 0 0))
   )
-  (wire (pts (xy 198.12 123.19) (xy 190.5 123.19))
+  (wire (pts (xy 205.74 123.19) (xy 203.2 123.19))
     (stroke (width 0) (type default) (color 0 0 0 0))
   )
@@
     (stroke (width 0) (type default) (color 0 0 0 0))
   )
+  (wire (pts (xy 78.74 97.79) (xy 83.82 97.79))
+    (stroke (width 0) (type default) (color 0 0 0 0))
+  )
   (wire (pts (xy 97.79 90.17) (xy 113.03 90.17))
     (stroke (width 0) (type default) (color 0 0 0 0))
@@
     (stroke (width 0) (type default) (color 0 0 0 0))
   )
-  (hierarchical_label "INL" (shape output) (at 76.2 97.79 180)
+  (hierarchical_label "INL" (shape output) (at 66.04 97.79 180)
     (effects (font (size 1.27 1.27)) (justify right))
   )
@@
     (effects (font (size 1.27 1.27)) (justify left))
   )
-  (hierarchical_label "INR" (shape output) (at 96.52 123.19 180)
+  (hierarchical_label "INR" (shape output) (at 86.36 123.19 180)
     (effects (font (size 1.27 1.27)) (justify right))
   )
@@
     (effects (font (size 1.27 1.27)) (justify right))
   )
-  (hierarchical_label "OUTR" (shape input) (at 198.12 123.19 0)
+  (hierarchical_label "OUTR" (shape input) (at 205.74 123.19 0)
     (effects (font (size 1.27 1.27)) (justify left))
   )
-  (hierarchical_label "OUTL" (shape input) (at 218.44 97.79 0)
+  (hierarchical_label "OUTL" (shape input) (at 226.06 97.79 0)
     (effects (font (size 1.27 1.27)) (justify left))
   )
@@
     (effects (font (size 1.27 1.27)) (justify left))
   )
+  (symbol (lib_id "Xenir:Capacitor") (at 74.93 97.79 0) (unit 1)
+    (in_bom yes) (on_board yes)
+    (property "Reference" "C39" (id 0) (at 72.39 99.06 0)
+      (effects (font (size 0.7112 0.7112)))
+    )
+    (property "Value" ".1uF" (id 1) (at 77.47 99.06 0)
+      (effects (font (size 0.7112 0.7112)))
+    )
+    (property "Footprint" "Capacitor_SMD:C_0805_2012Metric" (id 2) (at 74.93 101.6 0)
+      (effects (font (size 1.27 1.27)) hide)
+    )
+    (property "Datasheet" "" (id 3) (at 74.93 101.6 0)
+      (effects (font (size 1.27 1.27)) hide)
+    )
+    (pin "1")
+    (pin "2")
+  )
   (symbol (lib_id "Xenir:Capacitor") (at 102.87 110.49 0) (unit 1)
     (in_bom yes) (on_board yes) (fields_autoplaced)
@@
     )
     (property "Datasheet" "" (id 3) (at 88.9 104.14 0)
+      (effects (font (size 1.27 1.27)) hide)
+    )
+    (pin "1")
+    (pin "2")
+  )
+  (symbol (lib_id "Xenir:Capacitor") (at 199.39 123.19 0) (unit 1)
+    (in_bom yes) (on_board yes)
+    (property "Reference" "C41" (id 0) (at 196.85 124.46 0)
+      (effects (font (size 0.7112 0.7112)))
+    )
+    (property "Value" ".1uF" (id 1) (at 201.93 124.46 0)
+      (effects (font (size 0.7112 0.7112)))
+    )
+    (property "Footprint" "Capacitor_SMD:C_0805_2012Metric" (id 2) (at 199.39 127 0)
+      (effects (font (size 1.27 1.27)) hide)
+    )
+    (property "Datasheet" "" (id 3) (at 199.39 127 0)
       (effects (font (size 1.27 1.27)) hide)
     )
@@
     (pin "2")
   )
+  (symbol (lib_id "Xenir:Capacitor") (at 219.71 97.79 0) (unit 1)
+    (in_bom yes) (on_board yes)
+    (property "Reference" "C42" (id 0) (at 217.17 99.06 0)
+      (effects (font (size 0.7112 0.7112)))
+    )
+    (property "Value" ".1uF" (id 1) (at 222.25 99.06 0)
+      (effects (font (size 0.7112 0.7112)))
+    )
+    (property "Footprint" "Capacitor_SMD:C_0805_2012Metric" (id 2) (at 219.71 101.6 0)
+      (effects (font (size 1.27 1.27)) hide)
+    )
+    (property "Datasheet" "" (id 3) (at 219.71 101.6 0)
+      (effects (font (size 1.27 1.27)) hide)
+    )
+    (pin "1")
+    (pin "2")
+  )
   (symbol (lib_id "power:+5V") (at 147.32 76.2 0) (unit 1)
     (in_bom yes) (on_board yes)
@@
     (pin "2")
   )
+  (symbol (lib_id "Xenir:Capacitor") (at 95.25 123.19 0) (unit 1)
+    (in_bom yes) (on_board yes)
+    (property "Reference" "C40" (id 0) (at 92.71 124.46 0)
+      (effects (font (size 0.7112 0.7112)))
+    )
+    (property "Value" ".1uF" (id 1) (at 97.79 124.46 0)
+      (effects (font (size 0.7112 0.7112)))
+    )
+    (property "Footprint" "Capacitor_SMD:C_0805_2012Metric" (id 2) (at 95.25 127 0)
+      (effects (font (size 1.27 1.27)) hide)
+    )
+    (property "Datasheet" "" (id 3) (at 95.25 127 0)
+      (effects (font (size 1.27 1.27)) hide)
+    )
+    (pin "1")
+    (pin "2")
+  )
   (symbol (lib_id "power:GND") (at 165.1 92.71 0) (mirror y) (unit 1)
     (in_bom yes) (on_board yes)
-    (property "Reference" "#PWR?" (id 0) (at 165.1 99.06 0)
-      (effects (font (size 1.27 1.27)) hide)
-    )
+    (property "Reference" "#PWR0151" (id 0) (at 165.1 99.06 0)
+      (effects (font (size 1.27 1.27)) hide)
+    )

Commit message: added output resistors to switch
Parts:
- added R38, R39, R40, R41: 47k, Resistor_SMD:R_0805_2012Metric, symbol Xenir:Resistor
- C30, C31, C32, C33, C34, C35, C36, C37, C39, C40, C41, C42: value .1uF -> 1uF
Connections:
- net GND: now also R38.2, R39.2, R40.2, R41.2
- net OUTL1: now also R41.1
- net OUTL2: now also R40.1
- net OUTR1: now also R39.1
- net OUTR2: now also R38.1
