File: PA.kicad_sch (KiCad schematic)
At the start: 0 parts

Commit message: added pa
Parts:
- added J6, J7: PCB_SMA_EDGE, Xenir_V6:pcb-sma-edge, symbol Xenir:PCB_SMA_EDGE
- added J8: Audio_Jack, Xenir:Audio_Jack, symbol Xenir:Audio_Jack
- added Q2: AO3400A, Package_TO_SOT_SMD:SOT-23, symbol Transistor_FET:AO3400A
- added R32: 1k, Resistor_SMD:R_0805_2012Metric, symbol xenir:Resistor
Connections:
- net PA-IN: now also J6.1
- net PA-OUT: now also J7.1
- net T/R: now also R32.1
- new net: J8.TIP, J8.TSH, Q2.3 (D)
- new net: Q2.1 (G), R32.2
- new net GND: J6.2, J7.2, J8.SLEEVE, Q2.2 (S)
Changed lines of the file:
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@@
 (kicad_sch (version 20211123) (generator eeschema)
   (paper "A4")
-  (hierarchical_label "PA-IN" (shape input) (at 120.65 90.17 0)
+  (junction (at 209.55 87.63) (diameter 0) (color 0 0 0 0)
+  )
+  (wire (pts (xy 185.42 87.63) (xy 185.42 91.44))
+    (stroke (width 0) (type default) (color 0 0 0 0))
+  )
+  (wire (pts (xy 162.56 96.52) (xy 165.1 96.52))
+    (stroke (width 0) (type default) (color 0 0 0 0))
+  )
+  (wire (pts (xy 209.55 87.63) (xy 209.55 90.17))
+    (stroke (width 0) (type default) (color 0 0 0 0))
+  )
+  (wire (pts (xy 185.42 87.63) (xy 209.55 87.63))
+    (stroke (width 0) (type default) (color 0 0 0 0))
+  )
+  (wire (pts (xy 175.26 96.52) (xy 177.8 96.52))
+    (stroke (width 0) (type default) (color 0 0 0 0))
+  )
+  (hierarchical_label "T{slash}R" (shape input) (at 162.56 96.52 180)
+    (effects (font (size 1.27 1.27)) (justify right))
+  )
+  (hierarchical_label "PA-IN" (shape input) (at 123.19 96.52 0)
     (effects (font (size 1.27 1.27)) (justify left))
   )
-  (hierarchical_label "PA-OUT" (shape output) (at 120.65 96.52 0)
+  (hierarchical_label "PA-OUT" (shape output) (at 140.97 96.52 0)
     (effects (font (size 1.27 1.27)) (justify left))
   )
-  (hierarchical_label "T{slash}R" (shape input) (at 120.65 102.87 0)
-    (effects (font (size 1.27 1.27)) (justify left))
+  (symbol (lib_id "Xenir:Audio_Jack") (at 214.63 101.6 180) (unit 1)
+    (in_bom yes) (on_board yes) (fields_autoplaced)
+    (property "Reference" "J8" (id 0) (at 222.25 91.4399 0)
+      (effects (font (size 1.27 1.27)) (justify right))
+    )
+    (property "Value" "Audio_Jack" (id 1) (at 222.25 93.9799 0)
+      (effects (font (size 1.27 1.27)) (justify right))
+    )
+    (property "Footprint" "Xenir:Audio_Jack" (id 2) (at 214.63 101.6 0)
+      (effects (font (size 1.27 1.27)) hide)
+    )
+    (property "Datasheet" "" (id 3) (at 214.63 101.6 0)
+      (effects (font (size 1.27 1.27)) hide)
+    )
+    (pin "RING")
+    (pin "RSH")
+    (pin "SLEEVE")
+    (pin "TIP")
+    (pin "TSH")
+  )
+  (symbol (lib_id "power:GND") (at 209.55 97.79 0) (unit 1)
+    (in_bom yes) (on_board yes) (fields_autoplaced)
+    (property "Reference" "#PWR0163" (id 0) (at 209.55 104.14 0)
+      (effects (font (size 1.27 1.27)) hide)
+    )
+    (property "Value" "GND" (id 1) (at 209.55 102.87 0))
+    (property "Footprint" "" (id 2) (at 209.55 97.79 0)
+      (effects (font (size 1.27 1.27)) hide)
+    )
+    (property "Datasheet" "" (id 3) (at 209.55 97.79 0)
+      (effects (font (size 1.27 1.27)) hide)
+    )
+    (pin "1")
+  )
+  (symbol (lib_id "Transistor_FET:AO3400A") (at 182.88 96.52 0) (unit 1)
+    (in_bom yes) (on_board yes) (fields_autoplaced)
+    (property "Reference" "Q2" (id 0) (at 189.23 95.2499 0)
+      (effects (font (size 1.27 1.27)) (justify left))
+    )
+    (property "Value" "AO3400A" (id 1) (at 189.23 97.7899 0)
+      (effects (font (size 1.27 1.27)) (justify left))
+    )
+    (property "Footprint" "Package_TO_SOT_SMD:SOT-23" (id 2) (at 187.96 98.425 0)
+      (effects (font (size 1.27 1.27) italic) (justify left) hide)
+    )
+    (property "Datasheet" "http://www.aosmd.com/pdfs/datasheet/AO3400A.pdf" (id 3) (at 182.88 96.52 0)
+      (effects (font (size 1.27 1.27)) (justify left) hide)
+    )
+    (pin "1")
+    (pin "2")
+    (pin "3")
+  )
+  (symbol (lib_id "xenir:Resistor") (at 170.18 96.52 0) (unit 1)
+    (in_bom yes) (on_board yes) (fields_autoplaced)
+    (property "Reference" "R32" (id 0) (at 170.18 91.44 0)
+      (effects (font (size 0.7112 0.7112)))
+    )
+    (property "Value" "1k" (id 1) (at 170.18 93.98 0)
+      (effects (font (size 0.7112 0.7112)))
+    )
+    (property "Footprint" "Resistor_SMD:R_0805_2012Metric" (id 2) (at 170.18 99.06 0)
+      (effects (font (size 1.27 1.27)) hide)
+    )
+    (property "Datasheet" "" (id 3) (at 170.18 99.06 0)
+      (effects (font (size 1.27 1.27)) hide)
+    )
+    (pin "1")
+    (pin "2")
+  )
+  (symbol (lib_id "power:GND") (at 140.97 99.06 0) (unit 1)
+    (in_bom yes) (on_board yes) (fields_autoplaced)
+    (property "Reference" "#PWR0162" (id 0) (at 140.97 105.41 0)
+      (effects (font (size 1.27 1.27)) hide)
+    )
+    (property "Value" "GND" (id 1) (at 140.97 104.14 0))
+    (property "Footprint" "" (id 2) (at 140.97 99.06 0)
+      (effects (font (size 1.27 1.27)) hide)
+    )
+    (property "Datasheet" "" (id 3) (at 140.97 99.06 0)
+      (effects (font (size 1.27 1.27)) hide)
+    )
+    (pin "1")
+  )
+  (symbol (lib_id "power:GND") (at 123.19 99.06 0) (unit 1)
+    (in_bom yes) (on_board yes) (fields_autoplaced)
+    (property "Reference" "#PWR0161" (id 0) (at 123.19 105.41 0)
+      (effects (font (size 1.27 1.27)) hide)
+    )
+    (property "Value" "GND" (id 1) (at 123.19 104.14 0))
+    (property "Footprint" "" (id 2) (at 123.19 99.06 0)
+      (effects (font (size 1.27 1.27)) hide)
+    )
+    (property "Datasheet" "" (id 3) (at 123.19 99.06 0)
+      (effects (font (size 1.27 1.27)) hide)
+    )
+    (pin "1")
+  )
+  (symbol (lib_id "Xenir:PCB_SMA_EDGE") (at 120.65 91.44 0) (unit 1)
+    (in_bom yes) (on_board yes) (fields_autoplaced)
+    (property "Reference" "J6" (id 0) (at 119.38 88.9 0))
+    (property "Value" "PCB_SMA_EDGE" (id 1) (at 119.38 91.44 0))
+    (property "Footprint" "Xenir_V6:pcb-sma-edge" (id 2) (at 120.65 91.44 0)
+      (effects (font (size 1.27 1.27)) hide)
+    )
+    (property "Datasheet" "" (id 3) (at 120.65 91.44 0)
+      (effects (font (size 1.27 1.27)) hide)
+    )
+    (pin "1")
+    (pin "2")
+  )
+  (symbol (lib_id "power:GND") (at 185.42 101.6 0) (unit 1)
+    (in_bom yes) (on_board yes) (fields_autoplaced)
+    (property "Reference" "#PWR0160" (id 0) (at 185.42 107.95 0)
+      (effects (font (size 1.27 1.27)) hide)
+    )
+    (property "Value" "GND" (id 1) (at 185.42 106.68 0))
+    (property "Footprint" "" (id 2) (at 185.42 101.6 0)
+      (effects (font (size 1.27 1.27)) hide)
+    )
+    (property "Datasheet" "" (id 3) (at 185.42 101.6 0)
+      (effects (font (size 1.27 1.27)) hide)
+    )
+    (pin "1")
+  )
+  (symbol (lib_id "Xenir:PCB_SMA_EDGE") (at 138.43 91.44 0) (unit 1)
+    (in_bom yes) (on_board yes) (fields_autoplaced)
+    (property "Reference" "J7" (id 0) (at 137.16 88.9 0))
+    (property "Value" "PCB_SMA_EDGE" (id 1) (at 137.16 91.44 0))
+    (property "Footprint" "Xenir_V6:pcb-sma-edge" (id 2) (at 138.43 91.44 0)
+      (effects (font (size 1.27 1.27)) hide)
+    )
+    (property "Datasheet" "" (id 3) (at 138.43 91.44 0)
+      (effects (font (size 1.27 1.27)) hide)
+    )
+    (pin "1")
+    (pin "2")
   )
 )

Commit message: updated PA
Parts:
- added C1, C3: .1uF, Capacitor_SMD:C_0805_2012Metric, symbol Xenir:Capacitor
- added C2: 10nF, Capacitor_SMD:C_0805_2012Metric, symbol Xenir:Capacitor
- added L1: BN43-2402 6T, Xenir:BN-43-2402, symbol Xenir:Inductor
- added Q3: 2N2222, Package_TO_SOT_SMD:SOT-23, symbol Xenir:2N3904-SMD
- added R33: 2.2k, Resistor_SMD:R_0805_2012Metric, symbol Xenir:Resistor
- added R34: 475, Resistor_SMD:R_0805_2012Metric, symbol Xenir:Resistor
- added R35: 56, Resistor_SMD:R_0805_2012Metric, symbol Xenir:Resistor
- added R36: 50, Resistor_SMD:R_0805_2012Metric, symbol Xenir:Resistor
- J6: value PCB_SMA_EDGE -> TO-PA
- J7: value PCB_SMA_EDGE -> FROM-PA
Connections:
- net GND: now also C2.1, R34.1, R35.1
- net PA-IN: now also C1.1; no longer J6.1
- new net: C2.2, R36.1
- new net: Q3.2 (E), R35.2, R36.2
- new net: C1.2, Q3.1 (B), R33.1, R34.2
- new net: C3.1, L1.1, Q3.3 (C)
- new net: C3.2, J6.1
- new net +12V: L1.2, R33.2
Other:
- moved on the sheet: J6, J7, J8, Q2, R32

Commit message: added cap
Parts:
- added C4: .1uF, Capacitor_SMD:C_0805_2012Metric, symbol Xenir:Capacitor
Connections:
- net +12V: now also C4.2
- net GND: now also C4.1
Changed lines of the file:
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@@
+    (stroke (width 0) (type default) (color 0 0 0 0))
+  )
+  (wire (pts (xy 118.11 80.01) (xy 125.73 80.01))
     (stroke (width 0) (type default) (color 0 0 0 0))
   )
@@
     (pin "2")
   )
+  (symbol (lib_id "power:GND") (at 118.11 87.63 0) (mirror y) (unit 1)
+    (in_bom yes) (on_board yes) (fields_autoplaced)
+    (property "Reference" "#PWR0167" (id 0) (at 118.11 93.98 0)
+      (effects (font (size 1.27 1.27)) hide)
+    )
+    (property "Value" "GND" (id 1) (at 118.11 92.71 0))
+    (property "Footprint" "" (id 2) (at 118.11 87.63 0)
+      (effects (font (size 1.27 1.27)) hide)
+    )
+    (property "Datasheet" "" (id 3) (at 118.11 87.63 0)
+      (effects (font (size 1.27 1.27)) hide)
+    )
+    (pin "1")
+  )
   (symbol (lib_id "Xenir:Inductor") (at 137.16 83.82 90) (unit 1)
     (in_bom yes) (on_board yes) (fields_autoplaced)
@@
       (effects (font (size 1.27 1.27)) hide)
     )
+    (pin "1")
+    (pin "2")
+  )
+  (symbol (lib_id "Xenir:Capacitor") (at 118.11 83.82 90) (unit 1)
+    (in_bom yes) (on_board yes)
+    (property "Reference" "C4" (id 0) (at 116.84 86.36 0)
+      (effects (font (size 0.7112 0.7112)))
+    )
+    (property "Value" ".1uF" (id 1) (at 119.38 86.36 0)
+      (effects (font (size 0.7112 0.7112)))
+    )
+    (property "Footprint" "Capacitor_SMD:C_0805_2012Metric" (id 2) (at 121.92 83.82 0)
+      (effects (font (size 1.27 1.27)) hide)
+    )
+    (property "Datasheet" "" (id 3) (at 121.92 83.82 0)
+      (effects (font (size 1.27 1.27)) hide)
+    )

Commit message: gg
Parts:
- added R37: 50, Resistor_SMD:R_0805_2012Metric, symbol Xenir:Resistor
- added TP1: TestPoint, TestPoint:TestPoint_THTPad_1.0x1.0mm_Drill0.5mm, symbol Connector:TestPoint
Connections:
- net GND: now also R37.1
- net PA-IN: now also R37.2
- net at C3.2, J6.1: now also TP1.1
Changed lines of the file:
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@@
   (junction (at 144.78 120.65) (diameter 0) (color 0 0 0 0)
   )
+  (junction (at 109.22 96.52) (diameter 0) (color 0 0 0 0)
+  )
   (junction (at 125.73 96.52) (diameter 0) (color 0 0 0 0)
   )
+  (junction (at 154.94 90.17) (diameter 0) (color 0 0 0 0)
+  )
   (junction (at 137.16 90.17) (diameter 0) (color 0 0 0 0)
   )
@@
     (stroke (width 0) (type default) (color 0 0 0 0))
   )
+  (wire (pts (xy 105.41 96.52) (xy 109.22 96.52))
+    (stroke (width 0) (type default) (color 0 0 0 0))
+  )
   (wire (pts (xy 125.73 77.47) (xy 125.73 80.01))
     (stroke (width 0) (type default) (color 0 0 0 0))
@@
   )
   (wire (pts (xy 137.16 113.03) (xy 137.16 120.65))
+    (stroke (width 0) (type default) (color 0 0 0 0))
+  )
+  (wire (pts (xy 109.22 96.52) (xy 110.49 96.52))
     (stroke (width 0) (type default) (color 0 0 0 0))
   )
@@
     (effects (font (size 1.27 1.27)) (justify right))
   )
-  (hierarchical_label "PA-IN" (shape input) (at 110.49 96.52 180)
+  (hierarchical_label "PA-IN" (shape input) (at 105.41 96.52 180)
     (effects (font (size 1.27 1.27)) (justify right))
   )
@@
     (pin "1")
   )
+  (symbol (lib_id "Xenir:Resistor") (at 109.22 101.6 90) (unit 1)
+    (in_bom yes) (on_board yes) (fields_autoplaced)
+    (property "Reference" "R37" (id 0) (at 111.76 100.965 90)
+      (effects (font (size 0.7112 0.7112)) (justify right))
+    )
+    (property "Value" "50" (id 1) (at 111.76 103.505 90)
+      (effects (font (size 0.7112 0.7112)) (justify right))
+    )
+    (property "Footprint" "Resistor_SMD:R_0805_2012Metric" (id 2) (at 111.76 101.6 0)
+      (effects (font (size 1.27 1.27)) hide)
+    )
+    (property "Datasheet" "" (id 3) (at 111.76 101.6 0)
+      (effects (font (size 1.27 1.27)) hide)
+    )
+    (pin "1")
+    (pin "2")
+  )
   (symbol (lib_id "power:GND") (at 125.73 111.76 0) (unit 1)
     (in_bom yes) (on_board yes) (fields_autoplaced)
@@
     )
     (property "Datasheet" "" (id 3) (at 144.78 121.92 0)
+      (effects (font (size 1.27 1.27)) hide)
+    )
+    (pin "1")
+  )
+  (symbol (lib_id "power:GND") (at 109.22 106.68 0) (unit 1)
+    (in_bom yes) (on_board yes) (fields_autoplaced)
+    (property "Reference" "#PWR0168" (id 0) (at 109.22 113.03 0)
+      (effects (font (size 1.27 1.27)) hide)
+    )
+    (property "Value" "GND" (id 1) (at 109.22 111.76 0))
+    (property "Footprint" "" (id 2) (at 109.22 106.68 0)
+      (effects (font (size 1.27 1.27)) hide)
+    )
+    (property "Datasheet" "" (id 3) (at 109.22 106.68 0)
       (effects (font (size 1.27 1.27)) hide)
     )
@@
     (pin "1")
   )
+  (symbol (lib_id "Connector:TestPoint") (at 154.94 90.17 0) (unit 1)
+    (in_bom yes) (on_board yes)
+    (property "Reference" "TP1" (id 0) (at 153.67 85.09 0)
+      (effects (font (size 1.27 1.27)) (justify left))
+    )
+    (property "Value" "TestPoint" (id 1) (at 157.48 83.82 0)
+      (effects (font (size 1.27 1.27)) (justify left) hide)
+    )
+    (property "Footprint" "TestPoint:TestPoint_THTPad_1.0x1.0mm_Drill0.5mm" (id 2) (at 160.02 90.17 0)
+      (effects (font (size 1.27 1.27)) hide)
+    )
+    (property "Datasheet" "~" (id 3) (at 160.02 90.17 0)
+      (effects (font (size 1.27 1.27)) hide)
+    )
+    (pin "1")
+  )
   (symbol (lib_id "Xenir:Inductor") (at 137.16 83.82 90) (unit 1)
-    (in_bom yes) (on_board yes) (fields_autoplaced)
-    (property "Reference" "L1" (id 0) (at 138.43 82.5499 90)
-      (effects (font (size 1.27 1.27)) (justify right))
-    )
-    (property "Value" "BN43-2402 6T" (id 1) (at 138.43 85.0899 90)
-      (effects (font (size 1.27 1.27)) (justify right))
-    )
+    (in_bom yes) (on_board yes)
+    (property "Reference" "L1" (id 0) (at 134.62 82.55 0)
+      (effects (font (size 1.27 1.27)) (justify right))
+    )
+    (property "Value" "BN43-2402 6T" (id 1) (at 138.43 73.66 0)
+      (effects (font (size 1.27 1.27)) (justify right))
+    )

Commit message: gg
Parts:
- J8: value Audio_Jack -> Amplifier T/R
Changed lines of the file:
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@@
       (effects (font (size 1.27 1.27)) (justify right))
     )
-    (property "Value" "Audio_Jack" (id 1) (at 176.53 54.6099 0)
+    (property "Value" "Amplifier T/R" (id 1) (at 176.53 54.6099 0)
       (effects (font (size 1.27 1.27)) (justify right))
     )
