File: DSP.kicad_sch (KiCad schematic)
At the start: 9 parts, among them U6 ESP32-A1S

Commit message: more updates
Connections:
- net SDA: now reaches U6.31 (IO23)
- net SCL: now reaches U6.32 (IO19)
Changed lines of the file:
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@@
+    (effects (font (size 1.27 1.27)) (justify left))
+  )
+  (hierarchical_label "SDA" (shape output) (at 165.1 92.71 0)
     (effects (font (size 1.27 1.27)) (justify left))
   )
@@
     (effects (font (size 1.27 1.27)) (justify left))
   )
+  (hierarchical_label "SCL" (shape output) (at 165.1 90.17 0)
+    (effects (font (size 1.27 1.27)) (justify left))
+  )

Commit message: gg
Connections:
- net T/R: now reaches U6.33 (IO22)
Changed lines of the file:
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@@
+    (effects (font (size 1.27 1.27)) (justify left))
+  )
+  (hierarchical_label "T{slash}R" (shape output) (at 165.1 87.63 0)
     (effects (font (size 1.27 1.27)) (justify left))
   )

Commit message: updated DSP
Parts:
- added J10: Conn_01x07_Female, Connector_PinSocket_2.54mm:PinSocket_1x07_P2.54mm_Vertical, symbol Connector:Conn_01x07_Female
- added J11: Conn_01x04, Connector_PinSocket_2.54mm:PinSocket_1x04_P2.54mm_Vertical, symbol Connector_Generic:Conn_01x04
- added Q4, Q5: 2N3904-SMD, Package_TO_SOT_SMD:SOT-23, symbol Tayloe-Mixer-v3-rescue:2N3904-SMD-xenir
- added Q6: AO3400A, Package_TO_SOT_SMD:SOT-23, symbol Transistor_FET:AO3400A
- added R44, R45: 10k, Resistor_SMD:R_0805_2012Metric, symbol Tayloe-Mixer-v3-rescue:Resistor-Xenir-esp32-a1s-rescue
- added R46: 1k, Resistor_SMD:R_0805_2012Metric, symbol xenir:Resistor
- added R47: 10k, Resistor_SMD:R_0805_2012Metric, symbol xenir:Resistor
- added SW1: SW_DIP_x01, Button_Switch_THT:SW_PUSH_6mm, symbol Switch:SW_DIP_x01
- added SW2: Frequency, Rotary_Encoder:RotaryEncoder_Alps_EC11E-Switch_Vertical_H20mm, symbol Tayloe-Mixer-v3-rescue:Rotary_Encoder_Switch-Device
- added SW3: Menu, Rotary_Encoder:RotaryEncoder_Alps_EC11E-Switch_Vertical_H20mm, symbol Tayloe-Mixer-v3-rescue:Rotary_Encoder_Switch-Device
Connections:
- net GND: now also J10.6 (Pin_6), J11.1 (Pin_1), Q6.2 (S), SW1.1, SW2.C, SW2.S1, SW3.C, SW3.S1
- net SCL: now also J11.4 (Pin_4)
- net SDA: now also J11.3 (Pin_3)
- net T/R: now also Q6.3 (D), R47.1; no longer U6.33 (IO22)
- net GPIO21: now reaches U6.34 (IO21)
- net GPIO21: now also R46.1
- net EN: now reaches U6.35 (EN)
- net EN: now also Q4.3 (C), SW1.2
- net RX0: now reaches U6.36 (TXD0)
- net RX0: now also J10.2 (Pin_2)
- net TX0: now reaches U6.37 (RXD0)
- net TX0: now also J10.3 (Pin_3)
- net GPIO14: now reaches U6.7 (IO14)
- net GPIO14: now also SW2.A
- net GPIO12: now reaches U6.8 (IO12)
- net GPIO13: now reaches U6.9 (IO13)
- net GPIO13: now also SW2.B, SW2.S2
- new net: Q5.1 (B), R45.2
- new net: Q4.1 (B), R44.2
- new net: Q6.1 (G), R46.2
- new net +5V: J11.2 (Pin_2), R47.2
- new net DTR: J10.1 (Pin_1), Q5.2 (E), R44.1
- new net GPIO15: SW3.B
- new net GPIO34: SW3.A
- new net GPIO4: SW3.S2
- new net IO0: Q5.3 (C)
- new net RTS: J10.7 (Pin_7), Q4.2 (E), R45.1
Other:
- moved on the sheet: U6

Commit message: gg
Connections:
- net GPIO12: now also SW2.S2
- net GPIO13: no longer SW2.S2
- net GPIO15: now also U6.10 (IO15)
- net GPIO34: now also U6.5 (IO34)
- net GPIO4: now also U6.12 (IO4)
Changed lines of the file:
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@@
+    )
+  )
+  (global_label "GPIO34" (shape input) (at 118.11 85.09 180) (fields_autoplaced)
+    (effects (font (size 1.27 1.27)) (justify right))
+    (property "Intersheet References" "${INTERSHEET_REFS}" (id 0) (at 108.8026 85.1694 0)
+      (effects (font (size 1.27 1.27)) (justify right) hide)
     )
   )
@@
     )
   )
-  (global_label "GPIO13" (shape input) (at 92.71 143.51 180) (fields_autoplaced)
+  (global_label "GPIO12" (shape input) (at 92.71 143.51 180) (fields_autoplaced)
     (effects (font (size 1.27 1.27)) (justify right))
     (property "Intersheet References" "${INTERSHEET_REFS}" (id 0) (at 83.4026 143.4306 0)
@@
     (property "Intersheet References" "${INTERSHEET_REFS}" (id 0) (at 2.54 -109.22 0)
       (effects (font (size 1.27 1.27)) hide)
+    )
+  )
+  (global_label "GPIO15" (shape input) (at 118.11 97.79 180) (fields_autoplaced)
+    (effects (font (size 1.27 1.27)) (justify right))
+    (property "Intersheet References" "${INTERSHEET_REFS}" (id 0) (at 108.8026 97.8694 0)
+      (effects (font (size 1.27 1.27)) (justify right) hide)
     )
   )
@@
     )
   )
+  (global_label "GPIO4" (shape input) (at 118.11 102.87 180) (fields_autoplaced)
+    (effects (font (size 1.27 1.27)) (justify right))
+    (property "Intersheet References" "${INTERSHEET_REFS}" (id 0) (at 110.0121 102.7906 0)
+      (effects (font (size 1.27 1.27)) (justify right) hide)
+    )
+  )

Commit message: added LO
Connections:
- net GND: now also U6.1 (GND), U6.19 (GND), U6.20 (GND), U6.38 (GND)
- net +3V3: now reaches U6.2 (3V3)
Changed lines of the file:
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@@
+    (stroke (width 0) (type default) (color 0 0 0 0))
+  )
+  (wire (pts (xy 106.68 77.47) (xy 118.11 77.47))
     (stroke (width 0) (type default) (color 0 0 0 0))
   )
@@
     (pin "2")
   )
+  (symbol (lib_id "power:GND") (at 118.11 120.65 270) (unit 1)
+    (in_bom yes) (on_board yes) (fields_autoplaced)
+    (property "Reference" "#PWR0202" (id 0) (at 111.76 120.65 0)
+      (effects (font (size 1.27 1.27)) hide)
+    )
+    (property "Value" "GND" (id 1) (at 114.3 120.6499 90)
+      (effects (font (size 1.27 1.27)) (justify right))
+    )
+    (property "Footprint" "" (id 2) (at 118.11 120.65 0)
+      (effects (font (size 1.27 1.27)) hide)
+    )
+    (property "Datasheet" "" (id 3) (at 118.11 120.65 0)
+      (effects (font (size 1.27 1.27)) hide)
+    )
+    (pin "1")
+  )
   (symbol (lib_id "power:GND") (at 204.47 110.49 0) (unit 1)
     (in_bom yes) (on_board yes)
@@
     (pin "2")
   )
+  (symbol (lib_id "power:GND") (at 118.11 74.93 270) (unit 1)
+    (in_bom yes) (on_board yes) (fields_autoplaced)
+    (property "Reference" "#PWR0199" (id 0) (at 111.76 74.93 0)
+      (effects (font (size 1.27 1.27)) hide)
+    )
+    (property "Value" "GND" (id 1) (at 114.3 74.9299 90)
+      (effects (font (size 1.27 1.27)) (justify right))
+    )
+    (property "Footprint" "" (id 2) (at 118.11 74.93 0)
+      (effects (font (size 1.27 1.27)) hide)
+    )
+    (property "Datasheet" "" (id 3) (at 118.11 74.93 0)
+      (effects (font (size 1.27 1.27)) hide)
+    )
+    (pin "1")
+  )
   (symbol (lib_id "Connector_Generic:Conn_01x04") (at 184.15 147.32 270) (unit 1)
     (in_bom yes) (on_board yes)
@@
     (pin "3")
     (pin "4")
+  )
+  (symbol (lib_id "power:GND") (at 158.75 74.93 90) (unit 1)
+    (in_bom yes) (on_board yes) (fields_autoplaced)
+    (property "Reference" "#PWR0200" (id 0) (at 165.1 74.93 0)
+      (effects (font (size 1.27 1.27)) hide)
+    )
+    (property "Value" "GND" (id 1) (at 162.56 74.9299 90)
+      (effects (font (size 1.27 1.27)) (justify right))
+    )
+    (property "Footprint" "" (id 2) (at 158.75 74.93 0)
+      (effects (font (size 1.27 1.27)) hide)
+    )
+    (property "Datasheet" "" (id 3) (at 158.75 74.93 0)
+      (effects (font (size 1.27 1.27)) hide)
+    )
+    (pin "1")
   )
   (symbol (lib_id "Tayloe-Mixer-v3-rescue:2N3904-SMD-xenir") (at 59.69 114.3 0) (mirror x) (unit 1)
@@
     )
     (property "Datasheet" "" (id 3) (at 198.12 38.1 0)
+      (effects (font (size 1.27 1.27)) hide)
+    )
+    (pin "1")
+  )
+  (symbol (lib_id "power:+3V3") (at 106.68 77.47 0) (unit 1)
+    (in_bom yes) (on_board yes)
+    (property "Reference" "#PWR0201" (id 0) (at 106.68 81.28 0)
+      (effects (font (size 1.27 1.27)) hide)
+    )
+    (property "Value" "+3V3" (id 1) (at 105.41 73.66 0))
+    (property "Footprint" "" (id 2) (at 106.68 77.47 0)
+      (effects (font (size 1.27 1.27)) hide)
+    )
+    (property "Datasheet" "" (id 3) (at 106.68 77.47 0)
       (effects (font (size 1.27 1.27)) hide)
     )
@@
     (pin "2")
   )
+  (symbol (lib_id "power:GND") (at 158.75 120.65 90) (unit 1)
+    (in_bom yes) (on_board yes) (fields_autoplaced)
+    (property "Reference" "#PWR0203" (id 0) (at 165.1 120.65 0)
+      (effects (font (size 1.27 1.27)) hide)
+    )
+    (property "Value" "GND" (id 1) (at 162.56 120.6499 90)
+      (effects (font (size 1.27 1.27)) (justify right))
+    )
+    (property "Footprint" "" (id 2) (at 158.75 120.65 0)
+      (effects (font (size 1.27 1.27)) hide)
+    )
+    (property "Datasheet" "" (id 3) (at 158.75 120.65 0)
+      (effects (font (size 1.27 1.27)) hide)
+    )
+    (pin "1")
+  )
   (symbol (lib_id "power:GND") (at 87.63 83.82 0) (unit 1)

Commit message: gg
Parts:
- C24, C26: footprint Capacitor_SMD:C_1206_3216Metric -> Capacitor_SMD:CP_Elec_4x4.5
Changed lines of the file:
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@@
     (property "Reference" "C26" (id 0) (at 186.69 96.52 90))
     (property "Value" "22uF" (id 1) (at 191.77 96.52 90))
-    (property "Footprint" "Capacitor_SMD:C_1206_3216Metric" (id 2) (at 193.04 99.3648 0)
+    (property "Footprint" "Capacitor_SMD:CP_Elec_4x4.5" (id 2) (at 193.04 99.3648 0)
       (effects (font (size 1.27 1.27)) hide)
     )
@@
     (property "Reference" "C24" (id 0) (at 175.26 106.68 90))
     (property "Value" "22uF" (id 1) (at 180.34 106.68 90))
-    (property "Footprint" "Capacitor_SMD:C_1206_3216Metric" (id 2) (at 182.88 101.9048 0)
-      (effects (font (size 1.27 1.27)) hide)
-    )
+    (property "Footprint" "Capacitor_SMD:CP_Elec_4x4.5" (id 2) (at 182.88 101.9048 0)
+      (effects (font (size 1.27 1.27)) hide)
+    )

Commit message: gg
Parts:
- SW1: footprint Button_Switch_THT:SW_PUSH_6mm -> Button_Switch_SMD:SW_SPST_B3U-1000P
- U6: footprint Xenir:ESP32-A1S -> xenir_v6:esp32-a1s-header
Connections:
- net IO0: now also U6.6 (IO0)
Changed lines of the file:
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@@
+    )
+  )
+  (global_label "IO0" (shape input) (at 118.11 87.63 180) (fields_autoplaced)
+    (effects (font (size 1.27 1.27)) (justify right))
+    (property "Intersheet References" "${INTERSHEET_REFS}" (id 0) (at 184.15 318.77 0)
+      (effects (font (size 1.27 1.27)) hide)
     )
   )
@@
     (property "Reference" "SW1" (id 0) (at 95.25 77.0382 0))
     (property "Value" "SW_DIP_x01" (id 1) (at 95.25 79.3496 0))
-    (property "Footprint" "Button_Switch_THT:SW_PUSH_6mm" (id 2) (at 95.25 83.82 0)
+    (property "Footprint" "Button_Switch_SMD:SW_SPST_B3U-1000P" (id 2) (at 95.25 83.82 0)
       (effects (font (size 1.27 1.27)) hide)
     )
@@
     (property "Reference" "U6" (id 0) (at 138.43 64.77 0))
     (property "Value" "ESP32-A1S" (id 1) (at 138.43 67.31 0))
-    (property "Footprint" "Xenir:ESP32-A1S" (id 2) (at 123.19 67.31 0)
+    (property "Footprint" "xenir_v6:esp32-a1s-header" (id 2) (at 123.19 67.31 0)
       (effects (font (size 1.27 1.27)) (justify left bottom) hide)
     )

Commit message: gg
Parts:
- added C50, C51: 1uF, Capacitor_SMD:C_1206_3216Metric, symbol Xenir:Capacitor
- added SW4: BOOT, Button_Switch_SMD:SW_SPST_B3U-1000P, symbol Switch:SW_DIP_x01
- SW1: value SW_DIP_x01 -> RST
Connections:
- net EN: now also C51.2
- net GND: now also C50.1, C51.1, SW4.1
- net IO0: now also C50.2, SW4.2
Other:
- moved on the sheet: SW1
Changed lines of the file:
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@@
 (kicad_sch (version 20211123) (generator eeschema)
   (paper "A4")
+  (junction (at 62.23 63.5) (diameter 0) (color 0 0 0 0)
+  )
+  (junction (at 62.23 38.1) (diameter 0) (color 0 0 0 0)
+  )
   (junction (at 204.47 102.87) (diameter 0) (color 0 0 0 0)
   )
+  (junction (at 77.47 57.15) (diameter 0) (color 0 0 0 0)
+  )
   (junction (at 40.64 91.44) (diameter 0) (color 0 0 0 0)
   )
   (junction (at 214.63 100.33) (diameter 0) (color 0 0 0 0)
   )
+  (junction (at 77.47 31.75) (diameter 0) (color 0 0 0 0)
+  )
   (junction (at 39.37 110.49) (diameter 0) (color 0 0 0 0)
   )
@@
     (stroke (width 0) (type default) (color 0 0 0 0))
   )
+  (wire (pts (xy 77.47 57.15) (xy 77.47 63.5))
+    (stroke (width 0) (type default) (color 0 0 0 0))
+  )
   (wire (pts (xy 59.69 80.01) (xy 68.58 80.01))
     (stroke (width 0) (type default) (color 0 0 0 0))
@@
     (stroke (width 0) (type default) (color 0 0 0 0))
   )
+  (wire (pts (xy 62.23 38.1) (xy 62.23 31.75))
+    (stroke (width 0) (type default) (color 0 0 0 0))
+  )
   (wire (pts (xy 158.75 77.47) (xy 165.1 77.47))
     (stroke (width 0) (type default) (color 0 0 0 0))
@@
     (stroke (width 0) (type default) (color 0 0 0 0))
   )
-  (wire (pts (xy 106.68 77.47) (xy 118.11 77.47))
+  (wire (pts (xy 109.22 77.47) (xy 118.11 77.47))
     (stroke (width 0) (type default) (color 0 0 0 0))
   )
@@
     (stroke (width 0) (type default) (color 0 0 0 0))
   )
+  (wire (pts (xy 77.47 63.5) (xy 69.85 63.5))
+    (stroke (width 0) (type default) (color 0 0 0 0))
+  )
   (wire (pts (xy 158.75 102.87) (xy 175.26 102.87))
     (stroke (width 0) (type default) (color 0 0 0 0))
   )
+  (wire (pts (xy 62.23 67.31) (xy 62.23 63.5))
+    (stroke (width 0) (type default) (color 0 0 0 0))
+  )
   (wire (pts (xy 39.37 110.49) (xy 39.37 99.06))
     (stroke (width 0) (type default) (color 0 0 0 0))
@@
     (stroke (width 0) (type default) (color 0 0 0 0))
   )
+  (wire (pts (xy 62.23 63.5) (xy 62.23 57.15))
+    (stroke (width 0) (type default) (color 0 0 0 0))
+  )
   (wire (pts (xy 40.64 91.44) (xy 41.91 91.44))
     (stroke (width 0) (type default) (color 0 0 0 0))
@@
     (stroke (width 0) (type default) (color 0 0 0 0))
   )
+  (wire (pts (xy 77.47 31.75) (xy 78.74 31.75))
+    (stroke (width 0) (type default) (color 0 0 0 0))
+  )
+  (wire (pts (xy 77.47 57.15) (xy 78.74 57.15))
+    (stroke (width 0) (type default) (color 0 0 0 0))
+  )
   (wire (pts (xy 59.69 100.33) (xy 59.69 105.41))
     (stroke (width 0) (type default) (color 0 0 0 0))
@@
     (stroke (width 0) (type default) (color 0 0 0 0))
   )
+  (wire (pts (xy 62.23 41.91) (xy 62.23 38.1))
+    (stroke (width 0) (type default) (color 0 0 0 0))
+  )
   (wire (pts (xy 186.69 142.24) (xy 194.31 142.24))
     (stroke (width 0) (type default) (color 0 0 0 0))
@@
     (stroke (width 0) (type default) (color 0 0 0 0))
   )
+  (wire (pts (xy 77.47 38.1) (xy 69.85 38.1))
+    (stroke (width 0) (type default) (color 0 0 0 0))
+  )
   (wire (pts (xy 158.75 146.05) (xy 148.59 146.05))
     (stroke (width 0) (type default) (color 0 0 0 0))
   )
   (wire (pts (xy 158.75 82.55) (xy 165.1 82.55))
+    (stroke (width 0) (type default) (color 0 0 0 0))
+  )
+  (wire (pts (xy 77.47 31.75) (xy 77.47 38.1))
     (stroke (width 0) (type default) (color 0 0 0 0))
   )
@@
     )
   )
+  (global_label "IO0" (shape input) (at 78.74 31.75 0) (fields_autoplaced)
+    (effects (font (size 1.27 1.27)) (justify left))
+    (property "Intersheet References" "${INTERSHEET_REFS}" (id 0) (at 12.7 -199.39 0)
+      (effects (font (size 1.27 1.27)) hide)
+    )
+  )
   (global_label "GPIO4" (shape input) (at 133.35 143.51 180) (fields_autoplaced)
     (effects (font (size 1.27 1.27)) (justify right))
@@
     )
   )
-  (global_label "EN" (shape input) (at 102.87 83.82 0) (fields_autoplaced)
-    (effects (font (size 1.27 1.27)) (justify left))
-    (property "Intersheet References" "${INTERSHEET_REFS}" (id 0) (at 2.54 -109.22 0)
+  (global_label "EN" (shape input) (at 78.74 57.15 0) (fields_autoplaced)
+    (effects (font (size 1.27 1.27)) (justify left))
+    (property "Intersheet References" "${INTERSHEET_REFS}" (id 0) (at -21.59 -135.89 0)
       (effects (font (size 1.27 1.27)) hide)
     )
@@
     (pin "2")
   )
-  (symbol (lib_id "Switch:SW_DIP_x01") (at 95.25 83.82 0) (unit 1)
-    (in_bom yes) (on_board yes)
-    (property "Reference" "SW1" (id 0) (at 95.25 77.0382 0))
-    (property "Value" "SW_DIP_x01" (id 1) (at 95.25 79.3496 0))
-    (property "Footprint" "Button_Switch_SMD:SW_SPST_B3U-1000P" (id 2) (at 95.25 83.82 0)
-      (effects (font (size 1.27 1.27)) hide)
-    )
-    (property "Datasheet" "~" (id 3) (at 95.25 83.82 0)
+  (symbol (lib_id "Switch:SW_DIP_x01") (at 69.85 57.15 0) (unit 1)
+    (in_bom yes) (on_board yes)
+    (property "Reference" "SW1" (id 0) (at 69.85 50.3682 0))
+    (property "Value" "RST" (id 1) (at 69.85 52.6796 0))
+    (property "Footprint" "Button_Switch_SMD:SW_SPST_B3U-1000P" (id 2) (at 69.85 57.15 0)
+      (effects (font (size 1.27 1.27)) hide)
+    )
+    (property "Datasheet" "~" (id 3) (at 69.85 57.15 0)
       (effects (font (size 1.27 1.27)) hide)
     )
@@
     (pin "1")
   )
-  (symbol (lib_id "power:+3V3") (at 106.68 77.47 0) (unit 1)
-    (in_bom yes) (on_board yes)
-    (property "Reference" "#PWR0201" (id 0) (at 106.68 81.28 0)
-      (effects (font (size 1.27 1.27)) hide)
-    )
-    (property "Value" "+3V3" (id 1) (at 105.41 73.66 0))
-    (property "Footprint" "" (id 2) (at 106.68 77.47 0)
-      (effects (font (size 1.27 1.27)) hide)
-    )
-    (property "Datasheet" "" (id 3) (at 106.68 77.47 0)
+  (symbol (lib_id "power:+3V3") (at 109.22 77.47 0) (unit 1)
+    (in_bom yes) (on_board yes)
+    (property "Reference" "#PWR0201" (id 0) (at 109.22 81.28 0)
+      (effects (font (size 1.27 1.27)) hide)
+    )
+    (property "Value" "+3V3" (id 1) (at 107.95 73.66 0))
+    (property "Footprint" "" (id 2) (at 109.22 77.47 0)
+      (effects (font (size 1.27 1.27)) hide)
+    )
+    (property "Datasheet" "" (id 3) (at 109.22 77.47 0)
       (effects (font (size 1.27 1.27)) hide)
     )
@@
     (pin "7")
   )
+  (symbol (lib_id "Xenir:Capacitor") (at 66.04 63.5 0) (unit 1)
+    (in_bom yes) (on_board yes)
+    (property "Reference" "C51" (id 0) (at 63.5 62.23 0)
+      (effects (font (size 0.7112 0.7112)))
+    )
+    (property "Value" "1uF" (id 1) (at 68.58 62.23 0)
+      (effects (font (size 0.7112 0.7112)))
+    )
+    (property "Footprint" "Capacitor_SMD:C_1206_3216Metric" (id 2) (at 66.04 67.31 0)
+      (effects (font (size 1.27 1.27)) hide)
+    )
+    (property "Datasheet" "" (id 3) (at 66.04 67.31 0)
+      (effects (font (size 1.27 1.27)) hide)
+    )
+    (pin "1")
+    (pin "2")
+  )
+  (symbol (lib_id "power:GND") (at 62.23 41.91 0) (unit 1)
+    (in_bom yes) (on_board yes)
+    (property "Reference" "#PWR0205" (id 0) (at 62.23 48.26 0)
+      (effects (font (size 1.27 1.27)) hide)
+    )
+    (property "Value" "GND" (id 1) (at 62.357 46.3042 0))
+    (property "Footprint" "" (id 2) (at 62.23 41.91 0)
+      (effects (font (size 1.27 1.27)) hide)
+    )
+    (property "Datasheet" "" (id 3) (at 62.23 41.91 0)
+      (effects (font (size 1.27 1.27)) hide)
+    )
+    (pin "1")
+  )
   (symbol (lib_id "xenir:Resistor") (at 182.88 53.34 0) (unit 1)
     (in_bom yes) (on_board yes) (fields_autoplaced)
@@
     )
     (pin "1")
+  )
+  (symbol (lib_id "Switch:SW_DIP_x01") (at 69.85 31.75 0) (unit 1)
+    (in_bom yes) (on_board yes)
+    (property "Reference" "SW4" (id 0) (at 69.85 24.9682 0))
+    (property "Value" "BOOT" (id 1) (at 69.85 27.2796 0))
+    (property "Footprint" "Button_Switch_SMD:SW_SPST_B3U-1000P" (id 2) (at 69.85 31.75 0)
+      (effects (font (size 1.27 1.27)) hide)
+    )
+    (property "Datasheet" "~" (id 3) (at 69.85 31.75 0)
+      (effects (font (size 1.27 1.27)) hide)
+    )
+    (pin "1")
+    (pin "2")
   )
   (symbol (lib_id "Xenir:Capacitor") (at 204.47 106.68 90) (unit 1)
@@
     (pin "2")
   )
+  (symbol (lib_id "Xenir:Capacitor") (at 66.04 38.1 0) (unit 1)
+    (in_bom yes) (on_board yes)
+    (property "Reference" "C50" (id 0) (at 63.5 36.83 0)
+      (effects (font (size 0.7112 0.7112)))
+    )
+    (property "Value" "1uF" (id 1) (at 68.58 36.83 0)
+      (effects (font (size 0.7112 0.7112)))
+    )
+    (property "Footprint" "Capacitor_SMD:C_1206_3216Metric" (id 2) (at 66.04 41.91 0)
+      (effects (font (size 1.27 1.27)) hide)
+    )
+    (property "Datasheet" "" (id 3) (at 66.04 41.91 0)
+      (effects (font (size 1.27 1.27)) hide)
+    )
+    (pin "1")
+    (pin "2")
+  )
   (symbol (lib_id "power:GND") (at 158.75 120.65 90) (unit 1)
     (in_bom yes) (on_board yes) (fields_autoplaced)
@@
     (pin "1")
   )
-  (symbol (lib_id "power:GND") (at 87.63 83.82 0) (unit 1)
-    (in_bom yes) (on_board yes)
-    (property "Reference" "#PWR0195" (id 0) (at 87.63 90.17 0)
-      (effects (font (size 1.27 1.27)) hide)
-    )
-    (property "Value" "GND" (id 1) (at 87.757 88.2142 0))
-    (property "Footprint" "" (id 2) (at 87.63 83.82 0)
-      (effects (font (size 1.27 1.27)) hide)
-    )
-    (property "Datasheet" "" (id 3) (at 87.63 83.82 0)
-      (effects (font (size 1.27 1.27)) hide)
-    )
+  (symbol (lib_id "power:GND") (at 62.23 67.31 0) (unit 1)
+    (in_bom yes) (on_board yes)
+    (property "Reference" "#PWR0195" (id 0) (at 62.23 73.66 0)
+      (effects (font (size 1.27 1.27)) hide)
+    )
+    (property "Value" "GND" (id 1) (at 62.357 71.7042 0))
+    (property "Footprint" "" (id 2) (at 62.23 67.31 0)
+      (effects (font (size 1.27 1.27)) hide)
+    )
+    (property "Datasheet" "" (id 3) (at 62.23 67.31 0)
+      (effects (font (size 1.27 1.27)) hide)
+    )
