File: DSP.kicad_sch (KiCad schematic)
At the start: 24 parts, among them J10 Conn_01x07_Female, J11 Conn_01x04, Q4 2N3904-SMD, Q5 2N3904-SMD, Q6 AO3400A, SW1 RST, SW2 Frequency, SW3 Menu, SW4 BOOT, U6 ESP32-A1S

Commit message: gg
Changed lines of the file:
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@@
     (stroke (width 0) (type default) (color 0 0 0 0))
   )
-  (wire (pts (xy 109.22 77.47) (xy 118.11 77.47))
+  (wire (pts (xy 105.41 77.47) (xy 118.11 77.47))
     (stroke (width 0) (type default) (color 0 0 0 0))
   )
@@
     (pin "1")
   )
-  (symbol (lib_id "power:+3V3") (at 109.22 77.47 0) (unit 1)
-    (in_bom yes) (on_board yes)
-    (property "Reference" "#PWR0201" (id 0) (at 109.22 81.28 0)
-      (effects (font (size 1.27 1.27)) hide)
-    )
-    (property "Value" "+3V3" (id 1) (at 107.95 73.66 0))
-    (property "Footprint" "" (id 2) (at 109.22 77.47 0)
-      (effects (font (size 1.27 1.27)) hide)
-    )
-    (property "Datasheet" "" (id 3) (at 109.22 77.47 0)
-      (effects (font (size 1.27 1.27)) hide)
-    )
+  (symbol (lib_id "power:+3V3") (at 105.41 77.47 0) (unit 1)
+    (in_bom yes) (on_board yes)
+    (property "Reference" "#PWR0201" (id 0) (at 105.41 81.28 0)
+      (effects (font (size 1.27 1.27)) hide)
+    )
+    (property "Value" "+3V3" (id 1) (at 104.14 73.66 0))
+    (property "Footprint" "" (id 2) (at 105.41 77.47 0)
+      (effects (font (size 1.27 1.27)) hide)
+    )
+    (property "Datasheet" "" (id 3) (at 105.41 77.47 0)
+      (effects (font (size 1.27 1.27)) hide)
+    )

Commit message: added ptt
Connections:
- net PTT-IN: now reaches U6.29 (IO5)
Changed lines of the file:
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@@
+    (effects (font (size 1.27 1.27)) (justify left))
+  )
+  (hierarchical_label "PTT-IN" (shape input) (at 158.75 97.79 0)
     (effects (font (size 1.27 1.27)) (justify left))
   )

Commit message: gg
Parts:
- J10: value Conn_01x07_Female -> USB to Serial
- J11: value Conn_01x04 -> LCD
Changed lines of the file:
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@@
       (effects (font (size 1.27 1.27)) (justify left))
     )
-    (property "Value" "Conn_01x04" (id 1) (at 188.722 146.3802 90)
+    (property "Value" "LCD" (id 1) (at 188.722 146.3802 90)
       (effects (font (size 1.27 1.27)) (justify left))
     )
@@
     (in_bom yes) (on_board yes)
     (property "Reference" "J10" (id 0) (at 38.3032 52.705 0))
-    (property "Value" "Conn_01x07_Female" (id 1) (at 38.3032 55.0164 0))
+    (property "Value" "USB to Serial" (id 1) (at 38.3032 55.0164 0))
     (property "Footprint" "Connector_PinSocket_2.54mm:PinSocket_1x07_P2.54mm_Vertical" (id 2) (at 35.56 66.04 0)
       (effects (font (size 1.27 1.27)) hide)

Commit message: changed 1 to .1
Parts:
- C28, C29: value 1uF -> .1uF
Changed lines of the file:
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@@
       (effects (font (size 0.7112 0.7112)) (justify right))
     )
-    (property "Value" "1uF" (id 1) (at 217.17 104.14 90)
+    (property "Value" ".1uF" (id 1) (at 217.17 104.14 90)
       (effects (font (size 0.7112 0.7112)) (justify right))
     )
@@
       (effects (font (size 0.7112 0.7112)) (justify right))
     )
-    (property "Value" "1uF" (id 1) (at 207.01 106.68 90)
+    (property "Value" ".1uF" (id 1) (at 207.01 106.68 90)
       (effects (font (size 0.7112 0.7112)) (justify right))
     )

Commit message: moved GPIO34 to GPIO2 for encoder
Connections:
- net GPIO2: now reaches U6.11 (IO2)
- net GPIO2: now also SW3.A
- net GPIO34: no longer names the net of U6.5 (IO34)
- net GPIO34: no longer SW3.A
Changed lines of the file:
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@@
     )
   )
-  (global_label "GPIO34" (shape input) (at 118.11 85.09 180) (fields_autoplaced)
+  (global_label "GPIO2" (shape input) (at 118.11 100.33 180) (fields_autoplaced)
     (effects (font (size 1.27 1.27)) (justify right))
-    (property "Intersheet References" "${INTERSHEET_REFS}" (id 0) (at 108.8026 85.1694 0)
+    (property "Intersheet References" "${INTERSHEET_REFS}" (id 0) (at 110.0121 100.2506 0)
       (effects (font (size 1.27 1.27)) (justify right) hide)
     )
@@
     )
   )
+  (global_label "GPIO2" (shape input) (at 148.59 148.59 0) (fields_autoplaced)
+    (effects (font (size 1.27 1.27)) (justify left))
+    (property "Intersheet References" "${INTERSHEET_REFS}" (id 0) (at 156.6879 148.6694 0)
+      (effects (font (size 1.27 1.27)) (justify left) hide)
+    )
+  )
   (global_label "GPIO14" (shape input) (at 118.11 90.17 180) (fields_autoplaced)
     (effects (font (size 1.27 1.27)) (justify right))
@@
       (effects (font (size 1.27 1.27)) (justify left) hide)
     )
-  )
-  (global_label "GPIO34" (shape input) (at 148.59 148.59 0) (fields_autoplaced)
-    (effects (font (size 1.27 1.27)) (justify left))
-    (property "Intersheet References" "${INTERSHEET_REFS}" (id 0) (at 157.8974 148.5106 0)
-      (effects (font (size 1.27 1.27)) (justify left) hide)
-    )
