File: power.kicad_sch (KiCad schematic)
At the start: 10 parts, among them J9 Barrel_Jack_Switch, U8 L7805, U9 AMS1117CD-3.3

Commit message: gg
Connections:
- net +3.3V renamed +3V3
Changed lines of the file:
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@@
     (pin "2")
+  )
+  (symbol (lib_id "power:+3V3") (at 144.78 76.2 0) (unit 1)
+    (in_bom yes) (on_board yes) (fields_autoplaced)
+    (property "Reference" "#PWR0186" (id 0) (at 144.78 80.01 0)
+      (effects (font (size 1.27 1.27)) hide)
+    )
+    (property "Value" "+3V3" (id 1) (at 144.78 71.12 0))
+    (property "Footprint" "" (id 2) (at 144.78 76.2 0)
+      (effects (font (size 1.27 1.27)) hide)
+    )
+    (property "Datasheet" "" (id 3) (at 144.78 76.2 0)
+      (effects (font (size 1.27 1.27)) hide)
+    )
+    (pin "1")
   )
   (symbol (lib_id "Xenir:Resistor") (at 83.82 114.3 90) (unit 1)
@@
       (effects (font (size 1.27 1.27)) hide)
     )
-    (pin "1")
-  )
-  (symbol (lib_id "power:+3.3V") (at 144.78 76.2 0) (unit 1)
-    (in_bom yes) (on_board yes)
-    (property "Reference" "#PWR0186" (id 0) (at 144.78 80.01 0)
-      (effects (font (size 1.27 1.27)) hide)
-    )
-    (property "Value" "+3.3V" (id 1) (at 144.78 72.39 0))
-    (property "Footprint" "" (id 2) (at 144.78 76.2 0)
-      (effects (font (size 1.27 1.27)) hide)
-    )
-    (property "Datasheet" "" (id 3) (at 144.78 76.2 0)
-      (effects (font (size 1.27 1.27)) hide)
-    )
