File: mic.kicad_sch (KiCad schematic)
At the start: 0 parts

Commit message: gg
Parts:
- added C52: 10uF, Capacitor_SMD:CP_Elec_4x5.4, symbol mic-preamp-rescue:Cap_Polarized-Xenir
- added C53, C55: 100nF, Capacitor_SMD:C_1206_3216Metric, symbol mic-preamp-rescue:Capacitor-Xenir
- added C54: 330pF, Capacitor_SMD:C_1206_3216Metric, symbol mic-preamp-rescue:Capacitor-Xenir
- added J12: Conn_01x07_Female, Connector_PinHeader_2.54mm:PinHeader_1x07_P2.54mm_Vertical, symbol Connector:Conn_01x07_Female
- added R52: 5.1k, Resistor_SMD:R_0805_2012Metric, symbol mic-preamp-rescue:Resistor-Xenir
- added R53, R54: 10k, Resistor_SMD:R_0805_2012Metric, symbol mic-preamp-rescue:Resistor-Xenir
- added R55: 1k, Resistor_SMD:R_0805_2012Metric, symbol mic-preamp-rescue:Resistor-Xenir
- added R56: 100k, Resistor_SMD:R_0805_2012Metric, symbol mic-preamp-rescue:Resistor-Xenir
- added U11: LM358, xenir:SOIC8, symbol mic-preamp-rescue:LM358-Xenir
Connections:
- net MIC-OUT: now also C55.1
- new net: R53.2, R54.1, U11.5 (+IN)
- new net: C52.2, R55.1
- new net: C54.2, R55.2, R56.1, U11.6 (-IN)
- new net: C54.1, C55.2, R56.2, U11.7 (OUT)
- new net +5V: C53.1, R52.1, R53.1, U11.8 (P$V+)
- new net FREQUPDN: J12.3 (Pin_3)
- new net GND: C53.2, J12.6 (Pin_6), J12.7 (Pin_7), R54.2, U11.4 (P$V-)
- new net MICIN: C52.1, J12.1 (Pin_1), R52.2
- new net PTT: J12.5 (Pin_5)

Commit message: added ptt
Changed lines of the file:
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@@
     (stroke (width 0) (type default) (color 0 0 0 0))
-  )
-  (global_label "PTT" (shape input) (at 170.18 113.03 180) (fields_autoplaced)
-    (effects (font (size 1.27 1.27)) (justify right))
-    (property "Intersheet References" "${INTERSHEET_REFS}" (id 0) (at 8.89 22.225 0)
-      (effects (font (size 1.27 1.27)) hide)
-    )
   )
   (global_label "FREQUPDN" (shape input) (at 170.18 107.95 180) (fields_autoplaced)
@@
     )
   )
+  (hierarchical_label "PTT" (shape output) (at 170.18 113.03 180)
+    (effects (font (size 1.27 1.27)) (justify right))
+  )
   (hierarchical_label "MIC-OUT" (shape input) (at 137.16 113.03 0)

Commit message: gg
Parts:
- J12: value Conn_01x07_Female -> MIC
Changed lines of the file:
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@@
       (effects (font (size 1.27 1.27)) (justify left))
     )
-    (property "Value" "Conn_01x07_Female" (id 1) (at 175.9712 112.141 0)
+    (property "Value" "MIC" (id 1) (at 175.9712 112.141 0)
       (effects (font (size 1.27 1.27)) (justify left))
     )
