File: audio-amp.kicad_sch (KiCad schematic)
At the start: 0 parts

Commit message: gg
Parts:
- added J13: Audio_Jack, Xenir:Audio_Jack, symbol xenir:Audio_Jack
Connections:
- net AUDIO-AMP-IN: now also J13.RING, J13.RSH, J13.TIP, J13.TSH
- new net GND: J13.SLEEVE
Changed lines of the file:
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@@
 (kicad_sch (version 20211123) (generator eeschema)
   (paper "A4")
-  (hierarchical_label "AUDIO-AMP-IN" (shape input) (at 135.89 88.9 0)
+  (junction (at 121.92 71.12) (diameter 0) (color 0 0 0 0)
+  )
+  (junction (at 121.92 73.66) (diameter 0) (color 0 0 0 0)
+  )
+  (junction (at 121.92 76.2) (diameter 0) (color 0 0 0 0)
+  )
+  (wire (pts (xy 121.92 71.12) (xy 121.92 73.66))
+    (stroke (width 0) (type default) (color 0 0 0 0))
+  )
+  (wire (pts (xy 121.92 71.12) (xy 135.89 71.12))
+    (stroke (width 0) (type default) (color 0 0 0 0))
+  )
+  (wire (pts (xy 121.92 73.66) (xy 121.92 76.2))
+    (stroke (width 0) (type default) (color 0 0 0 0))
+  )
+  (wire (pts (xy 121.92 76.2) (xy 121.92 78.74))
+    (stroke (width 0) (type default) (color 0 0 0 0))
+  )
+  (hierarchical_label "AUDIO-AMP-IN" (shape input) (at 135.89 71.12 0)
     (effects (font (size 1.27 1.27)) (justify left))
   )
+  (symbol (lib_id "xenir:Audio_Jack") (at 116.84 85.09 0) (mirror x) (unit 1)
+    (in_bom yes) (on_board yes) (fields_autoplaced)
+    (property "Reference" "J13" (id 0) (at 109.22 74.9299 0)
+      (effects (font (size 1.27 1.27)) (justify right))
+    )
+    (property "Value" "Audio_Jack" (id 1) (at 109.22 77.4699 0)
+      (effects (font (size 1.27 1.27)) (justify right))
+    )
+    (property "Footprint" "Xenir:Audio_Jack" (id 2) (at 116.84 85.09 0)
+      (effects (font (size 1.27 1.27)) hide)
+    )
+    (property "Datasheet" "" (id 3) (at 116.84 85.09 0)
+      (effects (font (size 1.27 1.27)) hide)
+    )
+    (pin "RING")
+    (pin "RSH")
+    (pin "SLEEVE")
+    (pin "TIP")
+    (pin "TSH")
+  )
+  (symbol (lib_id "power:GND") (at 121.92 81.28 0) (unit 1)
+    (in_bom yes) (on_board yes) (fields_autoplaced)
+    (property "Reference" "#PWR0215" (id 0) (at 121.92 87.63 0)
+      (effects (font (size 1.27 1.27)) hide)
+    )
+    (property "Value" "GND" (id 1) (at 121.92 86.36 0))
+    (property "Footprint" "" (id 2) (at 121.92 81.28 0)
+      (effects (font (size 1.27 1.27)) hide)
+    )
+    (property "Datasheet" "" (id 3) (at 121.92 81.28 0)
+      (effects (font (size 1.27 1.27)) hide)
+    )
+    (pin "1")
+  )
 )

Commit message: gg
Parts:
- J13: value Audio_Jack -> Audio Out
Changed lines of the file:
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@@
       (effects (font (size 1.27 1.27)) (justify right))
     )
-    (property "Value" "Audio_Jack" (id 1) (at 109.22 77.4699 0)
+    (property "Value" "Audio Out" (id 1) (at 109.22 77.4699 0)
       (effects (font (size 1.27 1.27)) (justify right))
     )
