File: BPF.kicad_sch (KiCad schematic)
At the start: 8 parts, among them T1 T37-6 5:25, T2 T37-6 25:5

Commit message: removed bpf
Parts:
- removed C5, C8: 90pF, Capacitor_SMD:C_1206_3216Metric, symbol Xenir:Capacitor
- removed C6: N/C, Capacitor_SMD:C_1206_3216Metric, symbol Xenir:Capacitor
- removed C7: 12pF, Capacitor_SMD:C_1206_3216Metric, symbol Xenir:Capacitor
- removed T1: T37-6 5:25, Xenir:T37 Transformer, symbol Xenir:T37_XFRM
- removed T2: T37-6 25:5, Xenir:T37 Transformer, symbol Xenir:T37_XFRM
- removed VC1, VC2: 1-40pF, Xenir:trimcap, symbol Xenir:Trimcap
- added J2, J3: Conn_01x03_Female, Connector_PinSocket_2.54mm:PinSocket_1x03_P2.54mm_Vertical, symbol Connector:Conn_01x03_Female
Connections:
- net BPF-IN: now also J2.2 (Pin_2)
- net BPF-OUT: now also J3.2 (Pin_2)
- net GND: now also J2.1 (Pin_1), J2.3 (Pin_3), J3.1 (Pin_1), J3.3 (Pin_3)

Commit message: gg
Parts:
- J2: value Conn_01x03_Female -> IN-BPF
- J3: value Conn_01x03_Female -> OUT-LPF
Changed lines of the file:
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@@
       (effects (font (size 1.27 1.27)) (justify left))
     )
-    (property "Value" "Conn_01x03_Female" (id 1) (at 102.87 50.8 0)
+    (property "Value" "IN-BPF" (id 1) (at 102.87 50.8 0)
       (effects (font (size 1.27 1.27)) (justify left))
     )
@@
     (in_bom yes) (on_board yes) (fields_autoplaced)
     (property "Reference" "J3" (id 0) (at 144.145 48.26 0))
-    (property "Value" "Conn_01x03_Female" (id 1) (at 144.145 50.8 0))
+    (property "Value" "OUT-LPF" (id 1) (at 144.145 50.8 0))
     (property "Footprint" "Connector_PinSocket_2.54mm:PinSocket_1x03_P2.54mm_Vertical" (id 2) (at 143.51 55.88 0)
       (effects (font (size 1.27 1.27)) hide)

Commit message: gg
Parts:
- J3: value OUT-LPF -> OUT-BPF
Changed lines of the file:
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@@
     (in_bom yes) (on_board yes) (fields_autoplaced)
     (property "Reference" "J3" (id 0) (at 144.145 48.26 0))
-    (property "Value" "OUT-LPF" (id 1) (at 144.145 50.8 0))
+    (property "Value" "OUT-BPF" (id 1) (at 144.145 50.8 0))
     (property "Footprint" "Connector_PinSocket_2.54mm:PinSocket_1x03_P2.54mm_Vertical" (id 2) (at 143.51 55.88 0)
       (effects (font (size 1.27 1.27)) hide)

Commit message: added text to board
Parts:
- renumbered J3 to BPF1
Changed lines of the file:
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@@
   (symbol (lib_id "Connector:Conn_01x03_Female") (at 143.51 55.88 0) (mirror y) (unit 1)
     (in_bom yes) (on_board yes) (fields_autoplaced)
-    (property "Reference" "J3" (id 0) (at 144.145 48.26 0))
+    (property "Reference" "BPF1" (id 0) (at 144.145 48.26 0))
     (property "Value" "OUT-BPF" (id 1) (at 144.145 50.8 0))
     (property "Footprint" "Connector_PinSocket_2.54mm:PinSocket_1x03_P2.54mm_Vertical" (id 2) (at 143.51 55.88 0)
