File: LPF.kicad_sch (KiCad schematic)
At the start: 7 parts

Commit message: gg
Parts:
- removed C1: 270pF, Capacitor_SMD:C_1206_3216Metric, symbol Xenir:Capacitor
- removed C2, C3: 470pF, Capacitor_SMD:C_1206_3216Metric, symbol Xenir:Capacitor
- removed C4: 270Pf, Capacitor_SMD:C_1206_3216Metric, symbol Xenir:Capacitor
- removed L1, L2, L3: T37-6, Xenir:T37_Inductor, symbol Xenir:Inductor
- added J4, J5: Conn_01x03_Female, Connector_PinSocket_2.54mm:PinSocket_1x03_P2.54mm_Vertical, symbol Connector:Conn_01x03_Female
Connections:
- net GND: now also J4.1 (Pin_1), J4.3 (Pin_3), J5.1 (Pin_1), J5.3 (Pin_3)
- net IN-LPF: now also J4.2 (Pin_2)
- net OUT-LPF: now also J5.2 (Pin_2)

Commit message: gg
Parts:
- J4: value Conn_01x03_Female -> IN-LPF
- J5: value Conn_01x03_Female -> OUT-LPF
Changed lines of the file:
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@@
     (in_bom yes) (on_board yes) (fields_autoplaced)
     (property "Reference" "J5" (id 0) (at 146.685 76.2 0))
-    (property "Value" "Conn_01x03_Female" (id 1) (at 146.685 78.74 0))
+    (property "Value" "OUT-LPF" (id 1) (at 146.685 78.74 0))
     (property "Footprint" "Connector_PinSocket_2.54mm:PinSocket_1x03_P2.54mm_Vertical" (id 2) (at 146.05 83.82 0)
       (effects (font (size 1.27 1.27)) hide)
@@
       (effects (font (size 1.27 1.27)) (justify left))
     )
-    (property "Value" "Conn_01x03_Female" (id 1) (at 105.41 78.74 0)
+    (property "Value" "IN-LPF" (id 1) (at 105.41 78.74 0)
       (effects (font (size 1.27 1.27)) (justify left))
     )

Commit message: added text to board
Parts:
- renumbered J5 to LPF1
Changed lines of the file:
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@@
   (symbol (lib_id "Connector:Conn_01x03_Female") (at 146.05 83.82 0) (mirror y) (unit 1)
     (in_bom yes) (on_board yes) (fields_autoplaced)
-    (property "Reference" "J5" (id 0) (at 146.685 76.2 0))
+    (property "Reference" "LPF1" (id 0) (at 146.685 76.2 0))
     (property "Value" "OUT-LPF" (id 1) (at 146.685 78.74 0))
     (property "Footprint" "Connector_PinSocket_2.54mm:PinSocket_1x03_P2.54mm_Vertical" (id 2) (at 146.05 83.82 0)
