File: taylor-encoder.kicad_sch (KiCad schematic)
At the start: 0 parts

Commit message: lots of updates
Parts:
- added C17, C18, C23: .1uF, Capacitor_SMD:C_1206_3216Metric, symbol Xenir:Capacitor
- added C19, C20, C21, C22: 470nF, Capacitor_SMD:C_1206_3216Metric, symbol Xenir:Capacitor
- added R10, R7, R8, R9: 100, Resistor_SMD:R_0805_2012Metric, symbol Xenir:Resistor
- added R11, R12, R13, R14, R15, R16, R17, R18: 10k, Resistor_SMD:R_0805_2012Metric, symbol Xenir:Resistor
- added R19, R20: 50, Resistor_SMD:R_0805_2012Metric, symbol Xenir:Resistor
- added T4: T50_SPLITTER, Xenir:T50 Trifilar, symbol Xenir:T50_SPLITTER
- added U3: FST3253, Xenir:SO16, symbol Xenir:FST3253
- added U4, U5: LM4562, Xenir:SO08, symbol Amplifier_Operational:LM358
Connections:
- net 0-Degree: now also U3.2 (S1)
- net 90-Degree: now also U3.14 (S0)
- net Encoder-Out: now also T4.C1B
- new net: R14.2, R15.1, U5.2 (-)
- new net: R15.2, R17.1, R9.1, U5.1
- new net: R11.2, R16.1, R7.1, U4.1
- new net: R20.1, U3.7 (1A)
- new net: R19.1, U3.9 (2A)
- new net: R19.2, T4.C2B
- new net: R20.2, T4.C3A
- new net: R12.1, R16.2, U4.6 (-)
- new net: R12.2, R8.1, U4.7
- new net: R11.1, R13.2, U4.2 (-)
- new net: R17.2, R18.1, U5.6 (-)
- new net: R10.1, R18.2, U5.7
- new net +12V: C18.2, C23.2, U4.8 (V+), U5.8 (V+)
- new net +2V5: T4.C2A, T4.C3B, U4.3 (+), U4.5 (+), U5.3 (+), U5.5 (+)
- new net +5V: C17.2, U3.16 (VCC)
- new net Encoder-0: C19.2, R7.2, U3.13 (2B4), U3.6 (1B1)
- new net Encoder-180: C20.2, R8.2, U3.10 (2B1), U3.3 (1B4)
- new net Encoder-270: C22.2, R10.2, U3.11 (2B2), U3.4 (1B3)
- new net Encoder-90: C21.2, R9.2, U3.12 (2B3), U3.5 (1B2)
- new net Encoder-I: R13.1
- new net Encoder-Q: R14.1
- new net GND: C17.1, C18.1, C19.1, C20.1, C21.1, C22.1, C23.1, T4.C1A, U3.1 (OE1), U3.15 (OE2), U3.8 (GND), U4.4 (V-), U5.4 (V-)

Commit message: added caps in encoder
Parts:
- added C5, C6, C7, C8: 10uF, Capacitor_SMD:CP_Elec_4x4.5, symbol Xenir:Cap_Polarized
Connections:
- net at R15.2, R17.1, U5.1: now also C7.1; no longer R9.1
- net at R11.2, R16.1, U4.1: now also C5.1; no longer R7.1
- net at R12.2, U4.7: now also C6.1; no longer R8.1
- net at R18.2, U5.7: now also C8.1; no longer R10.1
- new net: C5.2, R7.1
- new net: C8.2, R10.1
- new net: C7.2, R9.1
- new net: C6.2, R8.1
Changed lines of the file:
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@@
   (junction (at 85.09 60.96) (diameter 0) (color 0 0 0 0)
   )
+  (wire (pts (xy 119.38 132.08) (xy 120.65 132.08))
+    (stroke (width 0) (type default) (color 0 0 0 0))
+  )
   (wire (pts (xy 107.95 105.41) (xy 107.95 96.52))
     (stroke (width 0) (type default) (color 0 0 0 0))
@@
     (stroke (width 0) (type default) (color 0 0 0 0))
   )
+  (wire (pts (xy 111.76 92.71) (xy 62.23 92.71))
+    (stroke (width 0) (type default) (color 0 0 0 0))
+  )
   (wire (pts (xy 238.76 135.89) (xy 238.76 147.32))
     (stroke (width 0) (type default) (color 0 0 0 0))
@@
     (stroke (width 0) (type default) (color 0 0 0 0))
   )
-  (wire (pts (xy 107.95 132.08) (xy 120.65 132.08))
+  (wire (pts (xy 119.38 105.41) (xy 120.65 105.41))
+    (stroke (width 0) (type default) (color 0 0 0 0))
+  )
+  (wire (pts (xy 107.95 132.08) (xy 111.76 132.08))
     (stroke (width 0) (type default) (color 0 0 0 0))
   )
@@
     (stroke (width 0) (type default) (color 0 0 0 0))
   )
-  (wire (pts (xy 120.65 119.38) (xy 62.23 119.38))
+  (wire (pts (xy 120.65 119.38) (xy 119.38 119.38))
     (stroke (width 0) (type default) (color 0 0 0 0))
   )
@@
     (stroke (width 0) (type default) (color 0 0 0 0))
   )
-  (wire (pts (xy 120.65 92.71) (xy 62.23 92.71))
+  (wire (pts (xy 120.65 92.71) (xy 119.38 92.71))
     (stroke (width 0) (type default) (color 0 0 0 0))
   )
@@
     (stroke (width 0) (type default) (color 0 0 0 0))
   )
+  (wire (pts (xy 111.76 119.38) (xy 62.23 119.38))
+    (stroke (width 0) (type default) (color 0 0 0 0))
+  )
   (wire (pts (xy 62.23 123.19) (xy 62.23 132.08))
     (stroke (width 0) (type default) (color 0 0 0 0))
@@
     (stroke (width 0) (type default) (color 0 0 0 0))
   )
-  (wire (pts (xy 107.95 105.41) (xy 120.65 105.41))
+  (wire (pts (xy 107.95 105.41) (xy 111.76 105.41))
     (stroke (width 0) (type default) (color 0 0 0 0))
   )
@@
     )
     (property "Datasheet" "" (id 3) (at 50.8 125.73 0)
+      (effects (font (size 1.27 1.27)) hide)
+    )
+    (pin "1")
+    (pin "2")
+  )
+  (symbol (lib_id "Xenir:Cap_Polarized") (at 115.57 90.17 0) (unit 1)
+    (in_bom yes) (on_board yes)
+    (property "Reference" "C5" (id 0) (at 113.03 91.44 0)
+      (effects (font (size 0.7112 0.7112)))
+    )
+    (property "Value" "10uF" (id 1) (at 118.11 91.44 0)
+      (effects (font (size 0.7112 0.7112)))
+    )
+    (property "Footprint" "Capacitor_SMD:CP_Elec_4x4.5" (id 2) (at 115.57 88.9 0)
+      (effects (font (size 1.27 1.27)) hide)
+    )
+    (property "Datasheet" "" (id 3) (at 115.57 88.9 0)
       (effects (font (size 1.27 1.27)) hide)
     )
@@
     (pin "1")
   )
+  (symbol (lib_id "Xenir:Cap_Polarized") (at 115.57 129.54 0) (unit 1)
+    (in_bom yes) (on_board yes)
+    (property "Reference" "C8" (id 0) (at 113.03 130.81 0)
+      (effects (font (size 0.7112 0.7112)))
+    )
+    (property "Value" "10uF" (id 1) (at 118.11 130.81 0)
+      (effects (font (size 0.7112 0.7112)))
+    )
+    (property "Footprint" "Capacitor_SMD:CP_Elec_4x4.5" (id 2) (at 115.57 128.27 0)
+      (effects (font (size 1.27 1.27)) hide)
+    )
+    (property "Datasheet" "" (id 3) (at 115.57 128.27 0)
+      (effects (font (size 1.27 1.27)) hide)
+    )
+    (pin "1")
+    (pin "2")
+  )
   (symbol (lib_id "power:GND") (at 203.2 123.19 0) (unit 1)
     (in_bom yes) (on_board yes)
@@
     (pin "2")
   )
+  (symbol (lib_id "Xenir:Cap_Polarized") (at 115.57 116.84 0) (unit 1)
+    (in_bom yes) (on_board yes)
+    (property "Reference" "C7" (id 0) (at 113.03 118.11 0)
+      (effects (font (size 0.7112 0.7112)))
+    )
+    (property "Value" "10uF" (id 1) (at 118.11 118.11 0)
+      (effects (font (size 0.7112 0.7112)))
+    )
+    (property "Footprint" "Capacitor_SMD:CP_Elec_4x4.5" (id 2) (at 115.57 115.57 0)
+      (effects (font (size 1.27 1.27)) hide)
+    )
+    (property "Datasheet" "" (id 3) (at 115.57 115.57 0)
+      (effects (font (size 1.27 1.27)) hide)
+    )
+    (pin "1")
+    (pin "2")
+  )
   (symbol (lib_id "Xenir:Capacitor") (at 74.93 71.12 90) (unit 1)
     (in_bom yes) (on_board yes) (fields_autoplaced)
@@
     (pin "1")
   )
+  (symbol (lib_id "Xenir:Cap_Polarized") (at 115.57 102.87 0) (unit 1)
+    (in_bom yes) (on_board yes)
+    (property "Reference" "C6" (id 0) (at 113.03 104.14 0)
+      (effects (font (size 0.7112 0.7112)))
+    )
+    (property "Value" "10uF" (id 1) (at 118.11 104.14 0)
+      (effects (font (size 0.7112 0.7112)))
+    )
+    (property "Footprint" "Capacitor_SMD:CP_Elec_4x4.5" (id 2) (at 115.57 101.6 0)
+      (effects (font (size 1.27 1.27)) hide)
+    )
+    (property "Datasheet" "" (id 3) (at 115.57 101.6 0)
+      (effects (font (size 1.27 1.27)) hide)
+    )
+    (pin "1")
+    (pin "2")
+  )
   (symbol (lib_id "Xenir:Resistor") (at 195.58 69.85 90) (unit 1)

Commit message: separated 2.5v for encoder
Parts:
- added C48, C49: 10uF, Capacitor_SMD:CP_Elec_4x4.5, symbol Xenir:Cap_Polarized
- added R48, R49, R50, R51: 10k, Resistor_SMD:R_0805_2012Metric, symbol Xenir:Resistor
Connections:
- net +5V: now also R48.2, R50.2
- net GND: now also C48.2, C49.2, R49.1, R51.1
- net +2V5 renamed Encoder2.5
- net Encoder2.5: now also C48.1, R48.1, R49.2; no longer T4.C2A, T4.C3B
- new net: C49.1, R50.1, R51.2, T4.C2A, T4.C3B

Commit message: updated opamp voltage - thanks andre!
Connections:
- net +12V is gone; now on net +5V: C18.2, C23.2, U4.8 (V+), U5.8 (V+)
Changed lines of the file:
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@@
     (pin "2")
+  )
+  (symbol (lib_id "power:+5V") (at 113.03 58.42 0) (unit 1)
+    (in_bom yes) (on_board yes) (fields_autoplaced)
+    (property "Reference" "#PWR0133" (id 0) (at 113.03 62.23 0)
+      (effects (font (size 1.27 1.27)) hide)
+    )
+    (property "Value" "+5V" (id 1) (at 113.03 53.34 0))
+    (property "Footprint" "" (id 2) (at 113.03 58.42 0)
+      (effects (font (size 1.27 1.27)) hide)
+    )
+    (property "Datasheet" "" (id 3) (at 113.03 58.42 0)
+      (effects (font (size 1.27 1.27)) hide)
+    )
+    (pin "1")
   )
   (symbol (lib_id "Xenir:Cap_Polarized") (at 115.57 129.54 0) (unit 1)
@@
     (pin "8")
   )
-  (symbol (lib_id "power:+12V") (at 85.09 58.42 0) (unit 1)
-    (in_bom yes) (on_board yes) (fields_autoplaced)
-    (property "Reference" "#PWR0126" (id 0) (at 85.09 62.23 0)
-      (effects (font (size 1.27 1.27)) hide)
-    )
-    (property "Value" "+12V" (id 1) (at 85.09 53.34 0))
-    (property "Footprint" "" (id 2) (at 85.09 58.42 0)
-      (effects (font (size 1.27 1.27)) hide)
-    )
-    (property "Datasheet" "" (id 3) (at 85.09 58.42 0)
-      (effects (font (size 1.27 1.27)) hide)
-    )
-    (pin "1")
-  )
   (symbol (lib_id "Xenir:Resistor") (at 142.24 64.77 90) (unit 1)
     (in_bom yes) (on_board yes)
@@
     (pin "1")
   )
+  (symbol (lib_id "power:+5V") (at 85.09 58.42 0) (unit 1)
+    (in_bom yes) (on_board yes) (fields_autoplaced)
+    (property "Reference" "#PWR0126" (id 0) (at 85.09 62.23 0)
+      (effects (font (size 1.27 1.27)) hide)
+    )
+    (property "Value" "+5V" (id 1) (at 85.09 53.34 0))
+    (property "Footprint" "" (id 2) (at 85.09 58.42 0)
+      (effects (font (size 1.27 1.27)) hide)
+    )
+    (property "Datasheet" "" (id 3) (at 85.09 58.42 0)
+      (effects (font (size 1.27 1.27)) hide)
+    )
+    (pin "1")
+  )
   (symbol (lib_id "power:+5V") (at 220.98 91.44 0) (unit 1)
     (in_bom yes) (on_board yes) (fields_autoplaced)
@@
     (pin "2")
   )
-  (symbol (lib_id "power:+12V") (at 113.03 58.42 0) (unit 1)
-    (in_bom yes) (on_board yes) (fields_autoplaced)
-    (property "Reference" "#PWR0133" (id 0) (at 113.03 62.23 0)
-      (effects (font (size 1.27 1.27)) hide)
-    )
-    (property "Value" "+12V" (id 1) (at 113.03 53.34 0))
-    (property "Footprint" "" (id 2) (at 113.03 58.42 0)
-      (effects (font (size 1.27 1.27)) hide)
-    )
-    (property "Datasheet" "" (id 3) (at 113.03 58.42 0)
-      (effects (font (size 1.27 1.27)) hide)
-    )
-    (pin "1")
-  )
   (symbol (lib_id "Xenir:Resistor") (at 35.56 129.54 0) (unit 1)

Commit message: gg
Parts:
- T4: value T50_SPLITTER -> T50_COMBINER
Changed lines of the file:
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@@
     (in_bom yes) (on_board yes) (fields_autoplaced)
     (property "Reference" "T4" (id 0) (at 229.3874 41.91 0))
-    (property "Value" "T50_SPLITTER" (id 1) (at 229.3874 44.45 0))
+    (property "Value" "T50_COMBINER" (id 1) (at 229.3874 44.45 0))
     (property "Footprint" "Xenir:T50 Trifilar" (id 2) (at 229.87 41.91 0)
       (effects (font (size 1.27 1.27)) hide)

Commit message: gg
Other:
- moved on the sheet: R10
Changed lines of the file:
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@@
   (junction (at 85.09 60.96) (diameter 0) (color 0 0 0 0)
   )
-  (wire (pts (xy 119.38 132.08) (xy 120.65 132.08))
-    (stroke (width 0) (type default) (color 0 0 0 0))
-  )
   (wire (pts (xy 107.95 105.41) (xy 107.95 96.52))
     (stroke (width 0) (type default) (color 0 0 0 0))
@@
   )
   (wire (pts (xy 201.93 130.81) (xy 203.2 130.81))
+    (stroke (width 0) (type default) (color 0 0 0 0))
+  )
+  (wire (pts (xy 129.54 132.08) (xy 130.81 132.08))
     (stroke (width 0) (type default) (color 0 0 0 0))
   )
@@
     (pin "1")
   )
-  (symbol (lib_id "Xenir:Resistor") (at 125.73 132.08 0) (unit 1)
-    (in_bom yes) (on_board yes)
-    (property "Reference" "R10" (id 0) (at 127 134.62 0)
-      (effects (font (size 0.7112 0.7112)))
-    )
-    (property "Value" "100" (id 1) (at 124.46 134.62 0)
-      (effects (font (size 0.7112 0.7112)))
-    )
-    (property "Footprint" "Resistor_SMD:R_0805_2012Metric" (id 2) (at 125.73 134.62 0)
-      (effects (font (size 1.27 1.27)) hide)
-    )
-    (property "Datasheet" "" (id 3) (at 125.73 134.62 0)
-      (effects (font (size 1.27 1.27)) hide)
-    )
+  (symbol (lib_id "Xenir:Resistor") (at 124.46 132.08 0) (unit 1)
+    (in_bom yes) (on_board yes)
+    (property "Reference" "R10" (id 0) (at 125.73 134.62 0)
+      (effects (font (size 0.7112 0.7112)))
+    )
+    (property "Value" "100" (id 1) (at 123.19 134.62 0)
+      (effects (font (size 0.7112 0.7112)))
+    )
+    (property "Footprint" "Resistor_SMD:R_0805_2012Metric" (id 2) (at 124.46 134.62 0)
+      (effects (font (size 1.27 1.27)) hide)
+    )
+    (property "Datasheet" "" (id 3) (at 124.46 134.62 0)
+      (effects (font (size 1.27 1.27)) hide)
+    )

Commit message: added more decoupling caps
Parts:
- added C57, C58: .1uF, Capacitor_SMD:C_1206_3216Metric, symbol Xenir:Capacitor
Connections:
- net Encoder2.5: now also C57.2
- net GND: now also C57.1, C58.1
- net at C49.1, R50.1, R51.2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: now also C58.2
Changed lines of the file:
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@@
   (junction (at 62.23 105.41) (diameter 0) (color 0 0 0 0)
   )
+  (junction (at 208.28 59.69) (diameter 0) (color 0 0 0 0)
+  )
   (junction (at 107.95 105.41) (diameter 0) (color 0 0 0 0)
   )
@@
   (junction (at 85.09 102.87) (diameter 0) (color 0 0 0 0)
   )
+  (junction (at 134.62 69.85) (diameter 0) (color 0 0 0 0)
+  )
   (junction (at 62.23 96.52) (diameter 0) (color 0 0 0 0)
   )
@@
     (stroke (width 0) (type default) (color 0 0 0 0))
   )
+  (wire (pts (xy 201.93 59.69) (xy 208.28 59.69))
+    (stroke (width 0) (type default) (color 0 0 0 0))
+  )
   (wire (pts (xy 200.66 74.93) (xy 200.66 72.39))
+    (stroke (width 0) (type default) (color 0 0 0 0))
+  )
+  (wire (pts (xy 127 69.85) (xy 134.62 69.85))
     (stroke (width 0) (type default) (color 0 0 0 0))
   )
@@
     (pin "1")
   )
+  (symbol (lib_id "Xenir:Capacitor") (at 201.93 63.5 90) (unit 1)
+    (in_bom yes) (on_board yes)
+    (property "Reference" "C58" (id 0) (at 199.39 60.96 90)
+      (effects (font (size 0.7112 0.7112)) (justify right))
+    )
+    (property "Value" ".1uF" (id 1) (at 203.2 60.96 90)
+      (effects (font (size 0.7112 0.7112)) (justify right))
+    )
+    (property "Footprint" "Capacitor_SMD:C_1206_3216Metric" (id 2) (at 205.74 63.5 0)
+      (effects (font (size 1.27 1.27)) hide)
+    )
+    (property "Datasheet" "" (id 3) (at 205.74 63.5 0)
+      (effects (font (size 1.27 1.27)) hide)
+    )
+    (pin "1")
+    (pin "2")
+  )
   (symbol (lib_id "power:+5V") (at 85.09 58.42 0) (unit 1)
     (in_bom yes) (on_board yes) (fields_autoplaced)
@@
     )
     (pin "1")
+  )
+  (symbol (lib_id "Xenir:Capacitor") (at 127 73.66 90) (unit 1)
+    (in_bom yes) (on_board yes)
+    (property "Reference" "C57" (id 0) (at 124.46 71.12 90)
+      (effects (font (size 0.7112 0.7112)) (justify right))
+    )
+    (property "Value" ".1uF" (id 1) (at 128.27 71.12 90)
+      (effects (font (size 0.7112 0.7112)) (justify right))
+    )
+    (property "Footprint" "Capacitor_SMD:C_1206_3216Metric" (id 2) (at 130.81 73.66 0)
+      (effects (font (size 1.27 1.27)) hide)
+    )
+    (property "Datasheet" "" (id 3) (at 130.81 73.66 0)
+      (effects (font (size 1.27 1.27)) hide)
+    )
+    (pin "1")
+    (pin "2")
   )
   (symbol (lib_id "power:GND") (at 215.9 69.85 0) (unit 1)
@@
     (pin "2")
   )
+  (symbol (lib_id "power:GND") (at 201.93 67.31 0) (unit 1)
+    (in_bom yes) (on_board yes)
+    (property "Reference" "#PWR0217" (id 0) (at 201.93 73.66 0)
+      (effects (font (size 1.27 1.27)) hide)
+    )
+    (property "Value" "GND" (id 1) (at 199.39 67.31 0))
+    (property "Footprint" "" (id 2) (at 201.93 67.31 0)
+      (effects (font (size 1.27 1.27)) hide)
+    )
+    (property "Datasheet" "" (id 3) (at 201.93 67.31 0)
+      (effects (font (size 1.27 1.27)) hide)
+    )
+    (pin "1")
+  )
   (symbol (lib_id "Xenir:Capacitor") (at 213.36 96.52 90) (unit 1)
     (in_bom yes) (on_board yes)
@@
       (effects (font (size 1.27 1.27)) hide)
     )
+    (pin "1")
+  )
+  (symbol (lib_id "power:GND") (at 127 77.47 0) (unit 1)
+    (in_bom yes) (on_board yes)
+    (property "Reference" "#PWR0218" (id 0) (at 127 83.82 0)
+      (effects (font (size 1.27 1.27)) hide)
+    )
+    (property "Value" "GND" (id 1) (at 124.46 77.47 0))
+    (property "Footprint" "" (id 2) (at 127 77.47 0)
+      (effects (font (size 1.27 1.27)) hide)
+    )
+    (property "Datasheet" "" (id 3) (at 127 77.47 0)
+      (effects (font (size 1.27 1.27)) hide)
+    )
