File: local-oscillator.kicad_sch (KiCad schematic)
At the start: 0 parts

Commit message: more updates
Changed lines of the file:
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@@
 (kicad_sch (version 20211123) (generator eeschema)
   (paper "A4")
+  (hierarchical_label "SDA" (shape input) (at 114.3 100.33 0)
+    (effects (font (size 1.27 1.27)) (justify left))
+  )
   (hierarchical_label "90-Degree" (shape output) (at 134.62 100.33 0)
     (effects (font (size 1.27 1.27)) (justify left))
@@
     (effects (font (size 1.27 1.27)) (justify left))
   )
+  (hierarchical_label "SCL" (shape input) (at 114.3 95.25 0)
+    (effects (font (size 1.27 1.27)) (justify left))
+  )

Commit message: added LO
Parts:
- added U10: si5351, Xenir:si5351, symbol Xenir:si5351
Connections:
- net 0-Degree: now also U10.0
- net 90-Degree: now also U10.2
- net SCL: now also U10.SCL
- net SDA: now also U10.SDA
- new net +5V: U10.VIN
- new net GND: U10.GND
Changed lines of the file:
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@@
 (kicad_sch (version 20211123) (generator eeschema)
   (paper "A4")
-  (hierarchical_label "SDA" (shape input) (at 114.3 100.33 0)
+  (hierarchical_label "SDA" (shape input) (at 142.24 62.23 0)
     (effects (font (size 1.27 1.27)) (justify left))
   )
-  (hierarchical_label "90-Degree" (shape output) (at 134.62 100.33 0)
+  (hierarchical_label "90-Degree" (shape output) (at 106.68 69.85 180)
+    (effects (font (size 1.27 1.27)) (justify right))
+  )
+  (hierarchical_label "0-Degree" (shape output) (at 106.68 59.69 180)
+    (effects (font (size 1.27 1.27)) (justify right))
+  )
+  (hierarchical_label "SCL" (shape input) (at 142.24 67.31 0)
     (effects (font (size 1.27 1.27)) (justify left))
   )
-  (hierarchical_label "0-Degree" (shape output) (at 134.62 95.25 0)
-    (effects (font (size 1.27 1.27)) (justify left))
+  (symbol (lib_id "power:+5V") (at 124.46 52.07 0) (unit 1)
+    (in_bom yes) (on_board yes) (fields_autoplaced)
+    (property "Reference" "#PWR0198" (id 0) (at 124.46 55.88 0)
+      (effects (font (size 1.27 1.27)) hide)
+    )
+    (property "Value" "+5V" (id 1) (at 124.46 46.99 0))
+    (property "Footprint" "" (id 2) (at 124.46 52.07 0)
+      (effects (font (size 1.27 1.27)) hide)
+    )
+    (property "Datasheet" "" (id 3) (at 124.46 52.07 0)
+      (effects (font (size 1.27 1.27)) hide)
+    )
+    (pin "1")
   )
-  (hierarchical_label "SCL" (shape input) (at 114.3 95.25 0)
-    (effects (font (size 1.27 1.27)) (justify left))
+  (symbol (lib_id "Xenir:si5351") (at 130.81 54.61 0) (unit 1)
+    (in_bom yes) (on_board yes) (fields_autoplaced)
+    (property "Reference" "U10" (id 0) (at 126.4794 52.07 0)
+      (effects (font (size 1.27 1.27)) (justify left))
+    )
+    (property "Value" "si5351" (id 1) (at 126.4794 54.61 0)
+      (effects (font (size 1.27 1.27)) (justify left))
+    )
+    (property "Footprint" "Xenir:si5351" (id 2) (at 123.19 66.04 0)
+      (effects (font (size 1.27 1.27)) hide)
+    )
+    (property "Datasheet" "" (id 3) (at 123.19 66.04 0)
+      (effects (font (size 1.27 1.27)) hide)
+    )
+    (pin "0")
+    (pin "1")
+    (pin "2")
+    (pin "GND")
+    (pin "SCL")
+    (pin "SDA")
+    (pin "VIN")
+  )
+  (symbol (lib_id "power:GND") (at 124.46 80.01 0) (unit 1)
+    (in_bom yes) (on_board yes) (fields_autoplaced)
+    (property "Reference" "#PWR0197" (id 0) (at 124.46 86.36 0)
+      (effects (font (size 1.27 1.27)) hide)
+    )
+    (property "Value" "GND" (id 1) (at 124.46 85.09 0))
+    (property "Footprint" "" (id 2) (at 124.46 80.01 0)
+      (effects (font (size 1.27 1.27)) hide)
+    )
+    (property "Datasheet" "" (id 3) (at 124.46 80.01 0)
+      (effects (font (size 1.27 1.27)) hide)
+    )
+    (pin "1")
   )
 )

Commit message: fixed 5v to 3.3v
Connections:
- net +5V renamed +3V3
Changed lines of the file:
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@@
     (effects (font (size 1.27 1.27)) (justify left))
-  )
-  (symbol (lib_id "power:+5V") (at 124.46 52.07 0) (unit 1)
-    (in_bom yes) (on_board yes) (fields_autoplaced)
-    (property "Reference" "#PWR0198" (id 0) (at 124.46 55.88 0)
-      (effects (font (size 1.27 1.27)) hide)
-    )
-    (property "Value" "+5V" (id 1) (at 124.46 46.99 0))
-    (property "Footprint" "" (id 2) (at 124.46 52.07 0)
-      (effects (font (size 1.27 1.27)) hide)
-    )
-    (property "Datasheet" "" (id 3) (at 124.46 52.07 0)
-      (effects (font (size 1.27 1.27)) hide)
-    )
-    (pin "1")
   )
   (symbol (lib_id "Xenir:si5351") (at 130.81 54.61 0) (unit 1)
@@
       (effects (font (size 1.27 1.27)) hide)
     )
+    (pin "1")
+  )
+  (symbol (lib_id "power:+3V3") (at 124.46 52.07 0) (unit 1)
+    (in_bom yes) (on_board yes) (fields_autoplaced)
+    (property "Reference" "#PWR?" (id 0) (at 124.46 55.88 0)
+      (effects (font (size 1.27 1.27)) hide)
+    )
+    (property "Value" "+3V3" (id 1) (at 124.46 46.99 0))
+    (property "Footprint" "" (id 2) (at 124.46 52.07 0)
+      (effects (font (size 1.27 1.27)) hide)
+    )
+    (property "Datasheet" "" (id 3) (at 124.46 52.07 0)
+      (effects (font (size 1.27 1.27)) hide)
+    )

Commit message: dd
Parts:
- U10: footprint Xenir:si5351 -> xenir:si5351
Changed lines of the file:
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@@
       (effects (font (size 1.27 1.27)) (justify left))
     )
-    (property "Footprint" "Xenir:si5351" (id 2) (at 123.19 66.04 0)
+    (property "Footprint" "xenir:si5351" (id 2) (at 123.19 66.04 0)
       (effects (font (size 1.27 1.27)) hide)
     )
