File: DSP-new.kicad_sch (KiCad schematic)
At the start: 16 parts, among them J11 LCD, Q6 AO3400A, SW2 Frequency, SW3 Menu, U12 PCBARTISTS-ES8388, U6 ESP32-S3

Commit message: more updates
Connections:
- net +3V3: no longer U6.1 (3V3), U6.2 (3V3)
- net GPIO15: now also SW3.A; no longer SW3.B
- net GPIO7: now also SW3.B; no longer SW3.A
- net PTT-IN: now also U6.39 (GPIO42); no longer U6.12 (GPIO8)
- net SCL: now also U6.32 (GPIO35); no longer U6.10 (GPIO17)
- net SDA: now also U6.33 (GPIO36); no longer U6.11 (GPIO18)
- net GPIO37: now reaches U6.34 (GPIO37)
- net GPIO37: now also R46.1
- net GPIO10: no longer names the net of U6.16 (GPIO10)
- net GPIO10: no longer R46.1
Changed lines of the file:
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@@
   (junction (at 102.87 92.71) (diameter 0) (color 0 0 0 0)
   )
-  (junction (at 59.69 36.83) (diameter 0) (color 0 0 0 0)
-  )
-  (wire (pts (xy 57.15 64.77) (xy 62.23 64.77))
-    (stroke (width 0) (type default) (color 0 0 0 0))
-  )
   (wire (pts (xy 173.99 72.39) (xy 191.77 72.39))
     (stroke (width 0) (type default) (color 0 0 0 0))
@@
     (stroke (width 0) (type default) (color 0 0 0 0))
   )
-  (wire (pts (xy 57.15 59.69) (xy 62.23 59.69))
-    (stroke (width 0) (type default) (color 0 0 0 0))
-  )
   (wire (pts (xy 173.99 74.93) (xy 180.34 74.93))
     (stroke (width 0) (type default) (color 0 0 0 0))
@@
     (stroke (width 0) (type default) (color 0 0 0 0))
   )
-  (wire (pts (xy 57.15 62.23) (xy 62.23 62.23))
-    (stroke (width 0) (type default) (color 0 0 0 0))
-  )
   (wire (pts (xy 173.99 58.42) (xy 186.69 58.42))
     (stroke (width 0) (type default) (color 0 0 0 0))
@@
     (stroke (width 0) (type default) (color 0 0 0 0))
   )
-  (wire (pts (xy 62.23 39.37) (xy 59.69 39.37))
-    (stroke (width 0) (type default) (color 0 0 0 0))
-  )
   (wire (pts (xy 226.06 49.53) (xy 226.06 55.88))
     (stroke (width 0) (type default) (color 0 0 0 0))
@@
     (stroke (width 0) (type default) (color 0 0 0 0))
   )
-  (wire (pts (xy 59.69 39.37) (xy 59.69 36.83))
-    (stroke (width 0) (type default) (color 0 0 0 0))
-  )
   (wire (pts (xy 114.3 130.81) (xy 104.14 130.81))
     (stroke (width 0) (type default) (color 0 0 0 0))
   )
-  (wire (pts (xy 59.69 36.83) (xy 62.23 36.83))
-    (stroke (width 0) (type default) (color 0 0 0 0))
-  )
   (wire (pts (xy 191.77 130.81) (xy 194.31 130.81))
     (stroke (width 0) (type default) (color 0 0 0 0))
@@
     )
   )
-  (global_label "GPIO10" (shape input) (at 181.61 130.81 180) (fields_autoplaced)
+  (global_label "GPIO37" (shape input) (at 181.61 130.81 180) (fields_autoplaced)
     (effects (font (size 1.27 1.27)) (justify right))
     (property "Intersheet References" "${INTERSHEET_REFS}" (id 0) (at 172.3026 130.7306 0)
@@
     )
   )
-  (global_label "GPIO10" (shape input) (at 62.23 74.93 180) (fields_autoplaced)
-    (effects (font (size 1.27 1.27)) (justify right))
-    (property "Intersheet References" "${INTERSHEET_REFS}" (id 0) (at 52.9226 74.8506 0)
-      (effects (font (size 1.27 1.27)) (justify right) hide)
+  (global_label "GPIO37" (shape input) (at 102.87 62.23 0) (fields_autoplaced)
+    (effects (font (size 1.27 1.27)) (justify left))
+    (property "Intersheet References" "${INTERSHEET_REFS}" (id 0) (at 112.1774 62.1506 0)
+      (effects (font (size 1.27 1.27)) (justify left) hide)
     )
   )
@@
     )
   )
-  (global_label "GPIO7" (shape input) (at 104.14 133.35 0) (fields_autoplaced)
-    (effects (font (size 1.27 1.27)) (justify left))
-    (property "Intersheet References" "${INTERSHEET_REFS}" (id 0) (at 112.2379 133.2706 0)
-      (effects (font (size 1.27 1.27)) (justify left) hide)
-    )
-  )
-  (global_label "GPIO15" (shape input) (at 104.14 128.27 0) (fields_autoplaced)
-    (effects (font (size 1.27 1.27)) (justify left))
-    (property "Intersheet References" "${INTERSHEET_REFS}" (id 0) (at 113.4474 128.1906 0)
+  (global_label "GPIO7" (shape input) (at 104.14 128.27 0) (fields_autoplaced)
+    (effects (font (size 1.27 1.27)) (justify left))
+    (property "Intersheet References" "${INTERSHEET_REFS}" (id 0) (at 112.2379 128.1906 0)
+      (effects (font (size 1.27 1.27)) (justify left) hide)
+    )
+  )
+  (global_label "GPIO15" (shape input) (at 104.14 133.35 0) (fields_autoplaced)
+    (effects (font (size 1.27 1.27)) (justify left))
+    (property "Intersheet References" "${INTERSHEET_REFS}" (id 0) (at 113.4474 133.2706 0)
       (effects (font (size 1.27 1.27)) (justify left) hide)
     )
@@
     (effects (font (size 1.27 1.27)) (justify left))
   )
-  (hierarchical_label "SDA" (shape output) (at 57.15 62.23 180)
-    (effects (font (size 1.27 1.27)) (justify right))
+  (hierarchical_label "SDA" (shape output) (at 102.87 64.77 0)
+    (effects (font (size 1.27 1.27)) (justify left))
   )
   (hierarchical_label "SDA" (shape output) (at 128.27 77.47 180)
@@
     (effects (font (size 1.27 1.27)) (justify left))
   )
-  (hierarchical_label "SCL" (shape output) (at 57.15 59.69 180)
-    (effects (font (size 1.27 1.27)) (justify right))
+  (hierarchical_label "SCL" (shape output) (at 102.87 67.31 0)
+    (effects (font (size 1.27 1.27)) (justify left))
   )
   (hierarchical_label "DSP-INL" (shape input) (at 203.2 72.39 0)
     (effects (font (size 1.27 1.27)) (justify left))
   )
-  (hierarchical_label "PTT-IN" (shape input) (at 57.15 64.77 180)
-    (effects (font (size 1.27 1.27)) (justify right))
+  (hierarchical_label "PTT-IN" (shape input) (at 102.87 49.53 0)
+    (effects (font (size 1.27 1.27)) (justify left))
   )
   (symbol (lib_id "xenir:Resistor") (at 201.93 120.65 90) (unit 1)
@@
   (symbol (lib_id "power:+3V3") (at 161.29 41.91 0) (unit 1)
     (in_bom yes) (on_board yes)
-    (property "Reference" "#PWR?" (id 0) (at 161.29 45.72 0)
+    (property "Reference" "#PWR0203" (id 0) (at 161.29 45.72 0)
       (effects (font (size 1.27 1.27)) hide)
     )
@@
     (pin "S2")
   )
-  (symbol (lib_id "power:+3V3") (at 59.69 36.83 0) (unit 1)
-    (in_bom yes) (on_board yes)
-    (property "Reference" "#PWR0195" (id 0) (at 59.69 40.64 0)
-      (effects (font (size 1.27 1.27)) hide)
-    )
-    (property "Value" "+3V3" (id 1) (at 58.42 33.02 0))
-    (property "Footprint" "" (id 2) (at 59.69 36.83 0)
-      (effects (font (size 1.27 1.27)) hide)
-    )
-    (property "Datasheet" "" (id 3) (at 59.69 36.83 0)
-      (effects (font (size 1.27 1.27)) hide)
-    )
-    (pin "1")
-  )
   (symbol (lib_id "power:+3V3") (at 151.13 41.91 0) (unit 1)
     (in_bom yes) (on_board yes)
-    (property "Reference" "#PWR?" (id 0) (at 151.13 45.72 0)
-      (effects (font (size 1.27 1.27)) hide)
-    )
+    (property "Reference" "#PWR0205" (id 0) (at 151.13 45.72 0)
+      (effects (font (size 1.27 1.27)) hide)
+    )
